Commit message: feat: add dual-walkie-arm, refact: arm_ros2_control.xacro

File: robots/left-walkie-arm.urdf.xacro (robot description, xacro)
@@ -8,5 +8,5 @@
     <xacro:include filename="$(find walkie_description)/urdf/walkie-arm/walkie_arm.urdf.xacro" />
     <xacro:include filename="$(find walkie_description)/urdf/walkie-gripper/walkie_gripper.urdf.xacro" />
-    <xacro:include filename="$(find walkie_description)/urdf/walkie/left_arm_ros2_control.xacro" />
+    <xacro:include filename="$(find walkie_description)/urdf/walkie/arm_ros2_control.xacro" />
     <xacro:walkie_arm base_link="$(arg base_link)" prefix="left" />
     <xacro:if value="$(arg use_gripper)">
@@ -36,5 +36,5 @@
       <material>Gazebo/Grey</material>
     </gazebo>
-    <xacro:left_arm_ros2_control
+    <xacro:arm_ros2_control
         name="LeftWalkieSystem"
         prefix="left"

File: urdf/walkie/arm_ros2_control.xacro (robot description, xacro)
@@ -1,8 +1,8 @@
 <?xml version="1.0"?>
 <robot xmlns:xacro="http://www.ros.org/wiki/xacro">
-  <xacro:macro name="left_arm_ros2_control" params="name prefix hardware_config_file">
+  <xacro:macro name="arm_ros2_control" params="name prefix hardware_config_file">
     <xacro:property name="hw_config" value="${xacro.load_yaml(hardware_config_file)}"/>
     <xacro:if value="${'cubemars' in hw_config['hardware_config'].values()}">
-      <ros2_control name="RealSystem" type="system">
+      <ros2_control name="${name}Real" type="system">
         <hardware>
           <plugin>cubemars_hardware/CubeMarsSystemHardware</plugin>
@@ -12,5 +12,5 @@
       </ros2_control>
     </xacro:if>
-    <ros2_control name="MockSystem" type="system">
+    <ros2_control name="${name}Mock" type="system">
       <hardware>
          <plugin>mock_components/GenericSystem</plugin>
