Commit message: refactor:urdf for moveit + joints axis fix

File: robots/gz_walkie_1arm_moveit.urdf.xacro (robot description, xacro)
@@ -11,8 +11,8 @@
   <xacro:arg name="dual_lidar" default="True"/>
   <xacro:include filename="$(find walkie_description)/urdf/walkie/base/base.urdf.xacro"/>
-  <xacro:include filename="$(find walkie_description)/urdf/walkie/omni_wheel/gz_omni_wheel.urdf.xacro"/>
+  <!-- <xacro:include filename="$(find walkie_description)/urdf/walkie/omni_wheel/gz_omni_wheel.urdf.xacro"/>
   <xacro:include filename="$(find walkie_description)/urdf/walkie/lidar/lidar_gz.urdf.xacro"/>
   <xacro:include filename="$(find walkie_description)/urdf/walkie/imu/imu_gz.urdf.xacro"/>
-  <xacro:include filename="$(find walkie_description)/urdf/walkie/depth_camera/d415.urdf.xacro"/>
+  <xacro:include filename="$(find walkie_description)/urdf/walkie/depth_camera/d415.urdf.xacro"/> -->
   <!-- Include the arm and gripper macros -->
   <xacro:include filename="$(find walkie_description)/urdf/walkie-arm/walkie_arm.urdf.xacro"/>
@@ -34,5 +34,5 @@
   <xacro:base_gazebo_v0/>
   <!-- Wheel -->
-  <xacro:wheel_v0 prefix="bl" parent="base_link">
+  <!-- <xacro:wheel_v0 prefix="bl" parent="base_link">
     <origin xyz="0.145261 0.145261 0.05" rpy="0 0 -${M_PI/4}"/>
     <axis xyz="0.0 1.0 0.0"/>
@@ -49,5 +49,5 @@
     <origin xyz="0.145261 -0.145261 0.05" rpy="0 0 ${5*M_PI/4}"/>
     <axis xyz="0.0 1.0 0.0"/>
-  </xacro:wheel_v0>
+  </xacro:wheel_v0> -->
   <!-- Left arm mount joint -->
   <joint name="left_arm_mount_joint" type="fixed">
@@ -89,5 +89,5 @@
   <!-- lidar sensor -->
   <!-- single lidar for simulation performance -->
- <xacro:if value="${'$(arg ros2_control)' == 'gazebo' and not $(arg dual_lidar)}">
+  <!-- <xacro:if value="${'$(arg ros2_control)' == 'gazebo' and not $(arg dual_lidar)}">
     <xacro:lidar_v0 prefix="single" parent="base_link">
       <origin xyz="0 0 0.315" rpy="0 0 -1.5707963"/>
@@ -119,5 +119,5 @@
   <xacro:imu_gazebo_v0 prefix="top"/>
   <xacro:include filename="$(find walkie_description)/urdf/walkie/ros2_control.xacro"/>
-  <xacro:ros2_control ros2_control="$(arg ros2_control)"/>
+  <xacro:ros2_control ros2_control="$(arg ros2_control)"/>  -->
   <xacro:arm_ros2_control name="LeftWalkieSystem" prefix="left" hardware_type="$(arg ros2_control_hardware_type)" hardware_config_file="$(arg hardware_config_file)"/>
 </robot>

File: urdf/walkie-arm/walkie_arm.urdf.xacro (robot description, xacro)
@@ -30,5 +30,5 @@
     </link>
     <joint name="${prefix}_joint1" type="revolute">
-      <axis xyz="1.0 0.0 0.0" />
+      <axis xyz="-1.0 0.0 0.0" />
       <limit effort="${joint_effort}" lower="-3.14" upper="3.14" velocity="${joint_velocity}" />
       <parent link="${base_link}" />
@@ -48,5 +48,5 @@
         <origin rpy="-1.57080 1.57080 0.00000" xyz="0.04418 0.00000 -0.00000"/>
         <geometry>
-          <cylinder radius="0.04393" length="0.09802"/>
+          <cylinder radius="0.04393" length="0.098"/>
         </geometry>
       </collision>
@@ -57,9 +57,9 @@
     </link>
     <joint name="${prefix}_joint2" type="revolute">
-      <axis xyz="0.0 -1.0 0.0" />
-      <limit effort="${joint_effort}" lower="-1.57" upper="1.57" velocity="${joint_velocity}" />
+      <axis xyz="0.0 1.0 0.0" />
+      <limit effort="${joint_effort}" lower="-3.14" upper="0.0" velocity="${joint_velocity}" />
       <parent link="${prefix}_link1" />
       <child link="${prefix}_link2" />
-      <origin xyz="0.04425 -0.03925 0.0" rpy="0.0 -1.57 0.0" />
+      <origin xyz="0.04425 -0.03925 0.0" rpy="0.0 0.0 0.0" />
       <dynamics damping="${joint_damping}" friction="${joint_friction}" />
     </joint>
@@ -75,5 +75,5 @@
         <origin rpy="0.00000 0.00000 0.00000" xyz="-0.00000 0.03929 -0.12406"/>
         <geometry>
-          <cylinder radius="0.04469" length="0.15440"/>
+          <cylinder radius="0.04469" length="0.15"/>
         </geometry>
       </collision>
@@ -84,5 +84,5 @@
     </link>
     <joint name="${prefix}_joint3" type="revolute">
-      <axis xyz="0.0 0.0 -1.0" />
+      <axis xyz="0.0 0.0 1.0" />
       <limit effort="${joint_effort}" lower="-3.14" upper="3.14" velocity="${joint_velocity}" />
       <parent link="${prefix}_link2" />
@@ -102,5 +102,5 @@
         <origin rpy="-0.00000 1.57080 -0.00000" xyz="-0.00103 -0.00000 -0.11471"/>
         <geometry>
-          <cylinder radius="0.04497" length="0.09083"/>
+          <cylinder radius="0.044" length="0.09"/>
         </geometry>
       </collision>
@@ -129,5 +129,5 @@
         <origin rpy="0.00000 0.00000 0.00000" xyz="-0.03467 -0.00059 -0.09265"/>
         <geometry>
-          <cylinder radius="0.03436" length="0.09152"/>
+          <cylinder radius="0.034" length="0.09"/>
         </geometry>
       </collision>
@@ -139,8 +139,8 @@
     <joint name="${prefix}_joint5" type="revolute">
       <axis xyz="-1.0 0.0 0.0" />
-      <limit effort="${joint_effort}" lower="-1.57" upper="1.57" velocity="${joint_velocity}" />
+      <limit effort="${joint_effort}" lower="-3.14" upper="0.0" velocity="${joint_velocity}" />
       <parent link="${prefix}_link4" />
       <child link="${prefix}_link5" />
-      <origin xyz="-0.05962 0.0 -0.12200" rpy="0.0 0.0 0.0" />
+      <origin xyz="-0.05962 0.0 -0.12200" rpy="-1.57 0.0 0.0" />
       <dynamics damping="${joint_damping}" friction="${joint_friction}" />
     </joint>
@@ -156,5 +156,5 @@
         <origin rpy="1.57080 0.00000 0.00000" xyz="0.02026 0.00000 -0.06561"/>
         <geometry>
-          <cylinder radius="0.03329" length="0.06786"/>
+          <cylinder radius="0.0285" length="0.067"/>
         </geometry>
       </collision>
@@ -165,5 +165,5 @@
     </link>
     <joint name="${prefix}_joint6" type="revolute">
-      <axis xyz="0.0 -1.0 0.0" />
+      <axis xyz="0.0 1.0 0.0" />
       <limit effort="${joint_effort}" lower="-1.57" upper="1.57" velocity="${joint_velocity}" />
       <parent link="${prefix}_link5" />
@@ -183,5 +183,5 @@
         <origin rpy="0.00000 0.00000 0.00000" xyz="-0.00000 0.02829 -0.08677"/>
         <geometry>
-          <cylinder radius="0.03852" length="0.10036"/>
+          <cylinder radius="0.038" length="0.100"/>
         </geometry>
       </collision>

File: urdf/walkie-gripper/walkie_gripper.urdf.xacro (robot description, xacro)
@@ -40,5 +40,5 @@
         <origin rpy="0.0 0.0 0.0" xyz="0.0 0.0 -0.03004"/>
         <geometry>
-          <box size="0.12520 0.05916 0.05330"/>
+          <box size="0.125 0.059 0.053"/>
         </geometry>
       </collision>
@@ -54,4 +54,10 @@
         </geometry>
       </visual>
+      <!-- <collision>
+        <origin rpy="0.0 0.0 0.0" xyz="0.0 0.0 0.0" />
+        <geometry>
+          <cylinder length="0.05" radius="0.015"/>
+        </geometry>
+      </collision> -->
     </link>
     <joint name="${prefix}_gripper_worm_gear_joint" type="revolute">
@@ -71,4 +77,12 @@
         </geometry>
       </visual>
+      <!-- collision removed to simplify planning / avoid duplicate geometry
+      <collision>
+        <origin rpy="0.0 0.0 0.0" xyz="0.0 0.0 0.0" />
+        <geometry>
+          <box size="0.02 0.02 0.06"/>
+        </geometry>
+      </collision>
+      -->
     </link>
     <joint name="${prefix}_gripper_gear_r_joint" type="revolute">
@@ -89,4 +103,12 @@
         </geometry>
       </visual>
+      <!-- collision removed to simplify planning / avoid duplicate geometry
+      <collision>
+        <origin rpy="0.0 0.0 0.0" xyz="0.0 0.0 0.0" />
+        <geometry>
+          <box size="0.02 0.02 0.06"/>
+        </geometry>
+      </collision>
+      -->
     </link>
     <joint name="${prefix}_gripper_gear_l_joint" type="revolute">
@@ -155,4 +177,10 @@
         </geometry>
       </visual>
+      <!-- <collision>
+        <origin rpy="0.0 0.0 0.0" xyz="0.0 0.0 0.0" />
+        <geometry>
+          <box size="0.01 0.015 0.03"/>
+        </geometry> -->
+      <!-- </collision> -->
     </link>
     <joint name="${prefix}_gripper_connector_r_joint" type="revolute">
@@ -173,4 +201,10 @@
         </geometry>
       </visual>
+      <!-- <collision> -->
+        <!-- <origin rpy="0.0 0.0 0.0" xyz="0.0 0.0 0.0" />
+        <geometry>
+          <box size="0.01 0.015 0.03"/>
+        </geometry>
+      </collision> -->
     </link>
     <joint name="${prefix}_gripper_connector_l_joint" type="revolute">

File: urdf/walkie/base/base.urdf.xacro (robot description, xacro)
@@ -21,15 +21,15 @@
         <material name="grey"/>
       </visual>
+      <!-- Simplified collision: single cylinder to reduce complexity for planning -->
       <collision>
         <origin xyz="0 0 0.165" rpy="0 0 0"/>
         <geometry>
-          <cylinder radius="0.3" length="0.33"/>
-          <!-- <mesh filename="package://walkie_description/meshes/walkie/base_link_collision.stl"/> -->
+          <cylinder radius="0.29" length="0.33"/>
         </geometry>
       </collision>
       <collision>
-        <origin xyz="0 0 0.615" rpy="0 0 0"/>
+        <origin xyz="0 0 0.605" rpy="0 0 0"/>
         <geometry>
-          <box size="0.32 0.2 0.57"/>
+          <box size="0.3 0.19 0.54"/>
         </geometry>
       </collision>

File: urdf/walkie/omni_wheel/gz_omni_wheel.urdf.xacro (robot description, xacro)
@@ -25,32 +25,16 @@
         </geometry>
       </visual>
+      <collision>
+        <geometry>
+          <cylinder length="${wheel_thickness}" radius="${wheel_radian}"/>
+        </geometry>
+        <origin xyz="0 ${wheel_thickness/2} 0" rpy="1.570796327 0 0"/>
+      </collision>
       <xacro:inertial_cylinder mass="${wheel_mass}" length="${wheel_thickness}" radius="${wheel_radian}">
         <origin xyz="0 ${wheel_thickness/2} 0" rpy="1.570796327 0 0"/>
       </xacro:inertial_cylinder>
     </link>
-    <xacro:roller prefix="${prefix}" num="1">
-      <origin xyz="0.0577 0.012 0.0" rpy="0.0 -0.0 0.0"/>
-      <axis xyz="0.0 0.0 1.0"/>
-    </xacro:roller>
-    <xacro:roller prefix="${prefix}" num="2">
-      <origin xyz="0.05 0.012 0.0289" rpy="0.0 -0.5236 0.0"/>
-      <axis xyz="0.0 0.0 1.0"/>
-    </xacro:roller>
-    <xacro:roller prefix="${prefix}" num="3">
-      <origin xyz="0.0289 0.012 0.05" rpy="0.0 -1.0472 0.0"/>
-      <axis xyz="0.0 0.0 1.0"/>
-    </xacro:roller>
-    <xacro:roller prefix="${prefix}" num="4">
-      <origin xyz="0.0 0.012 0.0577" rpy="0.0 -1.5708 0.0"/>
-      <axis xyz="0.0 0.0 1.0"/>
-    </xacro:roller>
-    <xacro:roller prefix="${prefix}" num="5">
-      <origin xyz="-0.0289 0.012 0.05" rpy="0.0 -2.0944 0.0"/>
-      <axis xyz="0.0 0.0 1.0"/>
-    </xacro:roller>
-    <xacro:roller prefix="${prefix}" num="6">
-      <origin xyz="-0.05 0.012 0.0289" rpy="0.0 -2.618 0.0"/>
-      <axis xyz="0.0 0.0 1.0"/>
-    </xacro:roller>
+    <!-- Rollers removed to simplify collision and joint count for planning -->
+    <!-- xacro:roller blocks intentionally omitted -->
     <xacro:roller prefix="${prefix}" num="7">
       <origin xyz="-0.0577 0.012 0.0" rpy="0.0 -3.1416 0.0"/>
