Commit message: refactor: switch main URDF from drivebase-with-arm to drivebase-only

File: robots/gz_walkie_1arm.urdf.xacro (robot description, xacro)
@@ -21,4 +21,11 @@
   <xacro:include
         filename="$(find walkie_description)/urdf/walkie/depth_camera/d415.urdf.xacro"
+    />
+  <!-- Include the arm and gripper macros -->
+  <xacro:include
+        filename="$(find walkie_description)/urdf/walkie-arm/walkie_arm.urdf.xacro"
+    />
+  <xacro:include
+        filename="$(find walkie_description)/urdf/walkie-gripper/walkie_gripper.urdf.xacro"
     />
   <!-- =============== Link & Joint =============== -->
@@ -50,4 +57,37 @@
     <axis xyz="0.0 1.0 0.0" />
   </xacro:wheel_v0>
+  <!-- Left arm base mount -->
+  <link name="left_arm_base">
+      <!-- <visual>
+        <geometry>
+          <cylinder radius="0.05" length="0.05" />
+        </geometry>
+        <origin xyz="0 0 0.025" rpy="0 0 0" />
+        <material name="mount_material">
+          <color rgba="0.3 0.3 0.3 1.0" />
+        </material>
+      </visual> -->
+  </link>
+  <!-- Left arm mount joint -->
+  <joint name="left_arm_mount_joint" type="fixed">
+    <parent link="base_link" />
+    <child link="left_arm_base" />
+    <origin
+          xyz="0.075 0 0.9018"
+          rpy="0 0 0"
+      />
+  </joint>
+  <!-- Left arm -->
+  <xacro:walkie_arm
+        base_link="arm_base"
+        flange_link="link_flange"
+        prefix="left"
+  >
+    <origin xyz="0 0 0.05" rpy="0 0 0" />
+  </xacro:walkie_arm>
+  <!-- Left gripper (optional) -->
+  <xacro:walkie_gripper parent="link_flange" prefix="left">
+      <origin xyz="0 0 0" rpy="3.141592653589793 0 0" />
+  </xacro:walkie_gripper>
   <!-- lidar sensor -->
   <!-- single lidar for simulation performance -->

Commit message: feat: update gzwalkie_robot model to latest walkie-arm

File: robots/gz_walkie_1arm.urdf.xacro (robot description, xacro)
@@ -1,162 +1,123 @@
-<?xml version="1.0" ?>
-<robot xmlns:xacro="http://ros.org/wiki/xacro" name="walkie_bot">
-  <xacro:property name="M_PI" value="3.14159274" />
-  <xacro:arg name="ros2_control" default="gazebo" />
+<?xml version="1.0"?>
+<robot xmlns:xacro="http://www.ros.org/wiki/xacro" name="walkie_bot">
+  <xacro:property name="M_PI" value="3.14159274"/>
+  <xacro:arg name="ros2_control" default="gazebo"/>
+  <xacro:arg name="use_gripper" default="true"/>
+  <xacro:arg name="ros2_control_hardware_type" default="mock_components"/>
+  <xacro:arg name="hardware_config_file" default="$(find walkie_description)/config/hardware_layout.yaml"/>
   <!-- Dual lidar option when only SIMULATION
   real robot force to be dual_lidar
   don't forgot to enable lidar topic to bridge in gz_bridge.yml -->
-  <xacro:arg name="dual_lidar" default="True" />
-  <xacro:include
-        filename="$(find walkie_description)/urdf/walkie/base/base.urdf.xacro"
-    />
-  <xacro:include
-        filename="$(find walkie_description)/urdf/walkie/omni_wheel/gz_omni_wheel.urdf.xacro"
-    />
-  <xacro:include
-        filename="$(find walkie_description)/urdf/walkie/lidar/lidar_gz.urdf.xacro"
-    />
-  <xacro:include
-        filename="$(find walkie_description)/urdf/walkie/imu/imu_gz.urdf.xacro"
-    />
-  <xacro:include
-        filename="$(find walkie_description)/urdf/walkie/depth_camera/d415.urdf.xacro"
-    />
+  <xacro:arg name="dual_lidar" default="True"/>
+  <xacro:include filename="$(find walkie_description)/urdf/walkie/base/base.urdf.xacro"/>
+  <xacro:include filename="$(find walkie_description)/urdf/walkie/omni_wheel/gz_omni_wheel.urdf.xacro"/>
+  <xacro:include filename="$(find walkie_description)/urdf/walkie/lidar/lidar_gz.urdf.xacro"/>
+  <xacro:include filename="$(find walkie_description)/urdf/walkie/imu/imu_gz.urdf.xacro"/>
+  <xacro:include filename="$(find walkie_description)/urdf/walkie/depth_camera/d415.urdf.xacro"/>
   <!-- Include the arm and gripper macros -->
-  <xacro:include
-        filename="$(find walkie_description)/urdf/walkie-arm/walkie_arm.urdf.xacro"
-    />
-  <xacro:include
-        filename="$(find walkie_description)/urdf/walkie-gripper/walkie_gripper.urdf.xacro"
-    />
+  <xacro:include filename="$(find walkie_description)/urdf/walkie-arm/walkie_arm.urdf.xacro"/>
+  <xacro:include filename="$(find walkie_description)/urdf/walkie-gripper/walkie_gripper.urdf.xacro"/>
+  <xacro:include filename="$(find walkie_description)/urdf/walkie-arm/arm_ros2_control.xacro"/>
   <!-- =============== Link & Joint =============== -->
   <!-- Base -->
-  <link name="base_footprint" />
+  <link name="base_footprint"/>
   <xacro:base_v0 parent="base_footprint">
-    <origin xyz="0 0 0" rpy="0 0 ${M_PI / 2}" />
+    <origin xyz="0 0 0" rpy="0 0 ${M_PI / 2}"/>
   </xacro:base_v0>
-  <xacro:base_gazebo_v0 />
+  <xacro:base_gazebo_v0/>
   <!-- Wheel -->
   <!-- 1st wheel -->
   <xacro:wheel_v0 prefix="bl" parent="base_link">
-    <origin xyz="0.145261 0.145261 0.05" rpy="0 0 -${M_PI/4}" />
-    <axis xyz="0.0 1.0 0.0" />
+    <origin xyz="0.145261 0.145261 0.05" rpy="0 0 -${M_PI/4}"/>
+    <axis xyz="0.0 1.0 0.0"/>
   </xacro:wheel_v0>
   <!-- 2nd wheel -->
   <xacro:wheel_v0 prefix="br" parent="base_link">
-    <origin xyz="-0.145261 0.145261 0.05" rpy="0 0 ${M_PI/4}" />
-    <axis xyz="0.0 1.0 0.0" />
+    <origin xyz="-0.145261 0.145261 0.05" rpy="0 0 ${M_PI/4}"/>
+    <axis xyz="0.0 1.0 0.0"/>
   </xacro:wheel_v0>
   <!-- 3rd wheel -->
   <xacro:wheel_v0 prefix="fr" parent="base_link">
-    <origin xyz="-0.145261 -0.145261 0.05" rpy="0 0 ${3*M_PI/4}" />
-    <axis xyz="0.0 1.0 0.0" />
+    <origin xyz="-0.145261 -0.145261 0.05" rpy="0 0 ${3*M_PI/4}"/>
+    <axis xyz="0.0 1.0 0.0"/>
   </xacro:wheel_v0>
   <!-- 4th wheel -->
   <xacro:wheel_v0 prefix="fl" parent="base_link">
-    <origin xyz="0.145261 -0.145261 0.05" rpy="0 0 ${5*M_PI/4}" />
-    <axis xyz="0.0 1.0 0.0" />
+    <origin xyz="0.145261 -0.145261 0.05" rpy="0 0 ${5*M_PI/4}"/>
+    <axis xyz="0.0 1.0 0.0"/>
   </xacro:wheel_v0>
-  <!-- Left arm base mount -->
-  <link name="left_arm_base">
-      <!-- <visual>
-        <geometry>
-          <cylinder radius="0.05" length="0.05" />
-        </geometry>
-        <origin xyz="0 0 0.025" rpy="0 0 0" />
-        <material name="mount_material">
-          <color rgba="0.3 0.3 0.3 1.0" />
-        </material>
-      </visual> -->
-  </link>
   <!-- Left arm mount joint -->
   <joint name="left_arm_mount_joint" type="fixed">
-    <parent link="base_link" />
-    <child link="left_arm_base" />
-    <origin
-          xyz="0.075 0 0.9018"
-          rpy="0 0 0"
-      />
+    <parent link="base_link"/>
+    <child link="left_arm_base"/>
+    <origin xyz="0.075 0 0.951268" rpy="0 0 0"/>
   </joint>
   <!-- Left arm -->
-  <xacro:walkie_arm
-        base_link="arm_base"
-        flange_link="link_flange"
-        prefix="left"
-  >
-    <origin xyz="0 0 0.05" rpy="0 0 0" />
-  </xacro:walkie_arm>
-  <!-- Left gripper (optional) -->
-  <xacro:walkie_gripper parent="link_flange" prefix="left">
-      <origin xyz="0 0 0" rpy="3.141592653589793 0 0" />
-  </xacro:walkie_gripper>
+  <xacro:walkie_arm base_link="left_arm_base" prefix="left"/>
+  <xacro:if value="$(arg use_gripper)">
+    <xacro:walkie_gripper parent="left_link6" prefix="left"/>
+  </xacro:if>
+  <xacro:if value="$(arg use_gripper)">
+    <link name="left_gripper_center">
+      <visual>
+        <geometry>
+          <sphere radius="0.01"/>
+        </geometry>
+        <material name="red">
+          <color rgba="1 0 0 1"/>
+        </material>
+      </visual>
+      <collision>
+        <geometry>
+          <sphere radius="0.01"/>
+        </geometry>
+      </collision>
+      <inertial>
+        <mass value="0.001"/>
+        <inertia ixx="1e-6" ixy="0" ixz="0" iyy="1e-6" iyz="0" izz="1e-6"/>
+      </inertial>
+    </link>
+    <joint name="left_gripper_center_joint" type="fixed">
+      <parent link="left_link7"/>
+      <child link="left_gripper_center"/>
+      <origin xyz="0.0 0.0 -0.18" rpy="0.0 0.0 0.0"/>
+    </joint>
+  </xacro:if>
   <!-- lidar sensor -->
   <!-- single lidar for simulation performance -->
-  <xacro:if
-        value="${'$(arg ros2_control)' == 'gazebo' and not $(arg dual_lidar)}"
-    >
+  <xacro:if value="${'$(arg ros2_control)' == 'gazebo' and not $(arg dual_lidar)}">
     <xacro:lidar_v0 prefix="single" parent="base_link">
-      <origin xyz="0 0 0.315" rpy="0 0 -1.5707963" />
+      <origin xyz="0 0 0.315" rpy="0 0 -1.5707963"/>
     </xacro:lidar_v0>
-    <xacro:lidar_gazebo_v0
-            prefix="single"
-            min_rad="-${M_PI}"
-            max_rad=" ${M_PI}"
-            min_range="0.2"
-            max_range="10"
-            yaw_offset="0"
-        />
+    <xacro:lidar_gazebo_v0 prefix="single" min_rad="-${M_PI}" max_rad=" ${M_PI}" min_range="0.2" max_range="10" yaw_offset="0"/>
   </xacro:if>
   <!-- dual lidar when ** REAL WORLD ** or ** SIMULATION ** but set argument ** DUAL_LIDAR ** to true -->
-  <xacro:unless
-        value="${'$(arg ros2_control)' == 'gazebo' and not $(arg dual_lidar)}"
-    >
-  <xacro:lidar_v0 prefix="front" parent="base_link">
-      <origin xyz="0 -0.240 0.28232" rpy="0 0 -1.5707963" />
+  <xacro:unless value="${'$(arg ros2_control)' == 'gazebo' and not $(arg dual_lidar)}">
+    <xacro:lidar_v0 prefix="front" parent="base_link">
+      <origin xyz="0 -0.240 0.28232" rpy="0 0 -1.5707963"/>
     </xacro:lidar_v0>
     <xacro:lidar_v0 prefix="back" parent="base_link">
-      <origin xyz="0 0.240 0.28232" rpy="0 0 1.5707963" />
+      <origin xyz="0 0.240 0.28232" rpy="0 0 1.5707963"/>
     </xacro:lidar_v0>
-    <xacro:lidar_gazebo_v0
-            prefix="front"
-            min_rad="-2.09333333"
-            max_rad=" 2.09333333"
-            min_range="0.18"
-            max_range="10"
-            yaw_offset="0"
-        />
-    <xacro:lidar_gazebo_v0
-            prefix="back"
-            min_rad="-2.09333333"
-            max_rad=" 2.09333333"
-            min_range="0.18"
-            max_range="10"
-            yaw_offset="0"
-        />
+    <xacro:lidar_gazebo_v0 prefix="front" min_rad="-2.09333333" max_rad=" 2.09333333" min_range="0.18" max_range="10" yaw_offset="0"/>
+    <xacro:lidar_gazebo_v0 prefix="back" min_rad="-2.09333333" max_rad=" 2.09333333" min_range="0.18" max_range="10" yaw_offset="0"/>
   </xacro:unless>
   <!-- depth cam sensor -->
-  <xacro:sensor_d415
-        name="bottom"
-        parent="base_link"
-        flag_color="1"
-        flag_ir="0"
-        flag_depth="1"
-        updaterate="2"
-    >
-    <origin xyz="0 -0.282713 0.1775" rpy="0 -0.453786 -${M_PI/2}" />
+  <xacro:sensor_d415 name="bottom" parent="base_link" flag_color="1" flag_ir="0" flag_depth="1" updaterate="2">
+    <origin xyz="0 -0.282713 0.1775" rpy="0 -0.453786 -${M_PI/2}"/>
   </xacro:sensor_d415>
-  <link name="bottombase" />
+  <link name="bottombase"/>
   <joint name="bottombase_joint" type="fixed">
-      <parent link="base_link" />
-      <child link="bottombase" />
-      <origin xyz="0 -0.282713 0.1775" rpy="0 0 -${M_PI/2}" />
+    <parent link="base_link"/>
+    <child link="bottombase"/>
+    <origin xyz="0 -0.282713 0.1775" rpy="0 0 -${M_PI/2}"/>
   </joint>
   <!-- imu sensor -->
   <xacro:imu_v0 prefix="top" parent="base_link">
-    <origin xyz="0 0 0.17" />
+    <origin xyz="0 0 0.17"/>
   </xacro:imu_v0>
-  <xacro:imu_gazebo_v0 prefix="top" />
-  <xacro:include
-        filename="$(find walkie_description)/urdf/walkie/ros2_control.xacro"
-    />
-  <xacro:ros2_control ros2_control="$(arg ros2_control)" />
+  <xacro:imu_gazebo_v0 prefix="top"/>
+  <xacro:include filename="$(find walkie_description)/urdf/walkie/ros2_control.xacro"/>
+  <xacro:arm_ros2_control name="LeftWalkieSystem" prefix="left" hardware_type="$(arg ros2_control_hardware_type)" hardware_config_file="$(arg hardware_config_file)"/>
+  <xacro:ros2_control ros2_control="$(arg ros2_control)"/>
 </robot>

Commit message: feat: add servo base and link for depthcam mount

File: robots/gz_walkie_1arm.urdf.xacro (robot description, xacro)
@@ -15,4 +15,5 @@
   <xacro:include filename="$(find walkie_description)/urdf/walkie/imu/imu_gz.urdf.xacro"/>
   <xacro:include filename="$(find walkie_description)/urdf/walkie/depth_camera/d415.urdf.xacro"/>
+  <xacro:include filename="$(find walkie_description)/urdf/walkie/head/servo_camera.urdf.xacro"/>
   <!-- Include the arm and gripper macros -->
   <xacro:include filename="$(find walkie_description)/urdf/walkie-arm/walkie_arm.urdf.xacro"/>
@@ -104,4 +105,5 @@
   </xacro:unless>
   <!-- depth cam sensor -->
+  <!-- d415 -->
   <xacro:sensor_d415 name="bottom" parent="base_link" flag_color="1" flag_ir="0" flag_depth="1" updaterate="2">
     <origin xyz="0 -0.282713 0.1775" rpy="0 -0.453786 -${M_PI/2}"/>
@@ -113,4 +115,7 @@
     <origin xyz="0 -0.282713 0.1775" rpy="0 0 -${M_PI/2}"/>
   </joint>
+  <xacro:servo_v0 prefix="head" parent="base_link">
+    <origin xyz="-0.098 -0.1195 0.848" rpy="0 0 0"/>
+  </xacro:servo_v0>
   <!-- imu sensor -->
   <xacro:imu_v0 prefix="top" parent="base_link">

Commit message: fix: restore gz_omni_wheel roller, gz_walkie_1arm to before changed

File: robots/gz_walkie_1arm.urdf.xacro (robot description, xacro)
@@ -19,11 +19,4 @@
   <xacro:include filename="$(find walkie_description)/urdf/walkie-gripper/walkie_gripper.urdf.xacro"/>
   <xacro:include filename="$(find walkie_description)/urdf/walkie-arm/arm_ros2_control.xacro"/>
-  <!-- =============== Virtual World Joint for MoveIt =============== -->
-  <link name="world"/>
-  <joint name="virtual_world_joint" type="fixed">
-    <parent link="world"/>
-    <child link="base_footprint"/>
-    <origin xyz="0 0 0" rpy="0 0 0"/>
-  </joint>
   <!-- =============== Link & Joint =============== -->
   <!-- Base -->
@@ -34,16 +27,20 @@
   <xacro:base_gazebo_v0/>
   <!-- Wheel -->
+  <!-- 1st wheel -->
   <xacro:wheel_v0 prefix="bl" parent="base_link">
     <origin xyz="0.145261 0.145261 0.05" rpy="0 0 -${M_PI/4}"/>
     <axis xyz="0.0 1.0 0.0"/>
   </xacro:wheel_v0>
+  <!-- 2nd wheel -->
   <xacro:wheel_v0 prefix="br" parent="base_link">
     <origin xyz="-0.145261 0.145261 0.05" rpy="0 0 ${M_PI/4}"/>
     <axis xyz="0.0 1.0 0.0"/>
   </xacro:wheel_v0>
+  <!-- 3rd wheel -->
   <xacro:wheel_v0 prefix="fr" parent="base_link">
     <origin xyz="-0.145261 -0.145261 0.05" rpy="0 0 ${3*M_PI/4}"/>
     <axis xyz="0.0 1.0 0.0"/>
   </xacro:wheel_v0>
+  <!-- 4th wheel -->
   <xacro:wheel_v0 prefix="fl" parent="base_link">
     <origin xyz="0.145261 -0.145261 0.05" rpy="0 0 ${5*M_PI/4}"/>
@@ -71,9 +68,9 @@
         </material>
       </visual>
-      <!-- <collision>
+      <collision>
         <geometry>
           <sphere radius="0.01"/>
         </geometry>
-      </collision> -->
+      </collision>
       <inertial>
         <mass value="0.001"/>
@@ -89,5 +86,5 @@
   <!-- lidar sensor -->
   <!-- single lidar for simulation performance -->
- <xacro:if value="${'$(arg ros2_control)' == 'gazebo' and not $(arg dual_lidar)}">
+  <xacro:if value="${'$(arg ros2_control)' == 'gazebo' and not $(arg dual_lidar)}">
     <xacro:lidar_v0 prefix="single" parent="base_link">
       <origin xyz="0 0 0.315" rpy="0 0 -1.5707963"/>
@@ -95,4 +92,5 @@
     <xacro:lidar_gazebo_v0 prefix="single" min_rad="-${M_PI}" max_rad=" ${M_PI}" min_range="0.6" max_range="10" yaw_offset="0"/>
   </xacro:if>
+  <!-- dual lidar when ** REAL WORLD ** or ** SIMULATION ** but set argument ** DUAL_LIDAR ** to true -->
   <xacro:unless value="${'$(arg ros2_control)' == 'gazebo' and not $(arg dual_lidar)}">
     <xacro:lidar_v0 prefix="front" parent="base_link">
@@ -105,4 +103,5 @@
     <xacro:lidar_gazebo_v0 prefix="back" min_rad="-2.09333333" max_rad=" 2.09333333" min_range="0.18" max_range="10" yaw_offset="0"/>
   </xacro:unless>
+  <!-- depth cam sensor -->
   <xacro:sensor_d415 name="bottom" parent="base_link" flag_color="1" flag_ir="0" flag_depth="1" updaterate="2">
     <origin xyz="0 -0.282713 0.1775" rpy="0 -0.453786 -${M_PI/2}"/>
@@ -114,4 +113,5 @@
     <origin xyz="0 -0.282713 0.1775" rpy="0 0 -${M_PI/2}"/>
   </joint>
+  <!-- imu sensor -->
   <xacro:imu_v0 prefix="top" parent="base_link">
     <origin xyz="0 0 0.17"/>

File: urdf/walkie/base/base.urdf.xacro (robot description, xacro)
@@ -16,10 +16,8 @@
       <visual>
         <geometry>
-          <!-- <mesh filename="package://walkie_description/meshes/walkie/base_link.dae"/> -->
           <mesh filename="package://walkie_description/meshes/walkie/base_link2.stl"/>
         </geometry>
         <material name="grey"/>
       </visual>
-      <!-- Simplified collision: single cylinder to reduce complexity for planning -->
       <collision>
         <origin xyz="0 0 0.165" rpy="0 0 0"/>

File: urdf/walkie/omni_wheel/gz_omni_wheel.urdf.xacro (robot description, xacro)
@@ -25,16 +25,32 @@
         </geometry>
       </visual>
-      <collision>
-        <geometry>
-          <cylinder length="${wheel_thickness}" radius="${wheel_radian}"/>
-        </geometry>
-        <origin xyz="0 ${wheel_thickness/2} 0" rpy="1.570796327 0 0"/>
-      </collision>
       <xacro:inertial_cylinder mass="${wheel_mass}" length="${wheel_thickness}" radius="${wheel_radian}">
         <origin xyz="0 ${wheel_thickness/2} 0" rpy="1.570796327 0 0"/>
       </xacro:inertial_cylinder>
     </link>
-    <!-- Rollers removed to simplify collision and joint count for planning -->
-    <!-- xacro:roller blocks intentionally omitted -->
+    <xacro:roller prefix="${prefix}" num="1">
+      <origin xyz="0.0577 0.012 0.0" rpy="0.0 -0.0 0.0"/>
+      <axis xyz="0.0 0.0 1.0"/>
+    </xacro:roller>
+    <xacro:roller prefix="${prefix}" num="2">
+      <origin xyz="0.05 0.012 0.0289" rpy="0.0 -0.5236 0.0"/>
+      <axis xyz="0.0 0.0 1.0"/>
+    </xacro:roller>
+    <xacro:roller prefix="${prefix}" num="3">
+      <origin xyz="0.0289 0.012 0.05" rpy="0.0 -1.0472 0.0"/>
+      <axis xyz="0.0 0.0 1.0"/>
+    </xacro:roller>
+    <xacro:roller prefix="${prefix}" num="4">
+      <origin xyz="0.0 0.012 0.0577" rpy="0.0 -1.5708 0.0"/>
+      <axis xyz="0.0 0.0 1.0"/>
+    </xacro:roller>
+    <xacro:roller prefix="${prefix}" num="5">
+      <origin xyz="-0.0289 0.012 0.05" rpy="0.0 -2.0944 0.0"/>
+      <axis xyz="0.0 0.0 1.0"/>
+    </xacro:roller>
+    <xacro:roller prefix="${prefix}" num="6">
+      <origin xyz="-0.05 0.012 0.0289" rpy="0.0 -2.618 0.0"/>
+      <axis xyz="0.0 0.0 1.0"/>
+    </xacro:roller>
     <xacro:roller prefix="${prefix}" num="7">
       <origin xyz="-0.0577 0.012 0.0" rpy="0.0 -3.1416 0.0"/>
