Commit message: feat: add use_zed args in servo_head xacro for non-zed sdk env
utils use_zed args for enable user without nvidia or zed-sdk to be able
to use this description. also add gazebo sensors for this too (high
performance impact)

File: robots/gz_walkie_1arm.urdf.xacro (robot description, xacro)
@@ -1,61 +1,64 @@
 <?xml version="1.0"?>
 <robot xmlns:xacro="http://www.ros.org/wiki/xacro" name="walkie_bot">
-  <xacro:property name="M_PI" value="3.14159274"/>
-  <xacro:arg name="ros2_control" default="gazebo"/>
-  <xacro:arg name="use_gripper" default="true"/>
-  <xacro:arg name="ros2_control_hardware_type" default="mock_components"/>
-  <xacro:arg name="hardware_config_file" default="$(find walkie_description)/config/hardware_layout.yaml"/>
+  <xacro:property name="M_PI" value="3.14159274" />
+  <xacro:arg name="ros2_control" default="gazebo" />
+  <xacro:arg name="use_gripper" default="true" />
+  <xacro:arg name="ros2_control_hardware_type" default="mock_components" />
+  <xacro:arg name="hardware_config_file"
+    default="$(find walkie_description)/config/hardware_layout.yaml" />
   <!-- Dual lidar option when only SIMULATION
   real robot force to be dual_lidar
   don't forgot to enable lidar topic to bridge in gz_bridge.yml -->
-  <xacro:arg name="dual_lidar" default="True"/>
-  <xacro:include filename="$(find walkie_description)/urdf/walkie/base/base.urdf.xacro"/>
-  <xacro:include filename="$(find walkie_description)/urdf/walkie/omni_wheel/gz_omni_wheel.urdf.xacro"/>
-  <xacro:include filename="$(find walkie_description)/urdf/walkie/lidar/lidar_gz.urdf.xacro"/>
-  <xacro:include filename="$(find walkie_description)/urdf/walkie/imu/imu_gz.urdf.xacro"/>
-  <xacro:include filename="$(find walkie_description)/urdf/walkie/depth_camera/d415.urdf.xacro"/>
-  <xacro:include filename="$(find walkie_description)/urdf/walkie/head/servo_camera.urdf.xacro"/>
+  <xacro:arg name="dual_lidar" default="True" />
+  <xacro:arg name="use_zed" default="false" />
+  <xacro:include filename="$(find walkie_description)/urdf/walkie/base/base.urdf.xacro" />
+  <xacro:include
+    filename="$(find walkie_description)/urdf/walkie/omni_wheel/gz_omni_wheel.urdf.xacro" />
+  <xacro:include filename="$(find walkie_description)/urdf/walkie/lidar/lidar_gz.urdf.xacro" />
+  <xacro:include filename="$(find walkie_description)/urdf/walkie/imu/imu_gz.urdf.xacro" />
+  <xacro:include filename="$(find walkie_description)/urdf/walkie/depth_camera/d415.urdf.xacro" />
+  <xacro:include filename="$(find walkie_description)/urdf/walkie/head/servo_camera.urdf.xacro" />
   <!-- Include the arm and gripper macros -->
-  <xacro:include filename="$(find walkie_description)/urdf/walkie-arm/walkie_arm.urdf.xacro"/>
-  <xacro:include filename="$(find walkie_description)/urdf/walkie-gripper/walkie_gripper.urdf.xacro"/>
-  <xacro:include filename="$(find walkie_description)/urdf/walkie-arm/arm_ros2_control.xacro"/>
+  <xacro:include filename="$(find walkie_description)/urdf/walkie-arm/walkie_arm.urdf.xacro" />
+  <xacro:include filename="$(find walkie_description)/urdf/walkie-gripper/walkie_gripper.urdf.xacro" />
+  <xacro:include filename="$(find walkie_description)/urdf/walkie-arm/arm_ros2_control.xacro" />
   <!-- =============== Link & Joint =============== -->
   <!-- Base -->
-  <link name="base_footprint"/>
+  <link name="base_footprint" />
   <xacro:base_v0 parent="base_footprint">
-    <origin xyz="0 0 0" rpy="0 0 ${M_PI / 2}"/>
+    <origin xyz="0 0 0" rpy="0 0 ${M_PI / 2}" />
   </xacro:base_v0>
-  <xacro:base_gazebo_v0/>
+  <xacro:base_gazebo_v0 />
   <!-- Wheel -->
   <!-- 1st wheel -->
   <xacro:wheel_v0 prefix="bl" parent="base_link">
-    <origin xyz="0.145261 0.145261 0.05" rpy="0 0 -${M_PI/4}"/>
-    <axis xyz="0.0 1.0 0.0"/>
+    <origin xyz="0.145261 0.145261 0.05" rpy="0 0 -${M_PI/4}" />
+    <axis xyz="0.0 1.0 0.0" />
   </xacro:wheel_v0>
   <!-- 2nd wheel -->
   <xacro:wheel_v0 prefix="br" parent="base_link">
-    <origin xyz="-0.145261 0.145261 0.05" rpy="0 0 ${M_PI/4}"/>
-    <axis xyz="0.0 1.0 0.0"/>
+    <origin xyz="-0.145261 0.145261 0.05" rpy="0 0 ${M_PI/4}" />
+    <axis xyz="0.0 1.0 0.0" />
   </xacro:wheel_v0>
   <!-- 3rd wheel -->
   <xacro:wheel_v0 prefix="fr" parent="base_link">
-    <origin xyz="-0.145261 -0.145261 0.05" rpy="0 0 ${3*M_PI/4}"/>
-    <axis xyz="0.0 1.0 0.0"/>
+    <origin xyz="-0.145261 -0.145261 0.05" rpy="0 0 ${3*M_PI/4}" />
+    <axis xyz="0.0 1.0 0.0" />
   </xacro:wheel_v0>
   <!-- 4th wheel -->
   <xacro:wheel_v0 prefix="fl" parent="base_link">
-    <origin xyz="0.145261 -0.145261 0.05" rpy="0 0 ${5*M_PI/4}"/>
-    <axis xyz="0.0 1.0 0.0"/>
+    <origin xyz="0.145261 -0.145261 0.05" rpy="0 0 ${5*M_PI/4}" />
+    <axis xyz="0.0 1.0 0.0" />
   </xacro:wheel_v0>
   <!-- Left arm mount joint -->
   <joint name="left_arm_mount_joint" type="fixed">
-    <parent link="base_link"/>
-    <child link="left_arm_base"/>
-    <origin xyz="0.075 0 0.951268" rpy="0 0 0"/>
+    <parent link="base_link" />
+    <child link="left_arm_base" />
+    <origin xyz="0.075 0 0.951268" rpy="0 0 0" />
   </joint>
   <!-- Left arm -->
-  <xacro:walkie_arm base_link="left_arm_base" prefix="left"/>
+  <xacro:walkie_arm base_link="left_arm_base" prefix="left" />
   <xacro:if value="$(arg use_gripper)">
-    <xacro:walkie_gripper parent="left_link6" prefix="left"/>
+    <xacro:walkie_gripper parent="left_link6" prefix="left" />
   </xacro:if>
   <xacro:if value="$(arg use_gripper)">
@@ -63,24 +66,24 @@
       <visual>
         <geometry>
-          <sphere radius="0.01"/>
+          <sphere radius="0.01" />
         </geometry>
         <material name="red">
-          <color rgba="1 0 0 1"/>
+          <color rgba="1 0 0 1" />
         </material>
       </visual>
       <collision>
         <geometry>
-          <sphere radius="0.01"/>
+          <sphere radius="0.01" />
         </geometry>
       </collision>
       <inertial>
-        <mass value="0.001"/>
-        <inertia ixx="1e-6" ixy="0" ixz="0" iyy="1e-6" iyz="0" izz="1e-6"/>
+        <mass value="0.001" />
+        <inertia ixx="1e-6" ixy="0" ixz="0" iyy="1e-6" iyz="0" izz="1e-6" />
       </inertial>
     </link>
     <joint name="left_gripper_center_joint" type="fixed">
-      <parent link="left_link7"/>
-      <child link="left_gripper_center"/>
-      <origin xyz="0.0 0.0 -0.18" rpy="0.0 0.0 0.0"/>
+      <parent link="left_link7" />
+      <child link="left_gripper_center" />
+      <origin xyz="0.0 0.0 -0.18" rpy="0.0 0.0 0.0" />
     </joint>
   </xacro:if>
@@ -89,40 +92,47 @@
   <xacro:if value="${'$(arg ros2_control)' == 'gazebo' and not $(arg dual_lidar)}">
     <xacro:lidar_v0 prefix="single" parent="base_link">
-      <origin xyz="0 0 0.315" rpy="0 0 -1.5707963"/>
+      <origin xyz="0 0 0.315" rpy="0 0 -1.5707963" />
     </xacro:lidar_v0>
-    <xacro:lidar_gazebo_v0 prefix="single" min_rad="-${M_PI}" max_rad=" ${M_PI}" min_range="0.6" max_range="10" yaw_offset="0"/>
+    <xacro:lidar_gazebo_v0 prefix="single" min_rad="-${M_PI}" max_rad=" ${M_PI}" min_range="0.6"
+      max_range="10" yaw_offset="0" />
   </xacro:if>
-  <!-- dual lidar when ** REAL WORLD ** or ** SIMULATION ** but set argument ** DUAL_LIDAR ** to true -->
+  <!-- dual lidar when ** REAL WORLD ** or ** SIMULATION **
+  set argument ** DUAL_LIDAR ** to true -->
   <xacro:unless value="${'$(arg ros2_control)' == 'gazebo' and not $(arg dual_lidar)}">
     <xacro:lidar_v0 prefix="front" parent="base_link">
-      <origin xyz="0 -0.240 0.28232" rpy="0 0 -1.5707963"/>
+      <origin xyz="0 -0.240 0.28232" rpy="0 0 -1.5707963" />
     </xacro:lidar_v0>
     <xacro:lidar_v0 prefix="back" parent="base_link">
-      <origin xyz="0 0.240 0.28232" rpy="0 0 1.5707963"/>
+      <origin xyz="0 0.240 0.28232" rpy="0 0 1.5707963" />
     </xacro:lidar_v0>
-    <xacro:lidar_gazebo_v0 prefix="front" min_rad="-2.09333333" max_rad=" 2.09333333" min_range="0.18" max_range="10" yaw_offset="0"/>
-    <xacro:lidar_gazebo_v0 prefix="back" min_rad="-2.09333333" max_rad=" 2.09333333" min_range="0.18" max_range="10" yaw_offset="0"/>
+    <xacro:lidar_gazebo_v0 prefix="front" min_rad="-2.09333333" max_rad=" 2.09333333"
+      min_range="0.18" max_range="10" yaw_offset="0" />
+    <xacro:lidar_gazebo_v0 prefix="back" min_rad="-2.09333333" max_rad=" 2.09333333"
+      min_range="0.18" max_range="10" yaw_offset="0" />
   </xacro:unless>
   <!-- depth cam sensor -->
   <!-- d415 -->
-  <xacro:sensor_d415 name="bottom" parent="base_link" flag_color="1" flag_ir="0" flag_depth="1" updaterate="2">
-    <origin xyz="0 -0.282713 0.1775" rpy="0 -0.453786 -${M_PI/2}"/>
+  <xacro:sensor_d415 name="bottom" parent="base_link" flag_color="1" flag_ir="0" flag_depth="0"
+    updaterate="2">
+    <origin xyz="0 -0.282713 0.1775" rpy="0 -0.453786 -${M_PI/2}" />
   </xacro:sensor_d415>
-  <link name="bottombase"/>
+  <link name="bottombase" />
   <joint name="bottombase_joint" type="fixed">
-    <parent link="base_link"/>
-    <child link="bottombase"/>
-    <origin xyz="0 -0.282713 0.1775" rpy="0 0 -${M_PI/2}"/>
+    <parent link="base_link" />
+    <child link="bottombase" />
+    <origin xyz="0 -0.282713 0.1775" rpy="0 0 -${M_PI/2}" />
   </joint>
   <xacro:servo_v0 prefix="head" parent="base_link">
-    <origin xyz="-0.098 -0.1195 0.848" rpy="0 0 0"/>
+    <origin xyz="-0.098 -0.1195 0.848" rpy="0 0 0" />
   </xacro:servo_v0>
   <!-- imu sensor -->
   <xacro:imu_v0 prefix="top" parent="base_link">
-    <origin xyz="0 0 0.17"/>
+    <origin xyz="0 0 0.17" />
   </xacro:imu_v0>
-  <xacro:imu_gazebo_v0 prefix="top"/>
-  <xacro:include filename="$(find walkie_description)/urdf/walkie/ros2_control.xacro"/>
-  <xacro:ros2_control ros2_control="$(arg ros2_control)"/>
-  <xacro:arm_ros2_control name="LeftWalkieSystem" prefix="left" hardware_type="$(arg ros2_control_hardware_type)" hardware_config_file="$(arg hardware_config_file)"/>
+  <xacro:imu_gazebo_v0 prefix="top" />
+  <xacro:include filename="$(find walkie_description)/urdf/walkie/ros2_control.xacro" />
+  <xacro:ros2_control ros2_control="$(arg ros2_control)" />
+  <xacro:arm_ros2_control name="LeftWalkieSystem" prefix="left"
+    hardware_type="$(arg ros2_control_hardware_type)"
+    hardware_config_file="$(arg hardware_config_file)" />
 </robot>

File: urdf/walkie/head/servo_camera.urdf.xacro (robot description, xacro)
@@ -1,9 +1,14 @@
 <?xml version="1.0"?>
 <robot xmlns:xacro="http://ros.org/wiki/xacro">
-  <xacro:include filename="$(find zed_wrapper)/urdf/zed_macro.urdf.xacro" />
+  <!-- Conditionally include zed_wrapper URDF only when use_zed is true (SDK mode) -->
+  <xacro:arg name="use_zed" default="false" />
+  <xacro:if value="$(arg use_zed)">
+    <xacro:include filename="$(find zed_wrapper)/urdf/zed_macro.urdf.xacro" />
+  </xacro:if>
   <xacro:macro name="servo_v0" params="prefix parent *joint_origin">
-    <xacro:arg name="camera_name" default="zed_${prefix}"/>
+    <xacro:arg name="camera_name" default="zed_${prefix}" />
     <xacro:arg name="camera_model" default="zed2i" />
     <xacro:arg name="use_zed_localization" default="false" />
+    <!-- ============ Servo Mount ============ -->
     <joint name="${prefix}_servobase_joint" type="fixed">
       <xacro:insert_block name="joint_origin" />
@@ -22,5 +27,10 @@
         </material>
       </visual>
+      <inertial>
+        <mass value="0.05" />
+        <inertia ixx="1e-5" ixy="0" ixz="0" iyy="1e-5" iyz="0" izz="1e-5" />
+      </inertial>
     </link>
+    <!-- ============ Servo Joint (tilt) ============ -->
     <joint name="${prefix}_servo_joint" type="revolute">
       <parent link="${prefix}_servobase_link" />
@@ -44,27 +54,133 @@
         </geometry>
       </collision>
+      <inertial>
+        <mass value="0.2" />
+        <inertia ixx="1e-4" ixy="0" ixz="0" iyy="1e-4" iyz="0" izz="1e-4" />
+      </inertial>
     </link>
-    <xacro:zed_camera name="zed" model="$(arg camera_model)">
-      <!-- <gnss_origin /> -->
-       <origin xyz="0 0 0" rpy="0 0 0" />
-    </xacro:zed_camera>
-    <!-- <xacro:zed_camera name="zed" model="zed2i">
-      <origin xyz="0 0 0" rpy="0 0 0"/>
-    </xacro:zed_camera> -->
-    <!-- Zed Camera Mounting Joint -->
-    <!-- <joint name="${prefix}_zed_mounting_joint" type="fixed">
-      <parent link="${prefix}_servo_link" />
-      <child link="zed_camera_link" />
-      <origin xyz="0.098 -0.02 0" rpy="0 0 -1.5708" />
-    </joint> -->
+    <!-- ============ ZED Camera Body ============ -->
+    <!-- SDK mode: use zed_wrapper macro -->
+    <xacro:if value="$(arg use_zed)">
+      <xacro:zed_camera name="zed" model="$(arg camera_model)">
+        <origin xyz="0 0 0" rpy="0 0 0" />
+      </xacro:zed_camera>
+    </xacro:if>
+    <!-- No-wrapper mode: define standalone camera links -->
+    <xacro:unless value="$(arg use_zed)">
+      <!-- Camera mount frame -->
+      <link name="$(arg camera_name)_camera_mount_link" />
+      <joint name="$(arg camera_name)_mount_joint" type="fixed">
+        <parent link="$(arg camera_name)_camera_mount_link" />
+        <child link="$(arg camera_name)_camera_link" />
+        <origin xyz="0 0 0.015" rpy="0 0 0" />
+      </joint>
+      <!-- Camera body link -->
+      <link name="$(arg camera_name)_camera_link">
+        <visual>
+          <origin xyz="0 0 0" rpy="0 0 0" />
+          <geometry>
+            <box size="0.030 0.16 0.033" />
+          </geometry>
+          <material name="zed_dark">
+            <color rgba="0.15 0.15 0.15 1" />
+          </material>
+        </visual>
+        <collision>
+          <geometry>
+            <box size="0.175 0.030 0.033" />
+          </geometry>
+        </collision>
+        <inertial>
+          <mass value="0.16" />
+          <origin xyz="0 0 0" />
+          <inertia ixx="1e-4" ixy="0" ixz="0" iyy="1e-4" iyz="0" izz="1e-4" />
+        </inertial>
+      </link>
+      <!-- Left camera frame (baseline origin) -->
+      <link name="$(arg camera_name)_left_camera_frame" />
+      <joint name="$(arg camera_name)_left_camera_joint" type="fixed">
+        <parent link="$(arg camera_name)_camera_link" />
+        <child link="$(arg camera_name)_left_camera_frame" />
+        <origin xyz="0 0.06 0" rpy="0 0 0" />
+      </joint>
+      <!-- Left camera optical frame -->
+      <link name="$(arg camera_name)_left_camera_optical_frame" />
+      <joint name="$(arg camera_name)_left_camera_optical_joint" type="fixed">
+        <parent link="$(arg camera_name)_left_camera_frame" />
+        <child link="$(arg camera_name)_left_camera_optical_frame" />
+        <origin xyz="0 0 0" rpy="0 0 0" />
+      </joint>
+      <!-- Right camera frame -->
+      <link name="$(arg camera_name)_right_camera_frame" />
+      <joint name="$(arg camera_name)_right_camera_joint" type="fixed">
+        <parent link="$(arg camera_name)_camera_link" />
+        <child link="$(arg camera_name)_right_camera_frame" />
+        <origin xyz="0 -0.06 0" rpy="0 0 0" />
+      </joint>
+      <!-- Right camera optical frame -->
+      <link name="$(arg camera_name)_right_camera_optical_frame" />
+      <joint name="$(arg camera_name)_right_camera_optical_joint" type="fixed">
+        <parent link="$(arg camera_name)_right_camera_frame" />
+        <child link="$(arg camera_name)_right_camera_optical_frame" />
+        <origin xyz="0 0 0" rpy="0 0 0" />
+      </joint>
+      <!-- Depth frame (co-located with left camera) -->
+      <link name="$(arg camera_name)_depth_frame" />
+      <joint name="$(arg camera_name)_depth_joint" type="fixed">
+        <parent link="$(arg camera_name)_left_camera_frame" />
+        <child link="$(arg camera_name)_depth_frame" />
+        <origin xyz="0 0 0" rpy="0 0 0" />
+      </joint>
+      <!-- ============ Gazebo Sensors (Gz Sim / Jazzy) ============ -->
+      <gazebo reference="$(arg camera_name)_camera_link">
+        <!-- Left RGB Camera -->
+        <sensor name="${prefix}_left_rgb_sensor" type="camera">
+          <pose relative_to="$(arg camera_name)_left_camera_optical_frame">0 0 0 0 0 0</pose>
+          <camera name="${prefix}_left">
+            <horizontal_fov>1.9199</horizontal_fov> <!-- ZED2i: 110 deg -->
+            <image>
+              <width>960</width>
+              <height>540</height>
+              <format>RGB_INT8</format>
+            </image> --> </camera>
+          <always_on>1</always_on>
+          <update_rate>15</update_rate>
+          <visualize>true</visualize>
+          <topic>${prefix}/rgb/image</topic>
+          <gz_frame_id>$(arg camera_name)_left_camera_optical_frame</gz_frame_id>
+        </sensor>
+        <!-- Depth Camera -->
+        <sensor name="${prefix}_depth_sensor" type="depth_camera">
+          <pose relative_to="$(arg camera_name)_left_camera_optical_frame">0 0 0 0 0 0</pose>
+          <camera name="${prefix}_depth">
+            <horizontal_fov>1.9199</horizontal_fov> <!-- ZED2i: 110 deg -->
+            <image>
+              <width>960</width>
+              <height>540</height>
+            </image>
+            <clip>
+              <near>0.3</near>
+              <far>20</far>
+            </clip>
+            <noise>
+              <type>gaussian</type>
+              <mean>0.0</mean>
+              <stddev>0.01</stddev>
+            </noise>
+          </camera>
+          <always_on>1</always_on>
+          <update_rate>5</update_rate>
+          <visualize>false</visualize>
+          <topic>${prefix}/depth</topic>
+          <gz_frame_id>$(arg camera_name)_left_camera_optical_frame</gz_frame_id>
+        </sensor>
+      </gazebo>
+    </xacro:unless>
+    <!-- ============ Camera Mounting Joint ============ -->
     <xacro:if value="$(arg use_zed_localization)">
       <joint name="$(arg camera_name)_joint" type="fixed">
-        <parent link="$(arg camera_name)_camera_link" />
+        <parent link="$(arg camera_name)_camera_mount_link" />
         <child link="${prefix}_servo_link" />
         <origin xyz="0.098 -0.02 -0.015" rpy="0 0 -1.5708" />
-        <!-- <origin
-          xyz="-0.12 0.0 -0.25"
-          rpy="0 0 0"
-        /> -->
       </joint>
     </xacro:if>
@@ -72,5 +188,5 @@
       <joint name="$(arg camera_name)_joint" type="fixed">
         <parent link="${prefix}_servo_link" />
-        <child link="zed_camera_link" />
+        <child link="$(arg camera_name)_camera_mount_link" />
         <origin xyz="0.098 -0.006 -0.015" rpy="0 0 -1.5708" />
       </joint>

File: urdf/walkie/ros2_control.xacro (robot description, xacro)
@@ -1,3 +1,3 @@
-<?xml version="1.0" ?>
+<?xml version="1.0"?>
 <robot xmlns:xacro="http://www.ros.org/wiki/xacro">
   <xacro:macro name="ros2_control" params="ros2_control">
@@ -38,4 +38,11 @@
           </command_interface>
           <state_interface name="velocity" />
+          <state_interface name="position" />
+        </joint>
+        <joint name="head_servo_joint">
+          <command_interface name="position">
+            <param name="min"> -1.54</param>
+            <param name="max"> 1.54</param>
+          </command_interface>
           <state_interface name="position" />
         </joint>
@@ -186,6 +193,5 @@
         filename="libgz_ros2_control-system.so"
       >
-        <parameters
-        >$(find walkie_description)/config/ros2_controller/sim_controllers.yaml</parameters>
+        <parameters>$(find walkie_description)/config/ros2_controller/sim_controllers.yaml</parameters>
       </plugin>
     </gazebo>
