Commit message: change to real robot calibrated params

File: robots/gz_walkie.urdf.xacro (robot description, xacro)
@@ -37,8 +37,12 @@
   </xacro:wheel_v0>
   <!-- lidar sensor -->
-  <xacro:lidar_v0 prefix="top" parent="base_link">
-    <origin xyz="0 -0.19 0.315"/>
+  <xacro:lidar_v0 prefix="front" parent="base_link">
+    <origin xyz="0 -0.19 0.315" rpy="0 0 -1.5707963"/>
+  </xacro:lidar_v0>
+  <xacro:lidar_v0 prefix="back" parent="base_link">
+    <origin xyz="0 0.19 0.315" rpy="0 0 1.5707963"/>
   </xacro:lidar_v0>
   <xacro:lidar_gazebo_v0 prefix="top" min_rad="-3.925" max_rad="0.785" min_range="0.18" max_range="10"/>
+  <xacro:lidar_gazebo_v0 prefix="back" min_rad="-3.925" max_rad="0.785" min_range="0.18" max_range="10"/>
   <!-- depth cam sensor -->
   <xacro:sensor_d415 name="bottom" parent="base_link" flag_color="1" flag_ir="0" flag_depth="1" updaterate="2">

File: urdf/walkie/ros2_control.xacro (robot description, xacro)
@@ -89,5 +89,5 @@
         </hardware>
         <joint name="fl_wheel_joint">
-          <param name="can_id">1</param>
+          <param name="can_id">3</param>
           <param name="pole_pairs">14</param>
           <param name="gear_ratio">10</param>
@@ -95,7 +95,5 @@
           <param name="enc_off">0.0</param>
           <param name="trq_limit">30</param>
-          <xacro:if value="${read_only}">
-            <param name="read_only">1</param>
-          </xacro:if>
+          <param name="read_only">0</param>
           <command_interface name="position" />
           <command_interface name="velocity">
@@ -111,5 +109,5 @@
         </joint>
         <joint name="fr_wheel_joint">
-          <param name="can_id">2</param>
+          <param name="can_id">1</param>
           <param name="pole_pairs">14</param>
           <param name="gear_ratio">10</param>
@@ -117,7 +115,5 @@
           <param name="enc_off">0.0</param>
           <param name="trq_limit">30</param>
-          <xacro:if value="${read_only}">
-            <param name="read_only">1</param>
-          </xacro:if>
+          <param name="read_only">0</param>
           <command_interface name="position" />
           <command_interface name="velocity">
@@ -133,5 +129,5 @@
         </joint>
         <joint name="br_wheel_joint">
-          <param name="can_id">3</param>
+          <param name="can_id">4</param>
           <param name="pole_pairs">14</param>
           <param name="gear_ratio">10</param>
@@ -139,7 +135,5 @@
           <param name="enc_off">0.0</param>
           <param name="trq_limit">30</param>
-          <xacro:if value="${read_only}">
-            <param name="read_only">1</param>
-          </xacro:if>
+          <param name="read_only">0</param>
           <command_interface name="position" />
           <command_interface name="velocity">
@@ -155,5 +149,5 @@
         </joint>
         <joint name="bl_wheel_joint">
-          <param name="can_id">4</param>
+          <param name="can_id">2</param>
           <param name="pole_pairs">14</param>
           <param name="gear_ratio">10</param>
@@ -161,7 +155,5 @@
           <param name="enc_off">0.0</param>
           <param name="trq_limit">30</param>
-          <xacro:if value="${read_only}">
-            <param name="read_only">1</param>
-          </xacro:if>
+          <param name="read_only">0</param>
           <command_interface name="position" />
           <command_interface name="velocity">

Commit message: adjust lidar position

File: robots/gz_walkie.urdf.xacro (robot description, xacro)
@@ -38,8 +38,8 @@
   <!-- lidar sensor -->
   <xacro:lidar_v0 prefix="front" parent="base_link">
-    <origin xyz="0 -0.19 0.315" rpy="0 0 -1.5707963"/>
+    <origin xyz="0 -0.240 0.315" rpy="0 0 -1.5707963"/>
   </xacro:lidar_v0>
   <xacro:lidar_v0 prefix="back" parent="base_link">
-    <origin xyz="0 0.19 0.315" rpy="0 0 1.5707963"/>
+    <origin xyz="0 0.240 0.315" rpy="0 0 1.5707963"/>
   </xacro:lidar_v0>
   <xacro:lidar_gazebo_v0 prefix="top" min_rad="-3.925" max_rad="0.785" min_range="0.18" max_range="10"/>

Commit message: add camerabase for human_detection

File: robots/gz_walkie.urdf.xacro (robot description, xacro)
@@ -50,4 +50,10 @@
     <origin xyz="0 -0.23813 0.18161" rpy="0 -0.5564807787058716 -${M_PI/2}"/>
   </xacro:sensor_d415>
+  <link name="bottombase"/>
+  <joint name="bottombase_joint" type="fixed">
+      <parent link="base_link"/>
+      <child link="bottombase"/>
+      <origin xyz="0 -0.23813 0.18161" rpy="0 0 -${M_PI/2}"/>
+  </joint>
   <!-- imu sensor -->
   <xacro:imu_v0 prefix="top" parent="base_link">

Commit message: feat: add dual_lidar optional for simulation (default: single lidar)

File: robots/gz_walkie.urdf.xacro (robot description, xacro)
@@ -1,65 +1,122 @@
-<?xml version="1.0"?>
+<?xml version="1.0" ?>
 <robot xmlns:xacro="http://ros.org/wiki/xacro" name="walkie_bot">
-  <xacro:property name="M_PI" value="3.14159274"/>
-  <xacro:arg name="ros2_control" default="gazebo"/>
-  <xacro:include filename="$(find walkie_description)/urdf/walkie/base/base.urdf.xacro"/>
-  <xacro:include filename="$(find walkie_description)/urdf/walkie/omni_wheel/gz_omni_wheel.urdf.xacro"/>
-  <xacro:include filename="$(find walkie_description)/urdf/walkie/lidar/lidar_gz.urdf.xacro"/>
-  <xacro:include filename="$(find walkie_description)/urdf/walkie/imu/imu_gz.urdf.xacro"/>
-  <xacro:include filename="$(find walkie_description)/urdf/walkie/depth_camera/d415.urdf.xacro"/>
+  <xacro:property name="M_PI" value="3.14159274" />
+  <xacro:arg name="ros2_control" default="gazebo" />
+  <!-- Dual lidar option when only SIMULATION
+  real robot force to be dual_lidar
+  don't forgot to enable lidar topic to bridge in gz_bridge.yml -->
+  <xacro:arg name="dual_lidar" default="False" />
+  <xacro:include
+    filename="$(find walkie_description)/urdf/walkie/base/base.urdf.xacro"
+  />
+  <xacro:include
+    filename="$(find walkie_description)/urdf/walkie/omni_wheel/gz_omni_wheel.urdf.xacro"
+  />
+  <xacro:include
+    filename="$(find walkie_description)/urdf/walkie/lidar/lidar_gz.urdf.xacro"
+  />
+  <xacro:include
+    filename="$(find walkie_description)/urdf/walkie/imu/imu_gz.urdf.xacro"
+  />
+  <xacro:include
+    filename="$(find walkie_description)/urdf/walkie/depth_camera/d415.urdf.xacro"
+  />
   <!-- =============== Link & Joint =============== -->
   <!-- Base -->
-  <link name="base_footprint"/>
+  <link name="base_footprint" />
   <xacro:base_v0 parent="base_footprint">
-    <origin xyz="0 0 0" rpy="0 0 ${M_PI / 2}"/>
+    <origin xyz="0 0 0" rpy="0 0 ${M_PI / 2}" />
   </xacro:base_v0>
-  <xacro:base_gazebo_v0/>
+  <xacro:base_gazebo_v0 />
   <!-- Wheel -->
   <!-- 1st wheel -->
   <xacro:wheel_v0 prefix="bl" parent="base_link">
-    <origin xyz="0.177622395 0.177622395 0.05" rpy="0 0 -${M_PI/4}"/>
-    <axis xyz="0.0 1.0 0.0"/>
+    <origin xyz="0.177622395 0.177622395 0.05" rpy="0 0 -${M_PI/4}" />
+    <axis xyz="0.0 1.0 0.0" />
   </xacro:wheel_v0>
   <!-- 2nd wheel -->
   <xacro:wheel_v0 prefix="br" parent="base_link">
-    <origin xyz="-0.177622395 0.177622395 0.05" rpy="0 0 ${M_PI/4}"/>
-    <axis xyz="0.0 1.0 0.0"/>
+    <origin xyz="-0.177622395 0.177622395 0.05" rpy="0 0 ${M_PI/4}" />
+    <axis xyz="0.0 1.0 0.0" />
   </xacro:wheel_v0>
   <!-- 3rd wheel -->
   <xacro:wheel_v0 prefix="fr" parent="base_link">
-    <origin xyz="-0.177622395 -0.177622395 0.05" rpy="0 0 ${3*M_PI/4}"/>
-    <axis xyz="0.0 1.0 0.0"/>
+    <origin xyz="-0.177622395 -0.177622395 0.05" rpy="0 0 ${3*M_PI/4}" />
+    <axis xyz="0.0 1.0 0.0" />
   </xacro:wheel_v0>
   <!-- 4th wheel -->
   <xacro:wheel_v0 prefix="fl" parent="base_link">
-    <origin xyz="0.177622395 -0.177622395 0.05" rpy="0 0 ${5*M_PI/4}"/>
-    <axis xyz="0.0 1.0 0.0"/>
+    <origin xyz="0.177622395 -0.177622395 0.05" rpy="0 0 ${5*M_PI/4}" />
+    <axis xyz="0.0 1.0 0.0" />
   </xacro:wheel_v0>
   <!-- lidar sensor -->
+  <!-- single lidar for simulation performance -->
+  <xacro:if
+    value="${'$(arg ros2_control)' == 'gazebo' and not $(arg dual_lidar)}"
+  >
+    <xacro:lidar_v0 prefix="single" parent="base_link">
+      <origin xyz="0 0 0.315" rpy="0 0 -1.5707963" />
+    </xacro:lidar_v0>
+    <xacro:lidar_gazebo_v0
+      prefix="single"
+      min_rad="-${M_PI}"
+      max_rad=" ${M_PI}"
+      min_range="0.2"
+      max_range="10"
+      yaw_offset="0"
+    />
+  </xacro:if>
+  <!-- dual lidar when ** REAL WORLD ** or ** SIMULATION ** but set argument ** DUAL_LIDAR ** to true -->
+  <xacro:unless
+    value="${'$(arg ros2_control)' == 'gazebo' and not $(arg dual_lidar)}"
+  >
   <xacro:lidar_v0 prefix="front" parent="base_link">
-    <origin xyz="0 -0.240 0.315" rpy="0 0 -1.5707963"/>
-  </xacro:lidar_v0>
-  <xacro:lidar_v0 prefix="back" parent="base_link">
-    <origin xyz="0 0.240 0.315" rpy="0 0 1.5707963"/>
-  </xacro:lidar_v0>
-  <xacro:lidar_gazebo_v0 prefix="top" min_rad="-3.925" max_rad="0.785" min_range="0.18" max_range="10"/>
-  <xacro:lidar_gazebo_v0 prefix="back" min_rad="-3.925" max_rad="0.785" min_range="0.18" max_range="10"/>
+      <origin xyz="0 -0.240 0.315" rpy="0 0 -1.5707963" />
+    </xacro:lidar_v0>
+    <xacro:lidar_v0 prefix="back" parent="base_link">
+      <origin xyz="0 0.240 0.315" rpy="0 0 1.5707963" />
+    </xacro:lidar_v0>
+    <xacro:lidar_gazebo_v0
+      prefix="front"
+      min_rad="-2.09333333"
+      max_rad=" 2.09333333"
+      min_range="0.18"
+      max_range="10"
+      yaw_offset="0"
+    />
+    <xacro:lidar_gazebo_v0
+      prefix="back"
+      min_rad="-2.09333333"
+      max_rad=" 2.09333333"
+      min_range="0.18"
+      max_range="10"
+      yaw_offset="0"
+    />
+  </xacro:unless>
   <!-- depth cam sensor -->
-  <xacro:sensor_d415 name="bottom" parent="base_link" flag_color="1" flag_ir="0" flag_depth="1" updaterate="2">
-    <!-- <origin xyz="0 -0.23813 0.18161" rpy="0 0 -${M_PI/4}"/> -->
-    <origin xyz="0 -0.23813 0.18161" rpy="0 -0.5564807787058716 -${M_PI/2}"/>
+  <xacro:sensor_d415
+    name="bottom"
+    parent="base_link"
+    flag_color="1"
+    flag_ir="0"
+    flag_depth="1"
+    updaterate="2"
+  >
+    <origin xyz="0 -0.23813 0.18161" rpy="0 -0.5564807787058716 -${M_PI/2}" />
   </xacro:sensor_d415>
-  <link name="bottombase"/>
+  <link name="bottombase" />
   <joint name="bottombase_joint" type="fixed">
-      <parent link="base_link"/>
-      <child link="bottombase"/>
-      <origin xyz="0 -0.23813 0.18161" rpy="0 0 -${M_PI/2}"/>
+      <parent link="base_link" />
+      <child link="bottombase" />
+      <origin xyz="0 -0.23813 0.18161" rpy="0 0 -${M_PI/2}" />
   </joint>
   <!-- imu sensor -->
   <xacro:imu_v0 prefix="top" parent="base_link">
-    <origin xyz="0 0 0.17"/>
+    <origin xyz="0 0 0.17" />
   </xacro:imu_v0>
-  <xacro:imu_gazebo_v0 prefix="top"/>
-  <xacro:include filename="$(find walkie_description)/urdf/walkie/ros2_control.xacro"/>
-  <xacro:ros2_control ros2_control="$(arg ros2_control)"/>
+  <xacro:imu_gazebo_v0 prefix="top" />
+  <xacro:include
+    filename="$(find walkie_description)/urdf/walkie/ros2_control.xacro"
+  />
+  <xacro:ros2_control ros2_control="$(arg ros2_control)" />
 </robot>

File: urdf/walkie/lidar/lidar.gz.xacro (robot description, xacro)
@@ -1,9 +1,12 @@
-<?xml version="1.0"?>
+<?xml version="1.0" ?>
 <robot xmlns:xacro="http://ros.org/wiki/xacro">
-	<xacro:macro name="lidar_gazebo_v0" params="prefix min_rad max_rad min_range max_range">
+	<xacro:macro
+        name="lidar_gazebo_v0"
+        params="prefix min_rad max_rad min_range max_range yaw_offset"
+    >
 		<gazebo reference="${prefix}_lidar_link">
-			<sensor name="laser" type="gpu_lidar">
+			<sensor name="${prefix}_lidar" type="gpu_lidar">
 				<visualize>false</visualize>
-				<pose>0 0 0 0 0 0</pose>
+				<pose>0 0 0 0 0 ${yaw_offset}</pose>
 				<update_rate>40</update_rate>
 				<lidar>
@@ -27,5 +30,5 @@
 					</noise>
 				</lidar>
-				<topic>scan</topic>
+				<topic>${prefix}_lidar</topic>
 				<gz_frame_id>${prefix}_lidar_link</gz_frame_id>
 			</sensor>

File: urdf/walkie/ros2_control.xacro (robot description, xacro)
@@ -1,3 +1,3 @@
-<?xml version="1.0"?>
+<?xml version="1.0" ?>
 <robot xmlns:xacro="http://www.ros.org/wiki/xacro">
   <xacro:macro name="ros2_control" params="ros2_control">
@@ -171,7 +171,10 @@
     </xacro:if>
     <gazebo>
-      <plugin name="gz_ros2_control::GazeboSimROS2ControlPlugin"
-        filename="libgz_ros2_control-system.so">
-        <parameters>$(find walkie_description)/config/ros2_controller/my_controllers.yaml</parameters>
+      <plugin
+        name="gz_ros2_control::GazeboSimROS2ControlPlugin"
+        filename="libgz_ros2_control-system.so"
+      >
+        <parameters
+        >$(find walkie_description)/config/ros2_controller/sim_controllers.yaml</parameters>
       </plugin>
     </gazebo>

Commit message: feat: update walkie drivebase mesh file to lastest and add walkie arm to walkie robot urdf file

File: robots/gz_walkie.urdf.xacro (robot description, xacro)
@@ -6,5 +6,5 @@
   real robot force to be dual_lidar
   don't forgot to enable lidar topic to bridge in gz_bridge.yml -->
-  <xacro:arg name="dual_lidar" default="False" />
+  <xacro:arg name="dual_lidar" default="True" />
   <xacro:include
         filename="$(find walkie_description)/urdf/walkie/base/base.urdf.xacro"
@@ -22,4 +22,11 @@
         filename="$(find walkie_description)/urdf/walkie/depth_camera/d415.urdf.xacro"
     />
+  <!-- Include the arm and gripper macros -->
+  <xacro:include
+        filename="$(find walkie_description)/urdf/walkie-arm/walkie_arm.urdf.xacro"
+    />
+  <xacro:include
+        filename="$(find walkie_description)/urdf/walkie-gripper/walkie_gripper.urdf.xacro"
+    />
   <!-- =============== Link & Joint =============== -->
   <!-- Base -->
@@ -32,22 +39,55 @@
   <!-- 1st wheel -->
   <xacro:wheel_v0 prefix="bl" parent="base_link">
-    <origin xyz="0.177622395 0.177622395 0.05" rpy="0 0 -${M_PI/4}" />
+    <origin xyz="0.145261 0.145261 0.05" rpy="0 0 -${M_PI/4}" />
     <axis xyz="0.0 1.0 0.0" />
   </xacro:wheel_v0>
   <!-- 2nd wheel -->
   <xacro:wheel_v0 prefix="br" parent="base_link">
-    <origin xyz="-0.177622395 0.177622395 0.05" rpy="0 0 ${M_PI/4}" />
+    <origin xyz="-0.145261 0.145261 0.05" rpy="0 0 ${M_PI/4}" />
     <axis xyz="0.0 1.0 0.0" />
   </xacro:wheel_v0>
   <!-- 3rd wheel -->
   <xacro:wheel_v0 prefix="fr" parent="base_link">
-    <origin xyz="-0.177622395 -0.177622395 0.05" rpy="0 0 ${3*M_PI/4}" />
+    <origin xyz="-0.145261 -0.145261 0.05" rpy="0 0 ${3*M_PI/4}" />
     <axis xyz="0.0 1.0 0.0" />
   </xacro:wheel_v0>
   <!-- 4th wheel -->
   <xacro:wheel_v0 prefix="fl" parent="base_link">
-    <origin xyz="0.177622395 -0.177622395 0.05" rpy="0 0 ${5*M_PI/4}" />
+    <origin xyz="0.145261 -0.145261 0.05" rpy="0 0 ${5*M_PI/4}" />
     <axis xyz="0.0 1.0 0.0" />
   </xacro:wheel_v0>
+  <!-- Left arm base mount -->
+  <link name="left_arm_base">
+      <!-- <visual>
+        <geometry>
+          <cylinder radius="0.05" length="0.05" />
+        </geometry>
+        <origin xyz="0 0 0.025" rpy="0 0 0" />
+        <material name="mount_material">
+          <color rgba="0.3 0.3 0.3 1.0" />
+        </material>
+      </visual> -->
+  </link>
+  <!-- Left arm mount joint -->
+  <joint name="left_arm_mount_joint" type="fixed">
+    <parent link="base_link" />
+    <child link="left_arm_base" />
+    <origin
+          xyz="0.075 0 0.9018"
+          rpy="0 0 0"
+      />
+  </joint>
+  <!-- Left arm -->
+  <xacro:walkie_arm
+        base_link="arm_base"
+        flange_link="link_flange"
+        prefix="left"
+  >
+    <origin xyz="0 0 0.05" rpy="0 0 0" />
+  </xacro:walkie_arm>
+  <!-- Left gripper (optional) -->
+  <xacro:walkie_gripper parent="link_flange" prefix="left">
+      <origin xyz="0 0 0" rpy="3.141592653589793 0 0" />
+  </xacro:walkie_gripper>
   <!-- lidar sensor -->
   <!-- single lidar for simulation performance -->

File: urdf/walkie/base/base.urdf.xacro (robot description, xacro)
@@ -17,5 +17,5 @@
         <geometry>
           <!-- <mesh filename="package://walkie_description/meshes/walkie/base_link.dae"/> -->
-          <mesh filename="package://walkie_description/meshes/walkie/base_link.stl" scale="0.001 0.001 0.001"/>
+          <mesh filename="package://walkie_description/meshes/walkie/base_link2.stl" scale="0.001 0.001 0.001"/>
         </geometry>
         <material name="grey"/>

Commit message: feat: add robot collision and fix robot transform

File: robots/gz_walkie.urdf.xacro (robot description, xacro)
@@ -112,8 +112,8 @@
     >
   <xacro:lidar_v0 prefix="front" parent="base_link">
-      <origin xyz="0 -0.240 0.315" rpy="0 0 -1.5707963" />
+      <origin xyz="0 -0.240 0.28232" rpy="0 0 -1.5707963" />
     </xacro:lidar_v0>
     <xacro:lidar_v0 prefix="back" parent="base_link">
-      <origin xyz="0 0.240 0.315" rpy="0 0 1.5707963" />
+      <origin xyz="0 0.240 0.28232" rpy="0 0 1.5707963" />
     </xacro:lidar_v0>
     <xacro:lidar_gazebo_v0
@@ -143,5 +143,5 @@
         updaterate="2"
     >
-    <origin xyz="0 -0.23813 0.18161" rpy="0 -0.5564807787058716 -${M_PI/2}" />
+    <origin xyz="0 -0.282713 0.1775" rpy="0 -0.453786 -${M_PI/2}" />
   </xacro:sensor_d415>
   <link name="bottombase" />
@@ -149,5 +149,5 @@
       <parent link="base_link" />
       <child link="bottombase" />
-      <origin xyz="0 -0.23813 0.18161" rpy="0 0 -${M_PI/2}" />
+      <origin xyz="0 -0.282713 0.1775" rpy="0 0 -${M_PI/2}" />
   </joint>
   <!-- imu sensor -->

File: urdf/walkie/base/base.urdf.xacro (robot description, xacro)
@@ -22,7 +22,15 @@
       </visual>
       <collision>
-        <geometry>
-          <mesh filename="package://walkie_description/meshes/walkie/base_link_collision.stl"/>
-        </geometry>
+        <origin xyz="0 0 0.165" rpy="0 0 0" />
+          <geometry>
+            <cylinder radius="0.3" length="0.33"/>
+          <!-- <mesh filename="package://walkie_description/meshes/walkie/base_link_collision.stl"/> -->
+          </geometry>
+      </collision>
+      <collision>
+        <origin xyz="0 0 0.615" rpy="0 0 0" />
+            <geometry>
+              <box size="0.32 0.2 0.57" />
+            </geometry>
       </collision>
       <xacro:inertial_cylinder mass="${base_mass}" length="${bass_thickness}" radius="${base_radian}">
