Commit message: fix: optimize omni wheel mesh model and add args for sim single lidar launch

File: robots/gz_walkie.urdf.xacro (robot description, xacro)
@@ -8,18 +8,18 @@
   <xacro:arg name="dual_lidar" default="True" />
   <xacro:include
-        filename="$(find walkie_description)/urdf/walkie/base/base.urdf.xacro"
-    />
+    filename="$(find walkie_description)/urdf/walkie/base/base.urdf.xacro"
+  />
   <xacro:include
-        filename="$(find walkie_description)/urdf/walkie/omni_wheel/gz_omni_wheel.urdf.xacro"
-    />
+    filename="$(find walkie_description)/urdf/walkie/omni_wheel/gz_omni_wheel.urdf.xacro"
+  />
   <xacro:include
-        filename="$(find walkie_description)/urdf/walkie/lidar/lidar_gz.urdf.xacro"
-    />
+    filename="$(find walkie_description)/urdf/walkie/lidar/lidar_gz.urdf.xacro"
+  />
   <xacro:include
-        filename="$(find walkie_description)/urdf/walkie/imu/imu_gz.urdf.xacro"
-    />
+    filename="$(find walkie_description)/urdf/walkie/imu/imu_gz.urdf.xacro"
+  />
   <xacro:include
-        filename="$(find walkie_description)/urdf/walkie/depth_camera/d415.urdf.xacro"
-    />
+    filename="$(find walkie_description)/urdf/walkie/depth_camera/d415.urdf.xacro"
+  />
   <!-- =============== Link & Joint =============== -->
   <!-- Base -->
@@ -53,23 +53,23 @@
   <!-- single lidar for simulation performance -->
   <xacro:if
-        value="${'$(arg ros2_control)' == 'gazebo' and not $(arg dual_lidar)}"
-    >
+    value="${'$(arg ros2_control)' == 'gazebo' and not $(arg dual_lidar)}"
+  >
     <xacro:lidar_v0 prefix="single" parent="base_link">
       <origin xyz="0 0 0.315" rpy="0 0 -1.5707963" />
     </xacro:lidar_v0>
     <xacro:lidar_gazebo_v0
-            prefix="single"
-            min_rad="-${M_PI}"
-            max_rad=" ${M_PI}"
-            min_range="0.2"
-            max_range="10"
-            yaw_offset="0"
-        />
+      prefix="single"
+      min_rad="-${M_PI}"
+      max_rad=" ${M_PI}"
+      min_range="0.4"
+      max_range="10"
+      yaw_offset="0"
+    />
   </xacro:if>
   <!-- dual lidar when ** REAL WORLD ** or ** SIMULATION ** but set argument ** DUAL_LIDAR ** to true -->
   <xacro:unless
-        value="${'$(arg ros2_control)' == 'gazebo' and not $(arg dual_lidar)}"
-    >
-  <xacro:lidar_v0 prefix="front" parent="base_link">
+    value="${'$(arg ros2_control)' == 'gazebo' and not $(arg dual_lidar)}"
+  >
+    <xacro:lidar_v0 prefix="front" parent="base_link">
       <origin xyz="0 -0.240 0.28232" rpy="0 0 -1.5707963" />
     </xacro:lidar_v0>
@@ -78,36 +78,36 @@
     </xacro:lidar_v0>
     <xacro:lidar_gazebo_v0
-            prefix="front"
-            min_rad="-2.09333333"
-            max_rad=" 2.09333333"
-            min_range="0.18"
-            max_range="10"
-            yaw_offset="0"
-        />
+      prefix="front"
+      min_rad="-2.09333333"
+      max_rad=" 2.09333333"
+      min_range="0.18"
+      max_range="10"
+      yaw_offset="0"
+    />
     <xacro:lidar_gazebo_v0
-            prefix="back"
-            min_rad="-2.09333333"
-            max_rad=" 2.09333333"
-            min_range="0.18"
-            max_range="10"
-            yaw_offset="0"
-        />
+      prefix="back"
+      min_rad="-2.09333333"
+      max_rad=" 2.09333333"
+      min_range="0.18"
+      max_range="10"
+      yaw_offset="0"
+    />
   </xacro:unless>
   <!-- depth cam sensor -->
   <xacro:sensor_d415
-        name="bottom"
-        parent="base_link"
-        flag_color="1"
-        flag_ir="0"
-        flag_depth="1"
-        updaterate="2"
-    >
+    name="bottom"
+    parent="base_link"
+    flag_color="1"
+    flag_ir="0"
+    flag_depth="1"
+    updaterate="2"
+  >
     <origin xyz="0 -0.282713 0.1775" rpy="0 -0.453786 -${M_PI/2}" />
   </xacro:sensor_d415>
   <link name="bottombase" />
   <joint name="bottombase_joint" type="fixed">
-      <parent link="base_link" />
-      <child link="bottombase" />
-      <origin xyz="0 -0.282713 0.1775" rpy="0 0 -${M_PI/2}" />
+    <parent link="base_link" />
+    <child link="bottombase" />
+    <origin xyz="0 -0.282713 0.1775" rpy="0 0 -${M_PI/2}" />
   </joint>
   <!-- imu sensor -->
@@ -117,6 +117,6 @@
   <xacro:imu_gazebo_v0 prefix="top" />
   <xacro:include
-        filename="$(find walkie_description)/urdf/walkie/ros2_control.xacro"
-    />
+    filename="$(find walkie_description)/urdf/walkie/ros2_control.xacro"
+  />
   <xacro:ros2_control ros2_control="$(arg ros2_control)" />
 </robot>

File: urdf/walkie/omni_wheel/gz_omni_wheel.urdf.xacro (robot description, xacro)
@@ -20,5 +20,6 @@
       <visual>
         <geometry>
-          <mesh filename="package://walkie_description/meshes/walkie/omni_wheel.dae" scale="1 1 1"/>
+          <mesh filename="package://walkie_description/meshes/walkie/omni_wheel_optimize.dae" scale="1 1 1"/>
+          <!-- <mesh filename="package://walkie_description/meshes/walkie/omni_wheel.dae" scale="1 1 1"/> -->
           <!-- <mesh filename="package://walkie_description/meshes/walkie/omni_wheel.stl" scale="1 1 1"/> -->
         </geometry>

Commit message: fix: adjust min range of lidar

File: robots/gz_walkie.urdf.xacro (robot description, xacro)
@@ -1,122 +1,78 @@
-<?xml version="1.0" ?>
+<?xml version="1.0"?>
 <robot xmlns:xacro="http://ros.org/wiki/xacro" name="walkie_bot">
-  <xacro:property name="M_PI" value="3.14159274" />
-  <xacro:arg name="ros2_control" default="gazebo" />
+  <xacro:property name="M_PI" value="3.14159274"/>
+  <xacro:arg name="ros2_control" default="gazebo"/>
   <!-- Dual lidar option when only SIMULATION
   real robot force to be dual_lidar
   don't forgot to enable lidar topic to bridge in gz_bridge.yml -->
-  <xacro:arg name="dual_lidar" default="True" />
-  <xacro:include
-    filename="$(find walkie_description)/urdf/walkie/base/base.urdf.xacro"
-  />
-  <xacro:include
-    filename="$(find walkie_description)/urdf/walkie/omni_wheel/gz_omni_wheel.urdf.xacro"
-  />
-  <xacro:include
-    filename="$(find walkie_description)/urdf/walkie/lidar/lidar_gz.urdf.xacro"
-  />
-  <xacro:include
-    filename="$(find walkie_description)/urdf/walkie/imu/imu_gz.urdf.xacro"
-  />
-  <xacro:include
-    filename="$(find walkie_description)/urdf/walkie/depth_camera/d415.urdf.xacro"
-  />
+  <xacro:arg name="dual_lidar" default="True"/>
+  <xacro:include filename="$(find walkie_description)/urdf/walkie/base/base.urdf.xacro"/>
+  <xacro:include filename="$(find walkie_description)/urdf/walkie/omni_wheel/gz_omni_wheel.urdf.xacro"/>
+  <xacro:include filename="$(find walkie_description)/urdf/walkie/lidar/lidar_gz.urdf.xacro"/>
+  <xacro:include filename="$(find walkie_description)/urdf/walkie/imu/imu_gz.urdf.xacro"/>
+  <xacro:include filename="$(find walkie_description)/urdf/walkie/depth_camera/d415.urdf.xacro"/>
   <!-- =============== Link & Joint =============== -->
   <!-- Base -->
-  <link name="base_footprint" />
+  <link name="base_footprint"/>
   <xacro:base_v0 parent="base_footprint">
-    <origin xyz="0 0 0" rpy="0 0 ${M_PI / 2}" />
+    <origin xyz="0 0 0" rpy="0 0 ${M_PI / 2}"/>
   </xacro:base_v0>
-  <xacro:base_gazebo_v0 />
+  <xacro:base_gazebo_v0/>
   <!-- Wheel -->
   <!-- 1st wheel -->
   <xacro:wheel_v0 prefix="bl" parent="base_link">
-    <origin xyz="0.145261 0.145261 0.05" rpy="0 0 -${M_PI/4}" />
-    <axis xyz="0.0 1.0 0.0" />
+    <origin xyz="0.145261 0.145261 0.05" rpy="0 0 -${M_PI/4}"/>
+    <axis xyz="0.0 1.0 0.0"/>
   </xacro:wheel_v0>
   <!-- 2nd wheel -->
   <xacro:wheel_v0 prefix="br" parent="base_link">
-    <origin xyz="-0.145261 0.145261 0.05" rpy="0 0 ${M_PI/4}" />
-    <axis xyz="0.0 1.0 0.0" />
+    <origin xyz="-0.145261 0.145261 0.05" rpy="0 0 ${M_PI/4}"/>
+    <axis xyz="0.0 1.0 0.0"/>
   </xacro:wheel_v0>
   <!-- 3rd wheel -->
   <xacro:wheel_v0 prefix="fr" parent="base_link">
-    <origin xyz="-0.145261 -0.145261 0.05" rpy="0 0 ${3*M_PI/4}" />
-    <axis xyz="0.0 1.0 0.0" />
+    <origin xyz="-0.145261 -0.145261 0.05" rpy="0 0 ${3*M_PI/4}"/>
+    <axis xyz="0.0 1.0 0.0"/>
   </xacro:wheel_v0>
   <!-- 4th wheel -->
   <xacro:wheel_v0 prefix="fl" parent="base_link">
-    <origin xyz="0.145261 -0.145261 0.05" rpy="0 0 ${5*M_PI/4}" />
-    <axis xyz="0.0 1.0 0.0" />
+    <origin xyz="0.145261 -0.145261 0.05" rpy="0 0 ${5*M_PI/4}"/>
+    <axis xyz="0.0 1.0 0.0"/>
   </xacro:wheel_v0>
   <!-- lidar sensor -->
   <!-- single lidar for simulation performance -->
-  <xacro:if
-    value="${'$(arg ros2_control)' == 'gazebo' and not $(arg dual_lidar)}"
-  >
+  <xacro:if value="${'$(arg ros2_control)' == 'gazebo' and not $(arg dual_lidar)}">
     <xacro:lidar_v0 prefix="single" parent="base_link">
-      <origin xyz="0 0 0.315" rpy="0 0 -1.5707963" />
+      <origin xyz="0 0 0.315" rpy="0 0 -1.5707963"/>
     </xacro:lidar_v0>
-    <xacro:lidar_gazebo_v0
-      prefix="single"
-      min_rad="-${M_PI}"
-      max_rad=" ${M_PI}"
-      min_range="0.4"
-      max_range="10"
-      yaw_offset="0"
-    />
+    <xacro:lidar_gazebo_v0 prefix="single" min_rad="-${M_PI}" max_rad=" ${M_PI}" min_range="0.6" max_range="10" yaw_offset="0"/>
   </xacro:if>
   <!-- dual lidar when ** REAL WORLD ** or ** SIMULATION ** but set argument ** DUAL_LIDAR ** to true -->
-  <xacro:unless
-    value="${'$(arg ros2_control)' == 'gazebo' and not $(arg dual_lidar)}"
-  >
+  <xacro:unless value="${'$(arg ros2_control)' == 'gazebo' and not $(arg dual_lidar)}">
     <xacro:lidar_v0 prefix="front" parent="base_link">
-      <origin xyz="0 -0.240 0.28232" rpy="0 0 -1.5707963" />
+      <origin xyz="0 -0.240 0.28232" rpy="0 0 -1.5707963"/>
     </xacro:lidar_v0>
     <xacro:lidar_v0 prefix="back" parent="base_link">
-      <origin xyz="0 0.240 0.28232" rpy="0 0 1.5707963" />
+      <origin xyz="0 0.240 0.28232" rpy="0 0 1.5707963"/>
     </xacro:lidar_v0>
-    <xacro:lidar_gazebo_v0
-      prefix="front"
-      min_rad="-2.09333333"
-      max_rad=" 2.09333333"
-      min_range="0.18"
-      max_range="10"
-      yaw_offset="0"
-    />
-    <xacro:lidar_gazebo_v0
-      prefix="back"
-      min_rad="-2.09333333"
-      max_rad=" 2.09333333"
-      min_range="0.18"
-      max_range="10"
-      yaw_offset="0"
-    />
+    <xacro:lidar_gazebo_v0 prefix="front" min_rad="-2.09333333" max_rad=" 2.09333333" min_range="0.18" max_range="10" yaw_offset="0"/>
+    <xacro:lidar_gazebo_v0 prefix="back" min_rad="-2.09333333" max_rad=" 2.09333333" min_range="0.18" max_range="10" yaw_offset="0"/>
   </xacro:unless>
   <!-- depth cam sensor -->
-  <xacro:sensor_d415
-    name="bottom"
-    parent="base_link"
-    flag_color="1"
-    flag_ir="0"
-    flag_depth="1"
-    updaterate="2"
-  >
-    <origin xyz="0 -0.282713 0.1775" rpy="0 -0.453786 -${M_PI/2}" />
+  <xacro:sensor_d415 name="bottom" parent="base_link" flag_color="1" flag_ir="0" flag_depth="1" updaterate="2">
+    <origin xyz="0 -0.282713 0.1775" rpy="0 -0.453786 -${M_PI/2}"/>
   </xacro:sensor_d415>
-  <link name="bottombase" />
+  <link name="bottombase"/>
   <joint name="bottombase_joint" type="fixed">
-    <parent link="base_link" />
-    <child link="bottombase" />
-    <origin xyz="0 -0.282713 0.1775" rpy="0 0 -${M_PI/2}" />
+    <parent link="base_link"/>
+    <child link="bottombase"/>
+    <origin xyz="0 -0.282713 0.1775" rpy="0 0 -${M_PI/2}"/>
   </joint>
   <!-- imu sensor -->
   <xacro:imu_v0 prefix="top" parent="base_link">
-    <origin xyz="0 0 0.17" />
+    <origin xyz="0 0 0.17"/>
   </xacro:imu_v0>
-  <xacro:imu_gazebo_v0 prefix="top" />
-  <xacro:include
-    filename="$(find walkie_description)/urdf/walkie/ros2_control.xacro"
-  />
-  <xacro:ros2_control ros2_control="$(arg ros2_control)" />
+  <xacro:imu_gazebo_v0 prefix="top"/>
+  <xacro:include filename="$(find walkie_description)/urdf/walkie/ros2_control.xacro"/>
+  <xacro:ros2_control ros2_control="$(arg ros2_control)"/>
 </robot>

File: robots/gz_walkie_1arm.urdf.xacro (robot description, xacro)
@@ -90,5 +90,5 @@
       <origin xyz="0 0 0.315" rpy="0 0 -1.5707963"/>
     </xacro:lidar_v0>
-    <xacro:lidar_gazebo_v0 prefix="single" min_rad="-${M_PI}" max_rad=" ${M_PI}" min_range="0.2" max_range="10" yaw_offset="0"/>
+    <xacro:lidar_gazebo_v0 prefix="single" min_rad="-${M_PI}" max_rad=" ${M_PI}" min_range="0.6" max_range="10" yaw_offset="0"/>
   </xacro:if>
   <!-- dual lidar when ** REAL WORLD ** or ** SIMULATION ** but set argument ** DUAL_LIDAR ** to true -->

Commit message: feat: update latest config

File: robots/gz_walkie.urdf.xacro (robot description, xacro)
@@ -12,4 +12,5 @@
   <xacro:include filename="$(find walkie_description)/urdf/walkie/imu/imu_gz.urdf.xacro"/>
   <xacro:include filename="$(find walkie_description)/urdf/walkie/depth_camera/d415.urdf.xacro"/>
+  <xacro:include filename="$(find walkie_description)/urdf/walkie/head/servo_camera.urdf.xacro"/>
   <!-- =============== Link & Joint =============== -->
   <!-- Base -->
@@ -69,4 +70,7 @@
     <origin xyz="0 -0.282713 0.1775" rpy="0 0 -${M_PI/2}"/>
   </joint>
+  <xacro:servo_v0 prefix="head" parent="base_link">
+    <origin xyz="-0.098 -0.1195 0.848" rpy="0 0 0"/>
+  </xacro:servo_v0>
   <!-- imu sensor -->
   <xacro:imu_v0 prefix="top" parent="base_link">

File: urdf/walkie-arm/arm_ros2_control.xacro (robot description, xacro)
@@ -46,38 +46,38 @@
     <xacro:if value="${use_global_config or hw_config['hardware_config'][prefix + '_joint1'] == target_type}">
       <xacro:configure_single_joint name="${prefix}_joint1" type="${target_type}"
-          can_id="${id_offset + 1}" gear_ratio="10.0" external_gear_ratio="10.0" pole_pairs="14" />
+          can_id="${id_offset + 1}" gear_ratio="10.0" external_gear_ratio="10.0" pole_pairs="14" read_only="1"/>
     </xacro:if>
     <xacro:if value="${use_global_config or hw_config['hardware_config'][prefix + '_joint2'] == target_type}">
       <xacro:configure_single_joint name="${prefix}_joint2" type="${target_type}"
-          can_id="${id_offset + 2}" gear_ratio="10.0" external_gear_ratio="10.0" pole_pairs="14" />
+          can_id="${id_offset + 2}" gear_ratio="10.0" external_gear_ratio="10.0" pole_pairs="14" read_only="1" />
     </xacro:if>
     <xacro:if value="${use_global_config or hw_config['hardware_config'][prefix + '_joint3'] == target_type}">
       <xacro:configure_single_joint name="${prefix}_joint3" type="${target_type}"
-          can_id="${id_offset + 3}" gear_ratio="10.0" external_gear_ratio="10.0" pole_pairs="14" />
+          can_id="${id_offset + 3}" gear_ratio="10.0" external_gear_ratio="10.0" pole_pairs="14" read_only="1" />
     </xacro:if>
     <xacro:if value="${use_global_config or hw_config['hardware_config'][prefix + '_joint4'] == target_type}">
       <xacro:configure_single_joint name="${prefix}_joint4" type="${target_type}"
-          can_id="${id_offset + 4}" gear_ratio="10.0" external_gear_ratio="10.0" pole_pairs="14" />
+          can_id="${id_offset + 4}" gear_ratio="10.0" external_gear_ratio="10.0" pole_pairs="14" read_only="1" />
     </xacro:if>
     <xacro:if value="${use_global_config or hw_config['hardware_config'][prefix + '_joint5'] == target_type}">
       <xacro:configure_single_joint name="${prefix}_joint5" type="${target_type}"
-          can_id="${id_offset + 5}" gear_ratio="10.0" external_gear_ratio="1.0"  pole_pairs="14" />
+          can_id="${id_offset + 5}" gear_ratio="10.0" external_gear_ratio="1.0"  pole_pairs="14" read_only="0"/>
     </xacro:if>
     <xacro:if value="${use_global_config or hw_config['hardware_config'][prefix + '_joint6'] == target_type}">
       <xacro:configure_single_joint name="${prefix}_joint6" type="${target_type}"
-          can_id="${id_offset + 6}" gear_ratio="10.0" external_gear_ratio="1.0"  pole_pairs="14" />
+          can_id="${id_offset + 6}" gear_ratio="10.0" external_gear_ratio="1.0"  pole_pairs="14" read_only="0"/>
     </xacro:if>
     <xacro:if value="${use_global_config or hw_config['hardware_config'][prefix + '_joint7'] == target_type}">
       <xacro:configure_single_joint name="${prefix}_joint7" type="${target_type}"
-          can_id="${id_offset + 7}" gear_ratio="10.0" external_gear_ratio="1.0"  pole_pairs="14" />
+          can_id="${id_offset + 7}" gear_ratio="10.0" external_gear_ratio="1.0"  pole_pairs="14" read_only="0"/>
     </xacro:if>
     <xacro:if value="${use_global_config or prefix + '_gripper_worm_gear_joint' in hw_config['hardware_config']}">
          <xacro:if value="${use_global_config or hw_config['hardware_config'][prefix + '_gripper_worm_gear_joint'] == target_type}">
             <xacro:configure_single_gripper name="${prefix}_gripper_worm_gear_joint" type="${target_type}"
-                can_id="${id_offset + 8}" gear_ratio="10.0" external_gear_ratio="10.0" />
+                can_id="${id_offset + 8}" gear_ratio="10.0" external_gear_ratio="10.0"/>
          </xacro:if>
     </xacro:if>
   </xacro:macro>
-  <xacro:macro name="configure_single_joint" params="name type can_id gear_ratio external_gear_ratio pole_pairs">
+  <xacro:macro name="configure_single_joint" params="name type can_id gear_ratio external_gear_ratio pole_pairs read_only">
     <joint name="${name}">
       <xacro:if value="${type == 'cubemars'}">
@@ -87,5 +87,5 @@
         <param name="kt">0.123</param>
         <param name="enc_off">0.0</param>
-        <param name="read_only">0</param>
+        <param name="read_only">${read_only}</param>
         <param name="external_gear_ratio">${external_gear_ratio}</param>
       </xacro:if>
