Commit message: feat: add zed og urdf from zed wrapper repo (have problem frame miss match in gazebo)

File: urdf/walkie/head/servo_camera.urdf.xacro (robot description, xacro)
@@ -2,192 +2,122 @@
 <robot xmlns:xacro="http://ros.org/wiki/xacro">
   <!-- Conditionally include zed_wrapper URDF only when use_zed is true (SDK mode) -->
-  <xacro:arg name="use_zed" default="false" />
-  <xacro:if value="$(arg use_zed)">
-    <xacro:include filename="$(find zed_wrapper)/urdf/zed_macro.urdf.xacro" />
-  </xacro:if>
+  <xacro:arg name="use_zed" default="false"/>
+  <xacro:include filename="$(find walkie_description)/urdf/walkie/depth_camera/zed/zed_macro.urdf.xacro"/>
   <xacro:macro name="servo_v0" params="prefix parent *joint_origin">
-    <xacro:arg name="camera_name" default="zed_${prefix}" />
-    <xacro:arg name="camera_model" default="zed2i" />
-    <xacro:arg name="use_zed_localization" default="false" />
+    <xacro:arg name="camera_name" default="zed_${prefix}"/>
+    <xacro:arg name="camera_model" default="zed2i"/>
+    <xacro:arg name="use_zed_localization" default="false"/>
     <!-- ============ Servo Mount ============ -->
     <joint name="${prefix}_servobase_joint" type="fixed">
-      <xacro:insert_block name="joint_origin" />
-      <parent link="${parent}" />
-      <child link="${prefix}_servobase_link" />
+      <xacro:insert_block name="joint_origin"/>
+      <parent link="${parent}"/>
+      <child link="${prefix}_servobase_link"/>
     </joint>
     <link name="${prefix}_servobase_link">
       <visual>
-        <origin xyz="0 0 0" rpy="0 0 0" />
+        <origin xyz="0 0 0" rpy="0 0 0"/>
         <geometry>
-          <mesh filename="package://walkie_description/meshes/walkie/ServoMountPlate.stl"
-            scale="0.001 0.001 0.001" />
+          <mesh filename="package://walkie_description/meshes/walkie/ServoMountPlate.stl" scale="0.001 0.001 0.001"/>
         </geometry>
         <material name="dark_grey">
-          <color rgba="0.2 0.2 0.2 1" />
+          <color rgba="0.2 0.2 0.2 1"/>
         </material>
       </visual>
       <inertial>
-        <mass value="0.05" />
-        <inertia ixx="1e-5" ixy="0" ixz="0" iyy="1e-5" iyz="0" izz="1e-5" />
+        <mass value="0.05"/>
+        <inertia ixx="1e-5" ixy="0" ixz="0" iyy="1e-5" iyz="0" izz="1e-5"/>
       </inertial>
     </link>
     <!-- ============ Servo Joint (tilt) ============ -->
     <joint name="${prefix}_servo_joint" type="revolute">
-      <parent link="${prefix}_servobase_link" />
-      <child link="${prefix}_servo_link" />
-      <origin xyz="0 0 0" rpy="0 0 0" />
-      <axis xyz="-1 0 0" />
-      <limit lower="-0.384" upper="0.436" effort="10.0" velocity="1.0" />
+      <parent link="${prefix}_servobase_link"/>
+      <child link="${prefix}_servo_link"/>
+      <origin xyz="0 0 0" rpy="0 0 0"/>
+      <axis xyz="-1 0 0"/>
+      <limit lower="-0.384" upper="0.436" effort="10.0" velocity="1.0"/>
     </joint>
     <link name="${prefix}_servo_link">
       <visual>
-        <origin xyz="0 0 0" rpy="0 0 0" />
+        <origin xyz="0 0 0" rpy="0 0 0"/>
         <geometry>
-          <mesh filename="package://walkie_description/meshes/walkie/ServoCameraCase.stl"
-            scale="0.001 0.001 0.001" />
+          <mesh filename="package://walkie_description/meshes/walkie/ServoCameraCase.stl" scale="0.001 0.001 0.001"/>
         </geometry>
       </visual>
       <collision>
-        <origin xyz="0.104 0 0" rpy="0 0 0" />
+        <origin xyz="0.104 0 0" rpy="0 0 0"/>
         <geometry>
-          <box size="0.208 0.039 0.039" />
+          <box size="0.208 0.039 0.039"/>
         </geometry>
       </collision>
       <inertial>
-        <mass value="0.2" />
-        <inertia ixx="1e-4" ixy="0" ixz="0" iyy="1e-4" iyz="0" izz="1e-4" />
+        <mass value="0.2"/>
+        <inertia ixx="1e-4" ixy="0" ixz="0" iyy="1e-4" iyz="0" izz="1e-4"/>
       </inertial>
     </link>
     <!-- ============ ZED Camera Body ============ -->
-    <!-- SDK mode: use zed_wrapper macro -->
-    <xacro:if value="$(arg use_zed)">
-      <xacro:zed_camera name="zed" model="$(arg camera_model)">
-        <origin xyz="0 0 0" rpy="0 0 0" />
-      </xacro:zed_camera>
-    </xacro:if>
-    <!-- No-wrapper mode: define standalone camera links -->
-    <xacro:unless value="$(arg use_zed)">
-      <!-- Camera mount frame -->
-      <link name="$(arg camera_name)_camera_mount_link" />
-      <joint name="$(arg camera_name)_mount_joint" type="fixed">
-        <parent link="$(arg camera_name)_camera_mount_link" />
-        <child link="$(arg camera_name)_camera_link" />
-        <origin xyz="0 0 0.015" rpy="0 0 0" />
-      </joint>
-      <!-- Camera body link -->
-      <link name="$(arg camera_name)_camera_link">
-        <visual>
-          <origin xyz="0 0 0" rpy="0 0 0" />
-          <geometry>
-            <box size="0.030 0.16 0.033" />
-          </geometry>
-          <material name="zed_dark">
-            <color rgba="0.15 0.15 0.15 1" />
-          </material>
-        </visual>
-        <collision>
-          <geometry>
-            <box size="0.175 0.030 0.033" />
-          </geometry>
-        </collision>
-        <inertial>
-          <mass value="0.16" />
-          <origin xyz="0 0 0" />
-          <inertia ixx="1e-4" ixy="0" ixz="0" iyy="1e-4" iyz="0" izz="1e-4" />
-        </inertial>
-      </link>
-      <!-- Left camera frame (baseline origin) -->
-      <link name="$(arg camera_name)_left_camera_frame" />
-      <joint name="$(arg camera_name)_left_camera_joint" type="fixed">
-        <parent link="$(arg camera_name)_camera_link" />
-        <child link="$(arg camera_name)_left_camera_frame" />
-        <origin xyz="0 0.06 0" rpy="0 0 0" />
-      </joint>
-      <!-- Left camera optical frame -->
-      <link name="$(arg camera_name)_left_camera_optical_frame" />
-      <joint name="$(arg camera_name)_left_camera_optical_joint" type="fixed">
-        <parent link="$(arg camera_name)_left_camera_frame" />
-        <child link="$(arg camera_name)_left_camera_optical_frame" />
-        <origin xyz="0 0 0" rpy="0 0 0" />
-      </joint>
-      <!-- Right camera frame -->
-      <link name="$(arg camera_name)_right_camera_frame" />
-      <joint name="$(arg camera_name)_right_camera_joint" type="fixed">
-        <parent link="$(arg camera_name)_camera_link" />
-        <child link="$(arg camera_name)_right_camera_frame" />
-        <origin xyz="0 -0.06 0" rpy="0 0 0" />
-      </joint>
-      <!-- Right camera optical frame -->
-      <link name="$(arg camera_name)_right_camera_optical_frame" />
-      <joint name="$(arg camera_name)_right_camera_optical_joint" type="fixed">
-        <parent link="$(arg camera_name)_right_camera_frame" />
-        <child link="$(arg camera_name)_right_camera_optical_frame" />
-        <origin xyz="0 0 0" rpy="0 0 0" />
-      </joint>
-      <!-- Depth frame (co-located with left camera) -->
-      <link name="$(arg camera_name)_depth_frame" />
-      <joint name="$(arg camera_name)_depth_joint" type="fixed">
-        <parent link="$(arg camera_name)_left_camera_frame" />
-        <child link="$(arg camera_name)_depth_frame" />
-        <origin xyz="0 0 0" rpy="0 0 0" />
-      </joint>
-      <!-- ============ Gazebo Sensors (Gz Sim / Jazzy) ============ -->
-      <gazebo reference="$(arg camera_name)_camera_link">
-        <!-- Left RGB Camera -->
-        <sensor name="${prefix}_left_rgb_sensor" type="camera">
-          <pose relative_to="$(arg camera_name)_left_camera_optical_frame">0 0 0 0 0 0</pose>
-          <camera name="${prefix}_left">
-            <horizontal_fov>1.9199</horizontal_fov> <!-- ZED2i: 110 deg -->
-            <image>
-              <width>960</width>
-              <height>540</height>
-              <format>RGB_INT8</format>
-            </image> --> </camera>
-          <always_on>1</always_on>
-          <update_rate>15</update_rate>
-          <visualize>true</visualize>
-          <topic>${prefix}/rgb/image</topic>
-          <gz_frame_id>$(arg camera_name)_left_camera_optical_frame</gz_frame_id>
-        </sensor>
-        <!-- Depth Camera -->
-        <sensor name="${prefix}_depth_sensor" type="depth_camera">
-          <pose relative_to="$(arg camera_name)_left_camera_optical_frame">0 0 0 0 0 0</pose>
-          <camera name="${prefix}_depth">
-            <horizontal_fov>1.9199</horizontal_fov> <!-- ZED2i: 110 deg -->
-            <image>
-              <width>960</width>
-              <height>540</height>
-            </image>
-            <clip>
-              <near>0.3</near>
-              <far>20</far>
-            </clip>
-            <noise>
-              <type>gaussian</type>
-              <mean>0.0</mean>
-              <stddev>0.01</stddev>
-            </noise>
-          </camera>
-          <always_on>1</always_on>
-          <update_rate>5</update_rate>
-          <visualize>false</visualize>
-          <topic>${prefix}/depth</topic>
-          <gz_frame_id>$(arg camera_name)_left_camera_optical_frame</gz_frame_id>
-        </sensor>
-      </gazebo>
-    </xacro:unless>
+    <xacro:zed_camera name="$(arg camera_name)" model="$(arg camera_model)">
+      <origin xyz="0 0 0" rpy="0 0 0"/>
+    </xacro:zed_camera>
+    <!-- ============ Gazebo Sensors (Gz Sim / Jazzy) ============ -->
+    <gazebo reference="$(arg camera_name)_camera_link">
+      <!-- Left RGB Camera -->
+      <sensor name="${prefix}_left_rgb_sensor" type="camera">
+        <!-- TO DO : zed and gazebo frame link miss match. gazebo prefer -90yaw from zed link -->
+        <pose relative_to="$(arg camera_name)_left_camera_frame_optical">0 0 0 1.570796326794897 -1.570796326794897 0</pose>
+        <camera name="${prefix}_left">
+          <horizontal_fov>1.9199</horizontal_fov>
+          <!-- ZED2i: 110 deg -->
+          <image>
+            <width>960</width>
+            <height>540</height>
+            <format>RGB_INT8</format>
+          </image>
+        </camera>
+        <always_on>1</always_on>
+        <update_rate>15</update_rate>
+        <visualize>true</visualize>
+        <topic>${prefix}/rgb/image</topic>
+        <gz_frame_id>$(arg camera_name)_left_camera_frame_optical</gz_frame_id>
+      </sensor>
+      <!-- Depth Camera -->
+      <sensor name="${prefix}_depth_sensor" type="depth_camera">
+        <pose relative_to="$(arg camera_name)_left_camera_frame_optical">0 0 0 0 -1.570796326794897 0</pose>
+        <camera name="${prefix}_depth">
+          <horizontal_fov>1.9199</horizontal_fov>
+          <!-- ZED2i: 110 deg -->
+          <image>
+            <width>960</width>
+            <height>540</height>
+          </image>
+          <clip>
+            <near>0.3</near>
+            <far>20</far>
+          </clip>
+          <noise>
+            <type>gaussian</type>
+            <mean>0.0</mean>
+            <stddev>0.01</stddev>
+          </noise>
+        </camera>
+        <always_on>1</always_on>
+        <update_rate>10</update_rate>
+        <visualize>false</visualize>
+        <topic>${prefix}/depth</topic>
+        <gz_frame_id>$(arg camera_name)_left_camera_frame_optical</gz_frame_id>
+      </sensor>
+    </gazebo>
     <!-- ============ Camera Mounting Joint ============ -->
     <xacro:if value="$(arg use_zed_localization)">
       <joint name="$(arg camera_name)_joint" type="fixed">
-        <parent link="$(arg camera_name)_camera_mount_link" />
-        <child link="${prefix}_servo_link" />
-        <origin xyz="0.098 -0.02 -0.015" rpy="0 0 -1.5708" />
+        <parent link="$(arg camera_name)_camera_link"/>
+        <child link="${prefix}_servo_link"/>
+        <origin xyz="0.098 -0.02 -0.015" rpy="0 0 -1.5708"/>
       </joint>
     </xacro:if>
     <xacro:unless value="$(arg use_zed_localization)">
       <joint name="$(arg camera_name)_joint" type="fixed">
-        <parent link="${prefix}_servo_link" />
-        <child link="$(arg camera_name)_camera_mount_link" />
-        <origin xyz="0.098 -0.006 -0.015" rpy="0 0 -1.5708" />
+        <parent link="${prefix}_servo_link"/>
+        <child link="$(arg camera_name)_camera_link"/>
+        <origin xyz="0.098 -0.006 -0.015" rpy="0 0 -1.5708"/>
       </joint>
     </xacro:unless>

Commit message: feat: update URDF with lift and open arm

File: robots/gz_walkie.urdf.xacro (robot description, xacro)
@@ -13,4 +13,6 @@
   <xacro:include filename="$(find walkie_description)/urdf/walkie/depth_camera/d415/d415.urdf.xacro"/>
   <xacro:include filename="$(find walkie_description)/urdf/walkie/head/servo_camera.urdf.xacro"/>
+  <xacro:include filename="$(find walkie_description)/urdf/walkie/lift/lift.urdf.xacro"/>
+  <xacro:include filename="$(find walkie_description)/urdf/openarm/robot/openarm_robot.xacro"/>
   <!-- =============== Link & Joint =============== -->
   <!-- Base -->
@@ -20,23 +22,27 @@
   </xacro:base_v0>
   <xacro:base_gazebo_v0/>
+  <!-- Lift -->
+  <xacro:lift_v0 prefix="lift" parent="base_link">
+    <origin xyz="0.00000 0.07000 0.90875" rpy="0 0 0"/>
+  </xacro:lift_v0>
   <!-- Wheel -->
   <!-- 1st wheel -->
   <xacro:wheel_v0 prefix="bl" parent="base_link">
-    <origin xyz="0.145261 0.145261 0.05" rpy="0 0 -${M_PI/4}"/>
+    <origin xyz="0.130943 0.130943 0.05" rpy="0 0 -${M_PI/4}"/>
     <axis xyz="0.0 1.0 0.0"/>
   </xacro:wheel_v0>
   <!-- 2nd wheel -->
   <xacro:wheel_v0 prefix="br" parent="base_link">
-    <origin xyz="-0.145261 0.145261 0.05" rpy="0 0 ${M_PI/4}"/>
+    <origin xyz="-0.130943 0.130943 0.05" rpy="0 0 ${M_PI/4}"/>
     <axis xyz="0.0 1.0 0.0"/>
   </xacro:wheel_v0>
   <!-- 3rd wheel -->
   <xacro:wheel_v0 prefix="fr" parent="base_link">
-    <origin xyz="-0.145261 -0.145261 0.05" rpy="0 0 ${3*M_PI/4}"/>
+    <origin xyz="-0.130943 -0.130943 0.05" rpy="0 0 ${3*M_PI/4}"/>
     <axis xyz="0.0 1.0 0.0"/>
   </xacro:wheel_v0>
   <!-- 4th wheel -->
   <xacro:wheel_v0 prefix="fl" parent="base_link">
-    <origin xyz="0.145261 -0.145261 0.05" rpy="0 0 ${5*M_PI/4}"/>
+    <origin xyz="0.130943 -0.130943 0.05" rpy="0 0 ${5*M_PI/4}"/>
     <axis xyz="0.0 1.0 0.0"/>
   </xacro:wheel_v0>
@@ -52,8 +58,8 @@
   <xacro:unless value="${'$(arg ros2_control)' == 'gazebo' and not $(arg dual_lidar)}">
     <xacro:lidar_v0 prefix="front" parent="base_link">
-      <origin xyz="0 -0.240 0.28232" rpy="0 0 -1.5707963"/>
+      <origin xyz="0 -0.235 0.28232" rpy="0 0 -1.5707963"/>
     </xacro:lidar_v0>
     <xacro:lidar_v0 prefix="back" parent="base_link">
-      <origin xyz="0 0.240 0.28232" rpy="0 0 1.5707963"/>
+      <origin xyz="0 0.235 0.28232" rpy="0 0 1.5707963"/>
     </xacro:lidar_v0>
     <xacro:lidar_gazebo_v0 prefix="front" min_rad="-2.09333333" max_rad=" 2.09333333" min_range="0.18" max_range="10" yaw_offset="0"/>
@@ -62,5 +68,5 @@
   <!-- depth cam sensor -->
   <xacro:sensor_d415 name="bottom" parent="base_link" flag_color="1" flag_ir="0" flag_depth="1" updaterate="2">
-    <origin xyz="0 -0.282713 0.1775" rpy="0 -0.453786 -${M_PI/2}"/>
+    <origin xyz="0 -0.245763 0.17000" rpy="0 0.34906585 -${M_PI/2}"/>
   </xacro:sensor_d415>
   <link name="bottombase"/>
@@ -68,9 +74,9 @@
     <parent link="base_link"/>
     <child link="bottombase"/>
-    <origin xyz="0 -0.282713 0.1775" rpy="0 0 -${M_PI/2}"/>
+    <origin xyz="0 -0.245763 0.17000" rpy="0 0 -${M_PI/2}"/>
   </joint>
-  <xacro:servo_v0 prefix="head" parent="base_link">
+  <!-- <xacro:servo_v0 prefix="head" parent="base_link">
     <origin xyz="-0.098 -0.1195 0.848" rpy="0 0 0"/>
-  </xacro:servo_v0>
+  </xacro:servo_v0> -->
   <!-- imu sensor -->
   <xacro:imu_v0 prefix="top" parent="base_link">
@@ -80,3 +86,21 @@
   <xacro:include filename="$(find walkie_description)/urdf/walkie/ros2_control.xacro"/>
   <xacro:ros2_control ros2_control="$(arg ros2_control)"/>
+  <!-- OpenArm -->
+  <xacro:openarm_robot
+    arm_type="v10"
+    body_type="v10"
+    joint_limits="${xacro.load_yaml('$(find walkie_description)/config/openarm/arm/v10/joint_limits.yaml')}"
+    control_gains="${xacro.load_yaml('$(find walkie_description)/config/openarm/arm/v10/control_gains.yaml')}"
+    inertials="${xacro.load_yaml('$(find walkie_description)/config/openarm/arm/v10/inertials.yaml')}"
+    kinematics="${xacro.load_yaml('$(find walkie_description)/config/openarm/arm/v10/kinematics.yaml')}"
+    kinematics_link="${xacro.load_yaml('$(find walkie_description)/config/openarm/arm/v10/kinematics_link.yaml')}"
+    kinematics_offset="${xacro.load_yaml('$(find walkie_description)/config/openarm/arm/v10/kinematics_offset.yaml')}"
+    body_inertials="${xacro.load_yaml('$(find walkie_description)/config/openarm/body/v10/inertials.yaml')}"
+    body_kinematics="${xacro.load_yaml('$(find walkie_description)/config/openarm/body/v10/kinematics.yaml')}"
+    body_kinematics_link="${xacro.load_yaml('$(find walkie_description)/config/openarm/body/v10/kinematics_link.yaml')}"
+    ee_kinematics_link="${xacro.load_yaml('$(find walkie_description)/config/openarm/hand/openarm_hand/kinematics_link.yaml')}"
+    arm_connected_to="lift_link"
+    bimanual="true"
+    ee_type="openarm_hand"
+  />
 </robot>

File: urdf/walkie/base/base.urdf.xacro (robot description, xacro)
@@ -15,6 +15,7 @@
     <link name="base_link">
       <visual>
+        <origin xyz="0 0 0" rpy="0 0 1.5708"/>
         <geometry>
-          <mesh filename="package://walkie_description/meshes/walkie/base_link2.stl"/>
+          <mesh filename="package://walkie_description/meshes/walkie/base_link3.stl" scale="0.01 0.01 0.01"/>
         </geometry>
         <material name="grey"/>
@@ -23,13 +24,13 @@
         <origin xyz="0 0 0.165" rpy="0 0 0"/>
         <geometry>
-          <cylinder radius="0.29" length="0.33"/>
+          <cylinder radius="0.275" length="0.33"/>
         </geometry>
       </collision>
-      <collision>
+      <!-- <collision>
         <origin xyz="0 0 0.605" rpy="0 0 0"/>
         <geometry>
           <box size="0.3 0.19 0.54"/>
         </geometry>
-      </collision>
+      </collision> -->
       <xacro:inertial_cylinder mass="${base_mass}" length="${bass_thickness}" radius="${base_radian}">
         <origin xyz="0 0 0" rpy="0 0 0"/>

Commit message: feat: update head camera urdf

File: robots/gz_walkie.urdf.xacro (robot description, xacro)
@@ -76,7 +76,9 @@
     <origin xyz="0 -0.245763 0.17000" rpy="0 0 -${M_PI/2}"/>
   </joint>
-  <!-- <xacro:servo_v0 prefix="head" parent="base_link">
-    <origin xyz="-0.098 -0.1195 0.848" rpy="0 0 0"/>
-  </xacro:servo_v0> -->
+  <!-- head servo -->
+  <xacro:servo_v0 prefix="head" parent="lift_link">
+    <origin xyz="-0.03403 -0.2650 0.21525" rpy="0 0 0" />
+    <!-- <origin xyz="-0.098 -0.1195 0.848" rpy="0 0 0"/> -->
+  </xacro:servo_v0>
   <!-- imu sensor -->
   <xacro:imu_v0 prefix="top" parent="base_link">
@@ -103,4 +105,5 @@
     bimanual="true"
     ee_type="openarm_hand"
+    use_fake_hardware="true"
   />
 </robot>

File: urdf/walkie/head/servo_camera.urdf.xacro (robot description, xacro)
@@ -7,32 +7,11 @@
     <xacro:arg name="camera_model" default="zed2i"/>
     <xacro:arg name="use_zed_localization" default="false"/>
-    <!-- ============ Servo Mount ============ -->
-    <joint name="${prefix}_servobase_joint" type="fixed">
-      <xacro:insert_block name="joint_origin"/>
-      <parent link="${parent}"/>
-      <child link="${prefix}_servobase_link"/>
-    </joint>
-    <link name="${prefix}_servobase_link">
-      <visual>
-        <origin xyz="0 0 0" rpy="0 0 0"/>
-        <geometry>
-          <mesh filename="package://walkie_description/meshes/walkie/ServoMountPlate.stl" scale="0.001 0.001 0.001"/>
-        </geometry>
-        <material name="dark_grey">
-          <color rgba="0.2 0.2 0.2 1"/>
-        </material>
-      </visual>
-      <inertial>
-        <mass value="0.05"/>
-        <inertia ixx="1e-5" ixy="0" ixz="0" iyy="1e-5" iyz="0" izz="1e-5"/>
-      </inertial>
-    </link>
     <!-- ============ Servo Joint (tilt) ============ -->
     <joint name="${prefix}_servo_joint" type="revolute">
-      <parent link="${prefix}_servobase_link"/>
+      <limit lower="-3.14000" upper="3.14000" effort="0.00000" velocity="0.00000"/>
+      <parent link="${parent}"/>
       <child link="${prefix}_servo_link"/>
-      <origin xyz="0 0 0" rpy="0 0 0"/>
-      <axis xyz="-1 0 0"/>
-      <limit lower="-0.384" upper="0.436" effort="10.0" velocity="1.0"/>
+      <xacro:insert_block name="joint_origin"/>
+      <axis xyz="1.00000 0.00000 0.00000"/>
     </joint>
     <link name="${prefix}_servo_link">
@@ -40,5 +19,5 @@
         <origin xyz="0 0 0" rpy="0 0 0"/>
         <geometry>
-          <mesh filename="package://walkie_description/meshes/walkie/ServoCameraCase.stl" scale="0.001 0.001 0.001"/>
+          <mesh filename="package://walkie_description/meshes/walkie/HeadCameraMount.stl" scale="0.01 0.01 0.01"/>
         </geometry>
       </visual>
@@ -111,5 +90,5 @@
         <parent link="$(arg camera_name)_camera_link"/>
         <child link="${prefix}_servo_link"/>
-        <origin xyz="0.098 -0.02 -0.015" rpy="0 0 -1.5708"/>
+        <origin xyz="0.03403 -0.32 -0.015" rpy="0 0 -1.5708"/>
       </joint>
     </xacro:if>
@@ -118,5 +97,5 @@
         <parent link="${prefix}_servo_link"/>
         <child link="$(arg camera_name)_camera_link"/>
-        <origin xyz="0.098 -0.006 -0.015" rpy="0 0 -1.5708"/>
+        <origin xyz="0.03403 -0.063145 -0.015" rpy="0 0 -1.5708"/>
       </joint>
     </xacro:unless>

File: urdf/walkie/lift/lift.urdf.xacro (robot description, xacro)
@@ -12,5 +12,5 @@
         <visual name="lift">
             <geometry>
-                <mesh filename="package://walkie_description/meshes/walkie/lift.stl" scale="0.01 0.01 0.01"/>
+                <mesh filename="package://walkie_description/meshes/walkie/Lift.stl" scale="0.01 0.01 0.01"/>
             </geometry>
             <material name="grey"/>

File: urdf/walkie/ros2_control.xacro (robot description, xacro)
@@ -47,4 +47,11 @@
             <state_interface name="position" />
         </joint>
+        <joint name="lift_joint">
+          <command_interface name="position">
+            <param name="min">-0.51510</param>
+            <param name="max">0.00000</param>
+          </command_interface>
+          <state_interface name="position" />
+        </joint>
         </ros2_control>
     </xacro:if>
@@ -91,4 +98,11 @@
             <param name="min"> -1.54</param>
             <param name="max"> 1.54</param>
+          </command_interface>
+          <state_interface name="position" />
+        </joint>
+        <joint name="lift_joint">
+          <command_interface name="position">
+            <param name="min">-0.51510</param>
+            <param name="max">0.00000</param>
           </command_interface>
           <state_interface name="position" />
