Commit message: feat: add bimanual arm joints into gazebo ros2_control block

File: robots/gz_walkie.urdf.xacro (robot description, xacro)
@@ -105,4 +105,5 @@
     bimanual="true"
     ee_type="openarm_hand"
+    ros2_control="false"
     use_fake_hardware="true"
   />

File: urdf/walkie/ros2_control.xacro (robot description, xacro)
@@ -108,4 +108,31 @@
           <state_interface name="position" />
         </joint>
+        <xacro:macro name="gazebo_arm_joint" params="joint_name">
+          <joint name="${joint_name}">
+            <command_interface name="position"/>
+            <state_interface name="position">
+              <param name="initial_value">0.0</param>
+            </state_interface>
+            <state_interface name="velocity">
+              <param name="initial_value">0.0</param>
+            </state_interface>
+          </joint>
+        </xacro:macro>
+        <xacro:gazebo_arm_joint joint_name="openarm_left_joint1"/>
+        <xacro:gazebo_arm_joint joint_name="openarm_left_joint2"/>
+        <xacro:gazebo_arm_joint joint_name="openarm_left_joint3"/>
+        <xacro:gazebo_arm_joint joint_name="openarm_left_joint4"/>
+        <xacro:gazebo_arm_joint joint_name="openarm_left_joint5"/>
+        <xacro:gazebo_arm_joint joint_name="openarm_left_joint6"/>
+        <xacro:gazebo_arm_joint joint_name="openarm_left_joint7"/>
+        <xacro:gazebo_arm_joint joint_name="openarm_right_joint1"/>
+        <xacro:gazebo_arm_joint joint_name="openarm_right_joint2"/>
+        <xacro:gazebo_arm_joint joint_name="openarm_right_joint3"/>
+        <xacro:gazebo_arm_joint joint_name="openarm_right_joint4"/>
+        <xacro:gazebo_arm_joint joint_name="openarm_right_joint5"/>
+        <xacro:gazebo_arm_joint joint_name="openarm_right_joint6"/>
+        <xacro:gazebo_arm_joint joint_name="openarm_right_joint7"/>
+        <xacro:gazebo_arm_joint joint_name="openarm_left_finger_joint1"/>
+        <xacro:gazebo_arm_joint joint_name="openarm_right_finger_joint1"/>
       </ros2_control>
     </xacro:if>

Commit message: feat(urdf): add merged lidar link

File: robots/gz_walkie.urdf.xacro (robot description, xacro)
@@ -66,14 +66,14 @@
     <xacro:lidar_gazebo_v0 prefix="back" min_rad="-2.09333333" max_rad=" 2.09333333" min_range="0.18" max_range="10" yaw_offset="0"/>
   </xacro:unless>
+  <link name="merged_lidar_link"/>
+  <joint name="merged_lidar_joint" type="fixed">
+    <parent link="base_link"/>
+    <child link="merged_lidar_link"/>
+    <origin xyz="0 0 0.28232" rpy="0 0 0"/>
+  </joint>
   <!-- depth cam sensor -->
   <xacro:sensor_d415 name="bottom" parent="base_link" flag_color="1" flag_ir="0" flag_depth="1" updaterate="2">
     <origin xyz="0 -0.245763 0.17000" rpy="0 0.34906585 -${M_PI/2}"/>
   </xacro:sensor_d415>
-  <link name="bottombase"/>
-  <joint name="bottombase_joint" type="fixed">
-    <parent link="base_link"/>
-    <child link="bottombase"/>
-    <origin xyz="0 -0.245763 0.17000" rpy="0 0 -${M_PI/2}"/>
-  </joint>
   <!-- head servo -->
   <xacro:servo_v0 prefix="head" parent="lift_link">

File: urdf/walkie/ros2_control.xacro (robot description, xacro)
@@ -245,4 +245,14 @@
         <xacro:cubemars_wheel_joint
                     name="fl_wheel_joint"
+                    can_id="1"
+                    pole_pairs="14"
+                    gear_ratio="10"
+                    kt="0.123"
+                    enc_off="0.0"
+                    trq_limit="30"
+                    read_only="0"
+                />
+        <xacro:cubemars_wheel_joint
+                    name="fr_wheel_joint"
                     can_id="3"
                     pole_pairs="14"
@@ -254,6 +264,6 @@
                 />
         <xacro:cubemars_wheel_joint
-                    name="fr_wheel_joint"
-                    can_id="1"
+                    name="br_wheel_joint"
+                    can_id="2"
                     pole_pairs="14"
                     gear_ratio="10"
@@ -264,16 +274,6 @@
                 />
         <xacro:cubemars_wheel_joint
-                    name="br_wheel_joint"
+                    name="bl_wheel_joint"
                     can_id="4"
-                    pole_pairs="14"
-                    gear_ratio="10"
-                    kt="0.123"
-                    enc_off="0.0"
-                    trq_limit="30"
-                    read_only="0"
-                />
-        <xacro:cubemars_wheel_joint
-                    name="bl_wheel_joint"
-                    can_id="2"
                     pole_pairs="14"
                     gear_ratio="10"

Commit message: feat: temp for zed static mount before dynamixel

File: robots/gz_walkie.urdf.xacro (robot description, xacro)
@@ -77,6 +77,6 @@
   </xacro:sensor_d415>
   <!-- head servo -->
-  <xacro:servo_v0 prefix="head" parent="lift_link">
-    <origin xyz="-0.03403 -0.2650 0.21525" rpy="0 0 0" />
+  <xacro:servo_v0 prefix="head" parent="base_link">
+    <origin xyz="-0.03403 -0.2650 0.61525" rpy="0 0 0" />
     <!-- <origin xyz="-0.098 -0.1195 0.848" rpy="0 0 0"/> -->
   </xacro:servo_v0>

Commit message: fix:depth-cam

File: robots/gz_walkie.urdf.xacro (robot description, xacro)
@@ -77,6 +77,6 @@
   </xacro:sensor_d415>
   <!-- head servo -->
-  <xacro:servo_v0 prefix="head" parent="base_link">
-    <origin xyz="-0.03403 -0.2650 0.61525" rpy="0 0 0" />
+  <xacro:servo_v0 prefix="head" parent="lift_link">
+    <origin xyz="-0.03403 -0.2650 0.21525" rpy="0 0 0" />
     <!-- <origin xyz="-0.098 -0.1195 0.848" rpy="0 0 0"/> -->
   </xacro:servo_v0>

Commit message: feat: update URDF for openarm and lift

File: robots/gz_walkie.urdf.xacro (robot description, xacro)
@@ -24,5 +24,5 @@
   <!-- Lift -->
   <xacro:lift_v0 prefix="lift" parent="base_link">
-    <origin xyz="0.00000 0.07000 0.90875" rpy="0 0 0"/>
+    <origin xyz="0.00000 0.07000 0.3985" rpy="0 0 0"/>
   </xacro:lift_v0>
   <!-- Wheel -->
@@ -78,5 +78,5 @@
   <!-- head servo -->
   <xacro:servo_v0 prefix="head" parent="lift_link">
-    <origin xyz="-0.03403 -0.2650 0.21525" rpy="0 0 0" />
+    <origin xyz="-0.03403 -0.2650 0.20075" rpy="0 0 0" />
     <!-- <origin xyz="-0.098 -0.1195 0.848" rpy="0 0 0"/> -->
   </xacro:servo_v0>

File: urdf/openarm/robot/openarm_robot.xacro (robot description, xacro)
@@ -29,6 +29,6 @@
             body_connected_to='world'
             bimanual:=false
-            right_arm_base_xyz='-0.083 -0.230 0.123'
-            left_arm_base_xyz='0.083 -0.230 0.123'
+            right_arm_base_xyz='-0.03 -0.230 0.1085'
+            left_arm_base_xyz='0.03 -0.230 0.1085'
             right_arm_base_rpy='1.5708 0 -1.5708'
             left_arm_base_rpy='-1.5708 0 -1.5708'

File: urdf/walkie/base/base.urdf.xacro (robot description, xacro)
@@ -15,7 +15,7 @@
     <link name="base_link">
       <visual>
-        <origin xyz="0 0 0" rpy="0 0 1.5708"/>
+        <origin xyz="0 0 0" rpy="0 0 0"/>
         <geometry>
-          <mesh filename="package://walkie_description/meshes/walkie/base_link3.stl" scale="0.01 0.01 0.01"/>
+          <mesh filename="package://walkie_description/meshes/walkie/base_link4.stl"/>
         </geometry>
         <material name="grey"/>
@@ -28,7 +28,7 @@
       </collision>
       <collision>
-        <origin xyz="0 0.07 0.725" rpy="0 0 0"/>
+        <origin xyz="0 0.07 0.845" rpy="0 0 0"/>
         <geometry>
-          <box size="0.196 0.18 0.80"/>
+          <box size="0.196 0.18 1.04"/>
         </geometry>
       </collision>

File: urdf/walkie/lift/lift.urdf.xacro (robot description, xacro)
@@ -4,5 +4,5 @@
     <joint name="${prefix}_joint" type="prismatic">
         <xacro:insert_block name="joint_origin"/>
-        <limit lower="-0.506" upper="0.00000" effort="100.0" velocity="0.1"/>
+        <limit lower="0.000" upper="0.743" effort="1000.0" velocity="0.1"/>
         <parent link="${parent}"/>
         <child link="${prefix}_link"/>
@@ -12,5 +12,5 @@
         <visual name="lift">
             <geometry>
-                <mesh filename="package://walkie_description/meshes/walkie/Lift.stl" scale="0.01 0.01 0.01"/>
+                <mesh filename="package://walkie_description/meshes/walkie/Lift2.stl"/>
             </geometry>
             <material name="grey"/>

File: urdf/walkie/ros2_control.xacro (robot description, xacro)
@@ -90,6 +90,6 @@
         <joint name="lift_joint">
           <command_interface name="position">
-            <param name="min">-0.51510</param>
-            <param name="max">0.00000</param>
+            <param name="min">0.000</param>
+            <param name="max">0.743</param>
           </command_interface>
           <state_interface name="position">
@@ -153,8 +153,10 @@
         <joint name="lift_joint">
           <command_interface name="position">
-            <param name="min">-0.51510</param>
-            <param name="max">0.00000</param>
-          </command_interface>
-          <state_interface name="position" />
+            <param name="min">0.000</param>
+            <param name="max">0.743</param>
+          </command_interface>
+          <state_interface name="position">
+            <param name="initial_value">0.51</param>
+          </state_interface>
         </joint>
         <xacro:position_arm_joint joint_name="openarm_left_joint1" />
@@ -218,6 +220,6 @@
             <command_interface name="effort" />
             <command_interface name="position">
-                <param name="min">-0.51510</param>
-                <param name="max">0.00000</param>
+                <param name="min">0.000</param>
+                <param name="max">0.743</param>
             </command_interface>
             <state_interface name="position" />
@@ -306,6 +308,6 @@
         <joint name="lift_joint">
           <command_interface name="position">
-            <param name="min">-0.51510</param>
-            <param name="max">0.00000</param>
+            <param name="min">0.00000</param>
+            <param name="max">0.74300</param>
           </command_interface>
           <state_interface name="position" />

Commit message: feat: add unitree lidar urdf

File: robots/gz_walkie.urdf.xacro (robot description, xacro)
@@ -10,4 +10,5 @@
   <xacro:include filename="$(find walkie_description)/urdf/walkie/omni_wheel/gz_omni_wheel.urdf.xacro"/>
   <xacro:include filename="$(find walkie_description)/urdf/walkie/lidar/lidar_gz.urdf.xacro"/>
+  <xacro:include filename="$(find walkie_description)/urdf/walkie/lidar/unitree_lidar.urdf.xacro"/>
   <xacro:include filename="$(find walkie_description)/urdf/walkie/imu/imu_gz.urdf.xacro"/>
   <xacro:include filename="$(find walkie_description)/urdf/walkie/depth_camera/d415/d415.urdf.xacro"/>
@@ -72,4 +73,9 @@
     <origin xyz="0 0 0.28232" rpy="0 0 0"/>
   </joint>
+  <!-- Unitree 4D L2 lidar sensor (3D) -->
+  <xacro:unitree4d_l2_lidar prefix="unitree4d_l2" parent="base_link" min_angle="-3.14159274" max_angle="3.14159274">
+    <origin xyz="0 0.07421152 1.53746187" rpy="3.14159 -0.5236 1.5707963"/>
+  </xacro:unitree4d_l2_lidar>
+  <xacro:unitree4d_l2_lidar_gazebo prefix="unitree4d_l2" min_angle="-3.14159274" max_angle="3.14159274"/>
   <!-- depth cam sensor -->
   <xacro:sensor_d415 name="bottom" parent="base_link" flag_color="1" flag_ir="0" flag_depth="1" updaterate="2">

File: urdf/walkie/ros2_control.xacro (robot description, xacro)
@@ -293,12 +293,32 @@
       <ros2_control name="HeadServoSystem" type="system">
         <hardware>
-          <plugin>mock_components/GenericSystem</plugin>
-          <param name="joint_commands_topic">/head_servo_joint_cmd</param>
-          <param name="joint_states_topic">/head_servo_joint_states</param>
+          <plugin>dynamixel_hardware_interface/DynamixelHardware</plugin>
+          <param name="port_name">/dev/ttyUSB0</param>
+          <param name="baud_rate">57600</param>
+          <param name="number_of_joints">1</param>
+          <param name="number_of_transmissions">1</param>
+          <param name="dynamixel_model_folder">/param/dxl_model</param>
         </hardware>
         <joint name="head_servo_joint">
-          <command_interface name="position" />
-          <state_interface name="position" />
-        </joint>
+          <command_interface name="position">
+            <param name="min">-0.7854</param>
+            <param name="max">0.7854</param>
+          </command_interface>
+          <state_interface name="position"/>
+          <state_interface name="velocity"/>
+          <state_interface name="effort"/>
+        </joint>
+        <gpio name="head_servo_joint">
+          <param name="type">dxl</param>
+          <param name="ID">2</param>
+          <command_interface name="Goal Position"/>
+          <state_interface name="Present Position"/>
+          <state_interface name="Present Velocity"/>
+          <state_interface name="Present Load"/>
+          <param name="Position P Gain">800</param>
+          <param name="Position I Gain">100</param>
+          <param name="Position D Gain">100</param>
+          <param name="Drive Mode">0</param>
+        </gpio>
       </ros2_control>
       <ros2_control name="LiftSystem" type="system">

Commit message: fix: update lidar urdf calibration

File: robots/gz_walkie.urdf.xacro (robot description, xacro)
@@ -74,8 +74,16 @@
   </joint>
   <!-- Unitree 4D L2 lidar sensor (3D) -->
-  <xacro:unitree4d_l2_lidar prefix="unitree4d_l2" parent="base_link" min_angle="-3.14159274" max_angle="3.14159274">
-    <origin xyz="0 0.07421152 1.53746187" rpy="3.14159 -0.5236 1.5707963"/>
-  </xacro:unitree4d_l2_lidar>
-  <xacro:unitree4d_l2_lidar_gazebo prefix="unitree4d_l2" min_angle="-3.14159274" max_angle="3.14159274"/>
+  <link name="unitree4d_l2_imu_initial"/>
+  <joint name="unitree4d_l2_imu_initial_joint" type="fixed">
+    <parent link="base_link"/>
+    <child link="unitree4d_l2_imu_initial"/>
+    <origin xyz="0 0.05196152 1.676" rpy="3.36159 -0.445 1.09"/>
+  </joint>
+  <link name="unitree4d_l2_imu"/>
+  <joint name="unitree4d_l2_imu_joint" type="fixed">
+    <parent link="unitree4d_l2_imu_initial"/>
+    <child link="unitree4d_l2_imu"/>
+    <origin xyz="-0.007698 -0.014655 0.00667" rpy="0 0 0"/>
+  </joint>
   <!-- depth cam sensor -->
   <xacro:sensor_d415 name="bottom" parent="base_link" flag_color="1" flag_ir="0" flag_depth="1" updaterate="2">

Commit message: feat(description): integrate openarm real hardware configuration
Updates the main robot URDF and ros2_control configuration to support the bimanual arms on the real robot.

NOTE: This configuration currently breaks simulation pipelines. The robot compiles and runs successfully on physical hardware, but additional gazebo/mock matching configurations are required to restore simulation functionality.

File: robots/gz_walkie.urdf.xacro (robot description, xacro)
@@ -7,4 +7,8 @@
   don't forgot to enable lidar topic to bridge in gz_bridge.yml -->
   <xacro:arg name="dual_lidar" default="True"/>
+  <xacro:arg name="use_arm" default="True"/>
+  <xacro:arg name="use_fake_arm_hardware" default="True"/>
+  <xacro:arg name="left_can_interface" default="can1"/>
+  <xacro:arg name="right_can_interface" default="can0"/>
   <xacro:include filename="$(find walkie_description)/urdf/walkie/base/base.urdf.xacro"/>
   <xacro:include filename="$(find walkie_description)/urdf/walkie/omni_wheel/gz_omni_wheel.urdf.xacro"/>
@@ -101,5 +105,11 @@
   <xacro:imu_gazebo_v0 prefix="top"/>
   <xacro:include filename="$(find walkie_description)/urdf/walkie/ros2_control.xacro"/>
-  <xacro:ros2_control ros2_control="$(arg ros2_control)"/>
+  <xacro:ros2_control ros2_control="$(arg ros2_control)"
+    use_fake_hardware="$(arg use_fake_arm_hardware)"
+    left_can_interface="$(arg left_can_interface)"
+    right_can_interface="$(arg right_can_interface)"
+    hand="true"
+    control_gains="${xacro.load_yaml('$(find walkie_description)/config/openarm/arm/v10/control_gains.yaml')}"
+  />
   <!-- OpenArm -->
   <xacro:openarm_robot
@@ -119,6 +129,9 @@
     bimanual="true"
     ee_type="openarm_hand"
-    ros2_control="false"
-    use_fake_hardware="true"
+    hand="true"
+    ros2_control="${'$(arg ros2_control)' == 'real_robot'}"
+    use_fake_hardware="$(arg use_fake_arm_hardware)"
+    left_can_interface="$(arg left_can_interface)"
+    right_can_interface="$(arg right_can_interface)"
   />
 </robot>

File: urdf/walkie/ros2_control.xacro (robot description, xacro)
@@ -24,4 +24,7 @@
       </state_interface>
       <state_interface name="velocity">
+        <param name="initial_value">0.0</param>
+      </state_interface>
+      <state_interface name="effort">
         <param name="initial_value">0.0</param>
       </state_interface>
@@ -54,5 +57,34 @@
     </joint>
   </xacro:macro>
-  <xacro:macro name="ros2_control" params="ros2_control">
+  <!-- Global helper macro to configure real arm hardware joints cleanly -->
+  <xacro:macro name="configure_joint" params="joint_name initial_position">
+    <joint name="${joint_name}">
+      <command_interface name="position"/>
+      <command_interface name="velocity"/>
+      <command_interface name="effort"/>
+      <state_interface name="position">
+        <param name="initial_value">${initial_position}</param>
+      </state_interface>
+      <state_interface name="velocity">
+        <param name="initial_value">0.0</param>
+      </state_interface>
+      <state_interface name="effort">
+        <param name="initial_value">0.0</param>
+      </state_interface>
+    </joint>
+  </xacro:macro>
+  <!-- Main Macro Declaration (ros2_control included back into parameters list) -->
+  <xacro:macro name="ros2_control"
+            params="ros2_control
+                arm_type:=^|openarm
+                control_gains:=^|{}
+                left_can_interface:=^|can1
+                right_can_interface:=^|can0
+                use_fake_hardware:=^|true
+                fake_sensor_commands:=^|false
+                hand:=^|false
+                left_arm_prefix:=^|left_
+                right_arm_prefix:=^|right_
+                can_fd:=^|true">
     <!-- Mock hardware -->
     <xacro:if value="${ros2_control == 'mock'}">
@@ -241,5 +273,5 @@
         <xacro:position_arm_joint joint_name="openarm_left_finger_joint1" />
         <xacro:position_arm_joint joint_name="openarm_right_finger_joint1" />
-        </ros2_control>
+      </ros2_control>
     </xacro:if>
     <!-- Real Hardware : real_robot based ros2_control -->
@@ -248,5 +280,5 @@
         <hardware>
           <plugin>cubemars_hardware/CubeMarsSystemHardware</plugin>
-          <param name="can_interface">can0</param>
+          <param name="can_interface">can2</param>
         </hardware>
         <xacro:cubemars_wheel_joint
@@ -299,4 +331,5 @@
           <param name="number_of_transmissions">1</param>
           <param name="dynamixel_model_folder">/param/dxl_model</param>
+          <param name="disable_torque_at_init">true</param>
         </hardware>
         <joint name="head_servo_joint">
@@ -331,27 +364,11 @@
             <param name="max">0.74300</param>
           </command_interface>
-          <state_interface name="position" />
-        </joint>
-      </ros2_control>
-      <ros2_control name="ArmSystem" type="system">
-        <hardware>
-          <plugin>mock_components/GenericSystem</plugin>
-        </hardware>
-        <xacro:position_arm_joint joint_name="openarm_left_joint1" />
-        <xacro:position_arm_joint joint_name="openarm_left_joint2" />
-        <xacro:position_arm_joint joint_name="openarm_left_joint3" />
-        <xacro:position_arm_joint joint_name="openarm_left_joint4" />
-        <xacro:position_arm_joint joint_name="openarm_left_joint5" />
-        <xacro:position_arm_joint joint_name="openarm_left_joint6" />
-        <xacro:position_arm_joint joint_name="openarm_left_joint7" />
-        <xacro:position_arm_joint joint_name="openarm_right_joint1" />
-        <xacro:position_arm_joint joint_name="openarm_right_joint2" />
-        <xacro:position_arm_joint joint_name="openarm_right_joint3" />
-        <xacro:position_arm_joint joint_name="openarm_right_joint4" />
-        <xacro:position_arm_joint joint_name="openarm_right_joint5" />
-        <xacro:position_arm_joint joint_name="openarm_right_joint6" />
-        <xacro:position_arm_joint joint_name="openarm_right_joint7" />
-        <xacro:position_arm_joint joint_name="openarm_left_finger_joint1" />
-        <xacro:position_arm_joint joint_name="openarm_right_finger_joint1" />
+          <state_interface name="position">
+            <param name="initial_value">0.0</param>
+          </state_interface>
+          <state_interface name="velocity">
+            <param name="initial_value">0.0</param>
+          </state_interface>
+        </joint>
       </ros2_control>
     </xacro:if>
