Commit message: feat: update head camera and lift model

File: robots/gz_walkie.urdf.xacro (robot description, xacro)
@@ -24,5 +24,5 @@
   <link name="base_footprint"/>
   <xacro:base_v0 parent="base_footprint">
-    <origin xyz="0 0 0" rpy="0 0 ${M_PI / 2}"/>
+    <origin xyz="0 0 0.0312" rpy="0 0 ${M_PI / 2}"/>
   </xacro:base_v0>
   <xacro:base_gazebo_v0/>
@@ -92,9 +92,9 @@
   <!-- depth cam sensor -->
   <xacro:sensor_d415 name="bottom" parent="base_link" flag_color="1" flag_ir="0" flag_depth="1" updaterate="2">
-    <origin xyz="0 -0.245763 0.17000" rpy="0 0.34906585 -${M_PI/2}"/>
+    <origin xyz="0 -0.26275 0.17747" rpy="0 -0.436332313 -${M_PI/2}"/>
   </xacro:sensor_d415>
   <!-- head servo -->
   <xacro:servo_v0 prefix="head" parent="lift_link">
-    <origin xyz="-0.03403 -0.2650 0.20075" rpy="0 0 0" />
+    <origin xyz="-0.03403 -0.2650 0.20075" rpy="0.0698132 0 0" />
     <!-- <origin xyz="-0.098 -0.1195 0.848" rpy="0 0 0"/> -->
   </xacro:servo_v0>

File: urdf/walkie/base/base.urdf.xacro (robot description, xacro)
@@ -17,5 +17,5 @@
         <origin xyz="0 0 0" rpy="0 0 0"/>
         <geometry>
-          <mesh filename="package://walkie_description/meshes/walkie/base_link4.stl"/>
+          <mesh filename="package://walkie_description/meshes/walkie/base_link.stl"/>
         </geometry>
         <material name="grey"/>

File: urdf/walkie/head/servo_camera.urdf.xacro (robot description, xacro)
@@ -9,5 +9,5 @@
     <!-- ============ Servo Joint (tilt) ============ -->
     <joint name="${prefix}_servo_joint" type="revolute">
-      <limit lower="-0.785398163" upper="0.785398163" effort="0.00000" velocity="0.00000"/>
+      <limit lower="-0.785398163" upper="1.04719755" effort="0.00000" velocity="0.00000"/>
       <parent link="${parent}"/>
       <child link="${prefix}_servo_link"/>
@@ -19,11 +19,11 @@
         <origin xyz="0 0 0" rpy="0 0 0"/>
         <geometry>
-          <mesh filename="package://walkie_description/meshes/walkie/HeadCameraMount.stl" scale="0.01 0.01 0.01"/>
+          <mesh filename="package://walkie_description/meshes/walkie/HeadCameraMount.stl"/>
         </geometry>
       </visual>
       <collision>
-        <origin xyz="0.034 -0.056649 0" rpy="0 0 0"/>
+        <origin xyz="0 0 0" rpy="0 0 0"/>
         <geometry>
-          <box size="0.186 0.044 0.040"/>
+          <mesh filename="package://walkie_description/meshes/walkie/HeadCameraMount.stl"/>
         </geometry>
       </collision>
@@ -90,5 +90,5 @@
         <parent link="$(arg camera_name)_camera_link"/>
         <child link="${prefix}_servo_link"/>
-        <origin xyz="0.03403 -0.32 -0.015" rpy="0 0 -1.5708"/>
+        <origin xyz="0.034 -0.088 0.005" rpy="0 0 -1.5708"/>
       </joint>
     </xacro:if>
@@ -97,5 +97,5 @@
         <parent link="${prefix}_servo_link"/>
         <child link="$(arg camera_name)_camera_link"/>
-        <origin xyz="0.03403 -0.063145 -0.015" rpy="0 0 -1.5708"/>
+        <origin xyz="0.034 -0.088 0.005" rpy="0 0 -1.5708"/>
       </joint>
     </xacro:unless>

File: urdf/walkie/lift/lift.urdf.xacro (robot description, xacro)
@@ -12,5 +12,5 @@
         <visual name="lift">
             <geometry>
-                <mesh filename="package://walkie_description/meshes/walkie/Lift2.stl"/>
+                <mesh filename="package://walkie_description/meshes/walkie/Lift.stl"/>
             </geometry>
             <material name="grey"/>
@@ -23,5 +23,5 @@
         </collision> -->
         <collision name="top_bar">
-            <origin xyz="0 0 0.122" rpy="0 0 0"/>
+            <origin xyz="0 0 0.109" rpy="0 0 0"/>
             <geometry>
             <box size="0.346 0.174 0.132"/>
@@ -30,5 +30,5 @@
         <!-- Vertical stem -->
         <collision name="stem">
-            <origin xyz="0 -0.172 0.122" rpy="0 0 0"/>
+            <origin xyz="0 -0.172 0.109" rpy="0 0 0"/>
             <geometry>
             <box size="0.190 0.190 0.132"/>

Commit message: feat:right joint 2 fixed

File: robots/gz_walkie.urdf.xacro (robot description, xacro)
@@ -11,4 +11,7 @@
   <xacro:arg name="left_use_fake_arm_hardware" default="$(arg use_fake_arm_hardware)"/>
   <xacro:arg name="right_use_fake_arm_hardware" default="$(arg use_fake_arm_hardware)"/>
+  <xacro:arg name="right_joint2_fixed" default="False"/>
+  <xacro:arg name="sim_controllers_yaml"
+             default="$(find walkie_description)/config/ros2_controller/sim_controllers.yaml"/>
   <xacro:arg name="left_can_interface" default="can1"/>
   <xacro:arg name="right_can_interface" default="can0"/>
@@ -109,4 +112,6 @@
   <xacro:ros2_control ros2_control="$(arg ros2_control)"
     use_fake_hardware="$(arg use_fake_arm_hardware)"
+    right_joint2_fixed="$(arg right_joint2_fixed)"
+    sim_controllers_yaml="$(arg sim_controllers_yaml)"
     left_can_interface="$(arg left_can_interface)"
     right_can_interface="$(arg right_can_interface)"
@@ -135,4 +140,5 @@
     left_use_fake_hardware="$(arg left_use_fake_arm_hardware)"
     right_use_fake_hardware="$(arg right_use_fake_arm_hardware)"
+    right_joint2_fixed="$(arg right_joint2_fixed)"
     left_can_interface="$(arg left_can_interface)"
     right_can_interface="$(arg right_can_interface)"

File: urdf/openarm/arm/openarm_arm.xacro (robot description, xacro)
@@ -2,5 +2,5 @@
 <robot xmlns:xacro="http://www.ros.org/wiki/xacro" name="openarm">
   <xacro:include filename="$(find walkie_description)/urdf/openarm/arm/openarm_macro.xacro" />
-  <xacro:macro name="openarm_arm" params="arm_type arm_prefix:='' no_prefix:=false description_pkg:='walkie_description' connected_to:='base' xyz:='0 0 0' rpy:='0 0 0' joint_limits inertials kinematics kinematics_link kinematics_offset:=none " >
+  <xacro:macro name="openarm_arm" params="arm_type arm_prefix:='' no_prefix:=false description_pkg:='walkie_description' connected_to:='base' xyz:='0 0 0' rpy:='0 0 0' joint_limits inertials kinematics kinematics_link kinematics_offset:=none joint2_fixed:=false " >
     <xacro:property name="prefix" value="${'' if no_prefix else 'openarm' + '_' + arm_prefix}" />
     <xacro:if value="${arm_prefix == 'right_'}">
@@ -35,11 +35,20 @@
       <xacro:property name="limit_offset_joint2" value="${-pi/2}" />
     </xacro:if>
-    <joint name="${prefix}joint2" type="revolute">
-      <xacro:openarm-kinematics name="joint2" config="${kinematics}" offset="${kinematics_offset}" reflect="${reflect}"/>
-      <parent link="${prefix}link1" />
-      <child link="${prefix}link2" />
-      <axis xyz="-1 0 0" />
-      <xacro:openarm-limits name="joint2" config="${joint_limits}" reflect="${reflect}" offset="${limit_offset_joint2}"/>
-    </joint>
+    <xacro:if value="${joint2_fixed}">
+      <joint name="${prefix}joint2" type="fixed">
+        <xacro:openarm-kinematics name="joint2" config="${kinematics}" offset="${kinematics_offset}" reflect="${reflect}"/>
+        <parent link="${prefix}link1" />
+        <child link="${prefix}link2" />
+      </joint>
+    </xacro:if>
+    <xacro:unless value="${joint2_fixed}">
+      <joint name="${prefix}joint2" type="revolute">
+        <xacro:openarm-kinematics name="joint2" config="${kinematics}" offset="${kinematics_offset}" reflect="${reflect}"/>
+        <parent link="${prefix}link1" />
+        <child link="${prefix}link2" />
+        <axis xyz="-1 0 0" />
+        <xacro:openarm-limits name="joint2" config="${joint_limits}" reflect="${reflect}" offset="${limit_offset_joint2}"/>
+      </joint>
+    </xacro:unless>
     <xacro:link_with_sc no_prefix="${no_prefix}" name="link3" kinematics_link="${kinematics_link}" inertials="${inertials}" reflect="${reflect}"/>
     <joint name="${prefix}joint3" type="revolute">

File: urdf/openarm/robot/openarm_robot.xacro (robot description, xacro)
@@ -24,4 +24,5 @@
             left_use_fake_hardware:=false
             right_use_fake_hardware:=false
+            right_joint2_fixed:=false
             fake_sensor_commands:=false
             no_prefix:='false'
@@ -83,5 +84,6 @@
         kinematics="${kinematics}"
         kinematics_link="${kinematics_link}"
-        kinematics_offset="${kinematics_offset}" />
+        kinematics_offset="${kinematics_offset}"
+        joint2_fixed="${right_joint2_fixed}" />
         <!-- ros2_control hardware interfaces for bimanual setup -->
         <xacro:if value="${ros2_control}">
@@ -93,4 +95,5 @@
             left_use_fake_hardware="${left_use_fake_hardware}"
             right_use_fake_hardware="${right_use_fake_hardware}"
+            right_joint2_fixed="${right_joint2_fixed}"
             fake_sensor_commands="${fake_sensor_commands}"
             left_arm_prefix="${left_arm_prefix}"

File: urdf/openarm/robot/v10.urdf.xacro (robot description, xacro)
@@ -22,4 +22,5 @@
   <xacro:arg name="left_use_fake_hardware" default="$(arg use_fake_hardware)" />
   <xacro:arg name="right_use_fake_hardware" default="$(arg use_fake_hardware)" />
+  <xacro:arg name="right_joint2_fixed" default="false" />
   <xacro:arg name="fake_sensor_commands" default="false" />
   <xacro:arg name="bimanual" default="true" />
@@ -51,4 +52,7 @@
   right_arm_prefix="$(arg right_arm_prefix)"
   use_fake_hardware="$(arg use_fake_hardware)"
+  left_use_fake_hardware="$(arg left_use_fake_hardware)"
+  right_use_fake_hardware="$(arg right_use_fake_hardware)"
+  right_joint2_fixed="$(arg right_joint2_fixed)"
   fake_sensor_commands="$(arg fake_sensor_commands)"
   no_prefix="$(arg no_prefix)"

File: urdf/openarm/ros2_control/openarm.bimanual.ros2_control.xacro (robot description, xacro)
@@ -8,4 +8,5 @@
              left_use_fake_hardware:=^|false
              right_use_fake_hardware:=^|false
+             right_joint2_fixed:=^|false
              fake_sensor_commands:=^|false
              hand:=^|false
@@ -117,5 +118,7 @@
         </hardware>
       <xacro:configure_joint joint_name="openarm_${right_arm_prefix}joint1" initial_position="0.0"/>
-      <xacro:configure_joint joint_name="openarm_${right_arm_prefix}joint2" initial_position="0.0"/>
+      <xacro:unless value="${right_joint2_fixed}">
+        <xacro:configure_joint joint_name="openarm_${right_arm_prefix}joint2" initial_position="0.0"/>
+      </xacro:unless>
       <xacro:configure_joint joint_name="openarm_${right_arm_prefix}joint3" initial_position="0.0"/>
       <xacro:configure_joint joint_name="openarm_${right_arm_prefix}joint4" initial_position="0.0"/>

File: urdf/walkie/ros2_control.xacro (robot description, xacro)
@@ -86,5 +86,7 @@
                 left_arm_prefix:=^|left_
                 right_arm_prefix:=^|right_
-                can_fd:=^|true">
+                can_fd:=^|true
+                right_joint2_fixed:=^|false
+                sim_controllers_yaml">
     <!-- Mock hardware -->
     <xacro:if value="${ros2_control == 'mock'}">
@@ -140,5 +142,7 @@
         <xacro:position_arm_joint joint_name="openarm_left_joint7" />
         <xacro:position_arm_joint joint_name="openarm_right_joint1" initial_position="-0.2618" />
-        <xacro:position_arm_joint joint_name="openarm_right_joint2" />
+        <xacro:unless value="${right_joint2_fixed}">
+          <xacro:position_arm_joint joint_name="openarm_right_joint2" />
+        </xacro:unless>
         <xacro:position_arm_joint joint_name="openarm_right_joint3" />
         <xacro:position_arm_joint joint_name="openarm_right_joint4" initial_position="0.2618" />
@@ -200,5 +204,7 @@
         <xacro:position_arm_joint joint_name="openarm_left_joint7" />
         <xacro:position_arm_joint joint_name="openarm_right_joint1" initial_position="-0.2618" />
-        <xacro:position_arm_joint joint_name="openarm_right_joint2" />
+        <xacro:unless value="${right_joint2_fixed}">
+          <xacro:position_arm_joint joint_name="openarm_right_joint2" />
+        </xacro:unless>
         <xacro:position_arm_joint joint_name="openarm_right_joint3" />
         <xacro:position_arm_joint joint_name="openarm_right_joint4" initial_position="0.2618" />
@@ -277,5 +283,7 @@
         <xacro:position_arm_joint joint_name="openarm_left_joint7" />
         <xacro:position_arm_joint joint_name="openarm_right_joint1" initial_position="-0.2618" />
-        <xacro:position_arm_joint joint_name="openarm_right_joint2" />
+        <xacro:unless value="${right_joint2_fixed}">
+          <xacro:position_arm_joint joint_name="openarm_right_joint2" />
+        </xacro:unless>
         <xacro:position_arm_joint joint_name="openarm_right_joint3" />
         <xacro:position_arm_joint joint_name="openarm_right_joint4" initial_position="0.2618" />
@@ -395,5 +403,5 @@
                 >
           <parameters
-                    >$(find walkie_description)/config/ros2_controller/sim_controllers.yaml</parameters>
+                    >${sim_controllers_yaml}</parameters>
         </plugin>
       </gazebo>
