Commit message: fix(urdf): tune bottom depth cam & head servo pose, base collision
- gz_walkie: lower bottom D415 origin and steepen pitch (-0.436 -> -0.873 rad); increase head servo roll (0.0698 -> 0.157 rad)
- base: trim base collision box depth 0.07 -> 0.069 m
- refresh base_link.stl mesh

Co-Authored-By: Claude Opus 4.8 (1M context) <noreply@anthropic.com>

File: robots/gz_walkie.urdf.xacro (robot description, xacro)
@@ -97,9 +97,9 @@
   <!-- depth cam sensor -->
   <xacro:sensor_d415 name="bottom" parent="base_link" flag_color="1" flag_ir="0" flag_depth="1" updaterate="2">
-    <origin xyz="0 -0.26275 0.17747" rpy="0 -0.436332313 -${M_PI/2}"/>
+    <origin xyz="0 -0.27386242 0.18004809" rpy="0 -0.872664626  -${M_PI/2}"/>
   </xacro:sensor_d415>
   <!-- head servo -->
   <xacro:servo_v0 prefix="head" parent="lift_link">
-    <origin xyz="-0.03403 -0.2650 0.20075" rpy="0.0698132 0 0" />
+    <origin xyz="-0.03403 -0.2650 0.20075" rpy="0.157079633 0 0" />
     <!-- <origin xyz="-0.098 -0.1195 0.848" rpy="0 0 0"/> -->
   </xacro:servo_v0>

File: urdf/walkie/base/base.urdf.xacro (robot description, xacro)
@@ -36,5 +36,5 @@
         <origin xyz="-0.115 0.07 0.845" rpy="0 0 0"/>
         <geometry>
-          <box size="0.23 0.07 1.04"/>
+          <box size="0.23 0.069 1.04"/>
         </geometry>
       </collision>
