Commit message: feat: add roller option (default: simple wheel colider)

File: robots/gz_walkie.urdf.xacro (robot description, xacro)
@@ -3,4 +3,5 @@
   <xacro:property name="M_PI" value="3.14159274"/>
   <xacro:arg name="ros2_control" default="gazebo"/>
+  <xacro:arg name="roller" default="false"/>
   <!-- Dual lidar option when only SIMULATION
   real robot force to be dual_lidar
@@ -38,20 +39,20 @@
   <!-- Wheel -->
   <!-- 1st wheel -->
-  <xacro:wheel_v0 prefix="bl" parent="base_link">
+  <xacro:wheel_v0 prefix="bl" parent="base_link" roller="$(arg roller)">
     <origin xyz="0.130943 0.130943 0.05" rpy="0 0 -${M_PI/4}"/>
     <axis xyz="0.0 1.0 0.0"/>
   </xacro:wheel_v0>
   <!-- 2nd wheel -->
-  <xacro:wheel_v0 prefix="br" parent="base_link">
+  <xacro:wheel_v0 prefix="br" parent="base_link" roller="$(arg roller)">
     <origin xyz="-0.130943 0.130943 0.05" rpy="0 0 ${M_PI/4}"/>
     <axis xyz="0.0 1.0 0.0"/>
   </xacro:wheel_v0>
   <!-- 3rd wheel -->
-  <xacro:wheel_v0 prefix="fr" parent="base_link">
+  <xacro:wheel_v0 prefix="fr" parent="base_link" roller="$(arg roller)">
     <origin xyz="-0.130943 -0.130943 0.05" rpy="0 0 ${3*M_PI/4}"/>
     <axis xyz="0.0 1.0 0.0"/>
   </xacro:wheel_v0>
   <!-- 4th wheel -->
-  <xacro:wheel_v0 prefix="fl" parent="base_link">
+  <xacro:wheel_v0 prefix="fl" parent="base_link" roller="$(arg roller)">
     <origin xyz="0.130943 -0.130943 0.05" rpy="0 0 ${5*M_PI/4}"/>
     <axis xyz="0.0 1.0 0.0"/>

File: urdf/walkie/omni_wheel/gz_omni_wheel.urdf.xacro (robot description, xacro)
@@ -4,4 +4,5 @@
   <xacro:arg name="prefix" default="wheel" />
   <xacro:arg name="parent" default="base_link" />
+  <xacro:arg name="roller" default="false" />
 	<xacro:include
     filename="$(find walkie_description)/urdf/inertial_macros.xacro"
@@ -19,5 +20,5 @@
 	<xacro:property name="wheel_radian" value="0.075" />
 	<xacro:property name="wheel_mass" value="0.05" />
-	<xacro:macro name="wheel_v0" params="prefix parent *joint_origin *joint_axis">
+	<xacro:macro name="wheel_v0" params="prefix parent roller:=^|$(arg roller) *joint_origin *joint_axis">
   	<joint name="${prefix}_wheel_joint" type="continuous">
   		<xacro:insert_block name="joint_origin" />
@@ -44,8 +45,16 @@
   			<origin xyz="0 0 0" rpy="1.570796327 0 0" />
   		</xacro:inertial_cylinder>
-  		<!-- <collision><origin xyz="0 0 0" rpy="1.570796327 0 0" /><geometry><cylinder radius="${wheel_radian}" length="${wheel_thickness}" /></geometry></collision> -->
+  		<xacro:unless value="${roller}">
+  			<collision>
+  				<origin xyz="0 0 0" rpy="1.570796327 0 0" />
+  				<geometry>
+  					<cylinder radius="${wheel_radian}" length="${wheel_thickness}" />
+  				</geometry>
+  			</collision>
+  		</xacro:unless>
   	</link>
   	<xacro:wheel_gazebo_v0 prefix="${prefix}" />
   	<!-- Individual Roller Joint and Link Instantiations -->
+  	<xacro:if value="${roller}">
   	<xacro:roller prefix="${prefix}" num="1">
   		<origin xyz="0.067000 -0.009500 0.000000" rpy="0.000000 -0.000000 0.000000" />
@@ -160,9 +169,10 @@
   		<axis xyz="0.000000 0.000000 1.000000" />
   	</xacro:roller>
+  	</xacro:if>
 	</xacro:macro>
   <!-- Standalone Wheel Instantiation for testing & export -->
   <xacro:if value="$(arg standalone)">
     <link name="$(arg parent)" />
-    <xacro:wheel_v0 prefix="$(arg prefix)" parent="$(arg parent)">
+    <xacro:wheel_v0 prefix="$(arg prefix)" parent="$(arg parent)" roller="$(arg roller)">
       <origin xyz="0 0 0" rpy="0 0 0" />
       <axis xyz="0 1 0" />

Commit message: feat: add lift at top option argument

File: robots/gz_walkie.urdf.xacro (robot description, xacro)
@@ -4,4 +4,5 @@
   <xacro:arg name="ros2_control" default="gazebo"/>
   <xacro:arg name="roller" default="false"/>
+  <xacro:arg name="lift_at_top" default="false"/>
   <!-- Dual lidar option when only SIMULATION
   real robot force to be dual_lidar
@@ -34,7 +35,14 @@
   <xacro:base_gazebo_v0/>
   <!-- Lift -->
-  <xacro:lift_v0 prefix="lift" parent="base_link">
-    <origin xyz="0.00000 0.07000 0.3985" rpy="0 0 0"/>
-  </xacro:lift_v0>
+  <xacro:if value="$(arg lift_at_top)">
+    <xacro:lift_v0 prefix="lift" parent="base_link" lift_at_top="true">
+      <origin xyz="0.00000 0.07000 1.1420" rpy="0 0 0"/>
+    </xacro:lift_v0>
+  </xacro:if>
+  <xacro:unless value="$(arg lift_at_top)">
+    <xacro:lift_v0 prefix="lift" parent="base_link" lift_at_top="false">
+      <origin xyz="0.00000 0.07000 0.3985" rpy="0 0 0"/>
+    </xacro:lift_v0>
+  </xacro:unless>
   <!-- Wheel -->
   <!-- 1st wheel -->
@@ -118,4 +126,5 @@
     right_can_interface="$(arg right_can_interface)"
     hand="true"
+    lift_at_top="$(arg lift_at_top)"
     control_gains="${xacro.load_yaml('$(find walkie_description)/config/openarm/arm/v10/control_gains.yaml')}"
   />

Commit message: refactor(description): remove base_link yaw rotation patch and align forward frame to +X
- Remove hardcoded rpy="0 0 ${M_PI/2}" patch between base_footprint and
base_link
- Reorient base_link to natively follow ROS REP-103 standard (+X
torward, +Y left, +Z up)
- Update base_link visual mesh orientation and collision bounding boxes
- Transform origins and orientations of all joints attached to base_link
(lift, omni wheels, lidars, depth camera, and Unitree 4D lidar) to
preserve exact physical geometry

File: robots/gz_walkie.urdf.xacro (robot description, xacro)
@@ -31,5 +31,5 @@
   <link name="base_footprint"/>
   <xacro:base_v0 parent="base_footprint">
-    <origin xyz="0 0 0.0312" rpy="0 0 ${M_PI / 2}"/>
+    <origin xyz="0 0 0.0312" rpy="0 0 0"/>
   </xacro:base_v0>
   <xacro:base_gazebo_v0/>
@@ -37,10 +37,10 @@
   <xacro:if value="$(arg lift_at_top)">
     <xacro:lift_v0 prefix="lift" parent="base_link" lift_at_top="true">
-      <origin xyz="0.00000 0.07000 1.1420" rpy="0 0 0"/>
+      <origin xyz="-0.07000 0.00000 1.1420" rpy="0 0 ${M_PI / 2}"/>
     </xacro:lift_v0>
   </xacro:if>
   <xacro:unless value="$(arg lift_at_top)">
     <xacro:lift_v0 prefix="lift" parent="base_link" lift_at_top="false">
-      <origin xyz="0.00000 0.07000 0.3985" rpy="0 0 0"/>
+      <origin xyz="-0.07000 0.00000 0.3985" rpy="0 0 ${M_PI / 2}"/>
     </xacro:lift_v0>
   </xacro:unless>
@@ -48,20 +48,20 @@
   <!-- 1st wheel -->
   <xacro:wheel_v0 prefix="bl" parent="base_link" roller="$(arg roller)">
-    <origin xyz="0.130943 0.130943 0.05" rpy="0 0 -${M_PI/4}"/>
+    <origin xyz="-0.130943 0.130943 0.05" rpy="0 0 ${M_PI/4}"/>
     <axis xyz="0.0 1.0 0.0"/>
   </xacro:wheel_v0>
   <!-- 2nd wheel -->
   <xacro:wheel_v0 prefix="br" parent="base_link" roller="$(arg roller)">
-    <origin xyz="-0.130943 0.130943 0.05" rpy="0 0 ${M_PI/4}"/>
+    <origin xyz="-0.130943 -0.130943 0.05" rpy="0 0 ${3*M_PI/4}"/>
     <axis xyz="0.0 1.0 0.0"/>
   </xacro:wheel_v0>
   <!-- 3rd wheel -->
   <xacro:wheel_v0 prefix="fr" parent="base_link" roller="$(arg roller)">
-    <origin xyz="-0.130943 -0.130943 0.05" rpy="0 0 ${3*M_PI/4}"/>
+    <origin xyz="0.130943 -0.130943 0.05" rpy="0 0 ${5*M_PI/4}"/>
     <axis xyz="0.0 1.0 0.0"/>
   </xacro:wheel_v0>
   <!-- 4th wheel -->
   <xacro:wheel_v0 prefix="fl" parent="base_link" roller="$(arg roller)">
-    <origin xyz="0.130943 -0.130943 0.05" rpy="0 0 ${5*M_PI/4}"/>
+    <origin xyz="0.130943 0.130943 0.05" rpy="0 0 -${M_PI/4}"/>
     <axis xyz="0.0 1.0 0.0"/>
   </xacro:wheel_v0>
@@ -70,5 +70,5 @@
   <xacro:if value="${'$(arg ros2_control)' == 'gazebo' and not $(arg dual_lidar)}">
     <xacro:lidar_v0 prefix="single" parent="base_link">
-      <origin xyz="0 0 0.315" rpy="0 0 -1.5707963"/>
+      <origin xyz="0 0 0.315" rpy="0 0 0"/>
     </xacro:lidar_v0>
     <xacro:lidar_gazebo_v0 prefix="single" min_rad="-${M_PI}" max_rad=" ${M_PI}" min_range="0.6" max_range="10" yaw_offset="0"/>
@@ -77,8 +77,8 @@
   <xacro:unless value="${'$(arg ros2_control)' == 'gazebo' and not $(arg dual_lidar)}">
     <xacro:lidar_v0 prefix="front" parent="base_link">
-      <origin xyz="0 -0.235 0.28232" rpy="0 0 -1.5707963"/>
+      <origin xyz="0.235 0 0.28232" rpy="0 0 0"/>
     </xacro:lidar_v0>
     <xacro:lidar_v0 prefix="back" parent="base_link">
-      <origin xyz="0 0.235 0.28232" rpy="0 0 1.5707963"/>
+      <origin xyz="-0.235 0 0.28232" rpy="0 0 ${M_PI}"/>
     </xacro:lidar_v0>
     <xacro:lidar_gazebo_v0 prefix="front" min_rad="-2.09333333" max_rad=" 2.09333333" min_range="0.18" max_range="10" yaw_offset="0"/>
@@ -96,5 +96,5 @@
     <parent link="base_link"/>
     <child link="unitree4d_l2_imu_initial"/>
-    <origin xyz="0 0.05196152 1.676" rpy="3.36159 -0.445 1.09"/>
+    <origin xyz="-0.05196152 0 1.676" rpy="3.36159 -0.445 2.6607963"/>
   </joint>
   <link name="unitree4d_l2_imu"/>
@@ -106,5 +106,5 @@
   <!-- depth cam sensor -->
   <xacro:sensor_d415 name="bottom" parent="base_link" flag_color="1" flag_ir="0" flag_depth="1" updaterate="2">
-    <origin xyz="0 -0.27386242 0.18004809" rpy="0 -0.872664626  -${M_PI/2}"/>
+    <origin xyz="0.27386242 0 0.18004809" rpy="0 -0.872664626 0"/>
   </xacro:sensor_d415>
   <!-- head servo -->

Commit message: feat(ros2_control): add mujoco hardware branch and controller config
Add ros2_control:=mujoco, backed by mujoco_ros2_control/MujocoSystemInterface
(params checked against the 0.1.2 package on robostack-jazzy). Wheels expose a
velocity command interface only; arm, gripper, lift and head joints expose
position only, matching the actuator types in the generated MJCF. Mimic finger
joints are left to MJCF equality constraints. The top_imu sensor maps to the
MJCF top_imu_{quat,gyro,accel} sensors.

New xacro args: mujoco_model (defaults to the installed mujoco/scene.xml) and
mujoco_headless. Other modes expand byte-identical to before.

mujoco_controllers.yaml is sim_controllers.yaml without the arm forward
velocity controllers (MuJoCo arms are position-driven) plus an
imu_sensor_broadcaster for top_imu.

File: robots/gz_walkie.urdf.xacro (robot description, xacro)
@@ -16,4 +16,9 @@
   <xacro:arg name="left_can_interface" default="can1"/>
   <xacro:arg name="right_can_interface" default="can0"/>
+  <!-- MuJoCo simulation only (ros2_control:=mujoco): scene loaded by the
+       hardware plugin, and whether to run without the Simulate window -->
+  <xacro:arg name="mujoco_model"
+             default="$(find walkie_description)/mujoco/scene.xml"/>
+  <xacro:arg name="mujoco_headless" default="false"/>
   <xacro:include filename="$(find walkie_description)/urdf/walkie/base/base.urdf.xacro"/>
   <xacro:include filename="$(find walkie_description)/urdf/walkie/omni_wheel/gz_omni_wheel.urdf.xacro"/>
@@ -116,4 +121,6 @@
     left_can_interface="$(arg left_can_interface)"
     right_can_interface="$(arg right_can_interface)"
+    mujoco_model="$(arg mujoco_model)"
+    mujoco_headless="$(arg mujoco_headless)"
     hand="true"
     control_gains="${xacro.load_yaml('$(find walkie_description)/config/openarm/arm/v10/control_gains.yaml')}"

File: urdf/walkie/ros2_control.xacro (robot description, xacro)
@@ -74,4 +74,32 @@
     </joint>
   </xacro:macro>
+  <!-- Sub-macro: Wheel joint driven by a MuJoCo velocity actuator (mujoco).
+       Exposes only the velocity command interface; the MJCF actuator must share the joint name. -->
+  <xacro:macro name="mujoco_wheel_joint" params="name vel_min vel_max">
+    <joint name="${name}">
+      <command_interface name="velocity">
+        <param name="min">${vel_min}</param>
+        <param name="max">${vel_max}</param>
+      </command_interface>
+      <state_interface name="position" />
+      <state_interface name="velocity" />
+    </joint>
+  </xacro:macro>
+  <!-- Sub-macro: Arm/gripper joint driven by a MuJoCo position actuator (mujoco).
+       Exposes only the position command interface; the MJCF actuator must share the joint name. -->
+  <xacro:macro name="mujoco_position_arm_joint" params="joint_name initial_position:=0.0">
+    <joint name="${joint_name}">
+      <command_interface name="position" />
+      <state_interface name="position">
+        <param name="initial_value">${initial_position}</param>
+      </state_interface>
+      <state_interface name="velocity">
+        <param name="initial_value">0.0</param>
+      </state_interface>
+      <state_interface name="effort">
+        <param name="initial_value">0.0</param>
+      </state_interface>
+    </joint>
+  </xacro:macro>
   <!-- Main Macro Declaration (ros2_control included back into parameters list) -->
   <xacro:macro name="ros2_control"
@@ -88,5 +116,7 @@
                 can_fd:=^|true
                 right_joint2_fixed:=^|false
-                sim_controllers_yaml">
+                sim_controllers_yaml
+                mujoco_model:=^|''
+                mujoco_headless:=^|false">
     <!-- Mock hardware -->
     <xacro:if value="${ros2_control == 'mock'}">
@@ -228,4 +258,93 @@
       </ros2_control>
     </xacro:if>
+    <!-- Simulation - MuJoCo based ros2_control (mujoco_ros2_control).
+         Every commanded joint below must have an MJCF actuator with the same name:
+         velocity actuators for the wheels, position actuators for everything else.
+         Mimic joints (openarm_*_finger_joint2) are not listed; the MJCF couples them
+         to openarm_*_finger_joint1 through equality constraints. -->
+    <xacro:if value="${ros2_control == 'mujoco'}">
+      <ros2_control name="MujocoSystem" type="system">
+        <hardware>
+          <plugin>mujoco_ros2_control/MujocoSystemInterface</plugin>
+          <param name="mujoco_model">${mujoco_model}</param>
+          <param name="headless">${'true' if mujoco_headless else 'false'}</param>
+          <!-- Ground-truth pose of the free-floating base (nav_msgs/Odometry, no TF) -->
+          <param name="odom_free_joint_name">floating_base_joint</param>
+          <param name="odom_topic">/mujoco_ground_truth/odom</param>
+        </hardware>
+        <xacro:mujoco_wheel_joint
+                    name="fl_wheel_joint"
+                    vel_min="-3.14"
+                    vel_max="3.14"
+                />
+        <xacro:mujoco_wheel_joint
+                    name="fr_wheel_joint"
+                    vel_min="-3.14"
+                    vel_max="3.14"
+                />
+        <xacro:mujoco_wheel_joint
+                    name="br_wheel_joint"
+                    vel_min="-3.14"
+                    vel_max="3.14"
+                />
+        <xacro:mujoco_wheel_joint
+                    name="bl_wheel_joint"
+                    vel_min="-3.14"
+                    vel_max="3.14"
+                />
+        <joint name="head_servo_joint">
+          <command_interface name="position">
+            <param name="min">-1.54</param>
+            <param name="max">1.54</param>
+          </command_interface>
+          <state_interface name="position" />
+          <state_interface name="velocity" />
+        </joint>
+        <joint name="lift_joint">
+          <command_interface name="position">
+            <param name="min">0.000</param>
+            <param name="max">0.743</param>
+          </command_interface>
+          <state_interface name="position">
+            <param name="initial_value">0.51</param>
+          </state_interface>
+          <state_interface name="velocity" />
+        </joint>
+        <xacro:mujoco_position_arm_joint joint_name="openarm_left_joint1" initial_position="0.2618" />
+        <xacro:mujoco_position_arm_joint joint_name="openarm_left_joint2" />
+        <xacro:mujoco_position_arm_joint joint_name="openarm_left_joint3" />
+        <xacro:mujoco_position_arm_joint joint_name="openarm_left_joint4" initial_position="0.2618" />
+        <xacro:mujoco_position_arm_joint joint_name="openarm_left_joint5" />
+        <xacro:mujoco_position_arm_joint joint_name="openarm_left_joint6" />
+        <xacro:mujoco_position_arm_joint joint_name="openarm_left_joint7" />
+        <xacro:mujoco_position_arm_joint joint_name="openarm_right_joint1" initial_position="-0.2618" />
+        <xacro:unless value="${right_joint2_fixed}">
+          <xacro:mujoco_position_arm_joint joint_name="openarm_right_joint2" />
+        </xacro:unless>
+        <xacro:mujoco_position_arm_joint joint_name="openarm_right_joint3" />
+        <xacro:mujoco_position_arm_joint joint_name="openarm_right_joint4" initial_position="0.2618" />
+        <xacro:mujoco_position_arm_joint joint_name="openarm_right_joint5" />
+        <xacro:mujoco_position_arm_joint joint_name="openarm_right_joint6" />
+        <xacro:mujoco_position_arm_joint joint_name="openarm_right_joint7" />
+        <xacro:mujoco_position_arm_joint joint_name="openarm_left_finger_joint1" />
+        <xacro:mujoco_position_arm_joint joint_name="openarm_right_finger_joint1" />
+        <!-- IMU: reads the MJCF sensors top_imu_quat, top_imu_gyro and top_imu_accel
+             attached to the top_imu site (frame of top_imu_link). -->
+        <sensor name="top_imu">
+          <param name="mujoco_type">imu</param>
+          <param name="mujoco_sensor_name">top_imu</param>
+          <state_interface name="orientation.x" />
+          <state_interface name="orientation.y" />
+          <state_interface name="orientation.z" />
+          <state_interface name="orientation.w" />
+          <state_interface name="angular_velocity.x" />
+          <state_interface name="angular_velocity.y" />
+          <state_interface name="angular_velocity.z" />
+          <state_interface name="linear_acceleration.x" />
+          <state_interface name="linear_acceleration.y" />
+          <state_interface name="linear_acceleration.z" />
+        </sensor>
+      </ros2_control>
+    </xacro:if>
     <!-- Isaac Sim / MicroROS : Topic based ros2_control -->
     <xacro:if value="${ros2_control == 'topic_base'}">

Commit message: fix(lidar): align unitree 3D lidar forward pose for simulation (topic_base/gazebo)

File: robots/gz_walkie.urdf.xacro (robot description, xacro)
@@ -101,5 +101,10 @@
     <parent link="base_link"/>
     <child link="unitree4d_l2_imu_initial"/>
-    <origin xyz="-0.05196152 0 1.676" rpy="3.36159 -0.445 2.6607963"/>
+    <xacro:if value="${'$(arg ros2_control)' == 'topic_base' or '$(arg ros2_control)' == 'gazebo'}">
+      <origin xyz="-0.05196152 0 1.676" rpy="${-M_PI} -0.488692 0"/>
+    </xacro:if>
+    <xacro:unless value="${'$(arg ros2_control)' == 'topic_base' or '$(arg ros2_control)' == 'gazebo'}">
+      <origin xyz="-0.05196152 0 1.676" rpy="3.36159 -0.445 2.6607963"/>
+    </xacro:unless>
   </joint>
   <link name="unitree4d_l2_imu"/>

Commit message: fix(lidar): correct 3D lidar pitch and yaw orientation for simulation

File: robots/gz_walkie.urdf.xacro (robot description, xacro)
@@ -102,5 +102,5 @@
     <child link="unitree4d_l2_imu_initial"/>
     <xacro:if value="${'$(arg ros2_control)' == 'topic_base' or '$(arg ros2_control)' == 'gazebo'}">
-      <origin xyz="-0.05196152 0 1.676" rpy="${-M_PI} -0.488692 0"/>
+      <origin xyz="-0.05196152 0 1.676" rpy="${M_PI} 0.488692 0.98"/>
     </xacro:if>
     <xacro:unless value="${'$(arg ros2_control)' == 'topic_base' or '$(arg ros2_control)' == 'gazebo'}">

Commit message: fix(lidar): set 3D lidar simulation yaw to 0 for proper forward alignment

File: robots/gz_walkie.urdf.xacro (robot description, xacro)
@@ -102,5 +102,5 @@
     <child link="unitree4d_l2_imu_initial"/>
     <xacro:if value="${'$(arg ros2_control)' == 'topic_base' or '$(arg ros2_control)' == 'gazebo'}">
-      <origin xyz="-0.05196152 0 1.676" rpy="${M_PI} 0.488692 0.98"/>
+      <origin xyz="-0.05196152 0 1.676" rpy="${M_PI} 0.488692 0"/>
     </xacro:if>
     <xacro:unless value="${'$(arg ros2_control)' == 'topic_base' or '$(arg ros2_control)' == 'gazebo'}">
