Commit message: fix: add gear_ratio args in gripper urdf

File: urdf/walkie-gripper/walkie_gripper.urdf.xacro (robot description, xacro)
@@ -7,4 +7,5 @@
   <xacro:property name="worm_joint_effort" value="20.0" />
   <xacro:property name="worm_joint_velocity" value="2.0" />
+  <xacro:property name="worm_gear_ratio" value="0.1" />
   <xacro:macro name="gripper_link_inertial" params="mass">
     <inertial>
@@ -73,5 +74,5 @@
     <joint name="${prefix}_gripper_gear_r" type="revolute">
       <limit lower="-3.14" upper="3.14" effort="${joint_effort}" velocity="${joint_velocity}"/>
-      <mimic multiplier="0.1" offset="0" joint="${prefix}_gripper_worm_gear"/>
+      <mimic multiplier="${worm_gear_ratio}" offset="0" joint="${prefix}_gripper_worm_gear"/>
       <origin rpy="0.0 0.0 0.0" xyz="-0.03240 -0.00100 -0.05335"/>
       <parent link="${prefix}_link7"/>
