Commit message: refactor: new mesh

File: urdf/walkie-gripper/walkie_gripper.urdf.xacro (robot description, xacro)
@@ -1,19 +1,10 @@
 <?xml version="1.0" ?>
 <robot xmlns:xacro="http://www.ros.org/wiki/xacro">
-  <!-- Joint properties -->
   <xacro:property name="joint_effort" value="10.0" />
   <xacro:property name="joint_velocity" value="1.0" />
   <xacro:property name="joint_damping" value="0.1" />
   <xacro:property name="joint_friction" value="0.1" />
-  <!-- Worm gear joint properties -->
   <xacro:property name="worm_joint_effort" value="20.0" />
   <xacro:property name="worm_joint_velocity" value="2.0" />
-  <xacro:property name="worm_gear_ratio" value="0.1" />
-  <!-- Inertial properties -->
-  <xacro:property name="base_mass" value="0.1" />
-  <xacro:property name="link_mass" value="0.01" />
-  <xacro:property name="grip_mass" value="0.015" />
-  <xacro:property name="worm_mass" value="0.02" />
-  <!-- Generic inertial macro -->
   <xacro:macro name="gripper_link_inertial" params="mass">
     <inertial>
@@ -23,285 +14,170 @@
     </inertial>
   </xacro:macro>
-  <!-- Material definitions -->
-  <material name="walkie_acetal_resin_white">
-    <color rgba="0.97255 0.96471 0.92941 1.00000" />
-  </material>
   <material name="walkie_aluminum_polished">
-    <color rgba="0.95686 0.96078 0.96471 1.00000" />
-  </material>
-  <material name="walkie_opaque_gray">
-    <color rgba="0.79216 0.79216 0.79216 1.00000" />
+    <color rgba="0.95686 0.96078 0.96471 1.0" />
   </material>
   <material name="walkie_opaque_gold">
-    <color rgba="0.83137 0.66667 0.12941 1.00000" />
+    <color rgba="0.83137 0.66667 0.12941 1.0" />
   </material>
-  <!-- Main gripper macro -->
-  <xacro:macro name="walkie_gripper" params="parent prefix *origin">
-    <!-- Base link -->
-    <link name="${prefix}_gripper_base">
-      <xacro:gripper_link_inertial mass="${base_mass}" />
-      <visual name="${prefix}_base">
-        <material name="walkie_acetal_resin_white" />
+  <xacro:macro name="walkie_gripper" params="parent prefix">
+    <joint name="${prefix}_joint7" type="revolute">
+      <axis xyz="0.0 0.0 -1.0" />
+      <limit effort="30.0" lower="-3.14" upper="3.14" velocity="2.0" />
+      <parent link="${parent}" /> <child link="${prefix}_link7" />
+      <origin xyz="0.0 0.02800 -0.13825" rpy="0.0 0.0 0.0" />
+      <dynamics damping="${joint_damping}" friction="${joint_friction}" />
+    </joint>
+    <link name="${prefix}_link7">
+      <visual>
+        <material name="walkie_opaque_gold" />
+        <origin rpy="0.0 0.0 0.0" xyz="0.0 0.02116 -0.03906" />
+        <geometry>
+          <mesh filename="package://walkie_description/meshes/walkie-gripper/stl/Body1.121.stl" scale="1 1 1"/>
+        </geometry>
+      </visual>
+      <collision>
+        <origin rpy="0.0 0.0 0.0" xyz="0.0 0.0 -0.03004"/>
+        <geometry>
+          <box size="0.12520 0.05916 0.05330"/>
+        </geometry>
+      </collision>
+      <xacro:gripper_link_inertial mass="0.2" />
+    </link>
+    <link name="${prefix}_gripper_worm_gear">
+      <xacro:gripper_link_inertial mass="0.02" />
+      <visual>
+        <material name="walkie_aluminum_polished" />
         <origin rpy="0.0 0.0 0.0" xyz="0.0 0.0 0.0" />
         <geometry>
-          <mesh
-                        filename="package://walkie_description/meshes/walkie-gripper/dae/Body1.523.dae"
-                        scale="0.01 0.01 0.01"
-                    />
+          <mesh filename="package://walkie_description/meshes/walkie-gripper/stl/Body1.133.stl" scale="1 1 1"/>
         </geometry>
       </visual>
     </link>
-    <!-- Joint connecting gripper to parent -->
-    <joint name="${prefix}_${parent}_to_${prefix}_gripper_base" type="fixed">
-      <parent link="${prefix}_${parent}" />
-      <child link="${prefix}_gripper_base" />
-      <xacro:insert_block name="origin" />
+    <joint name="${prefix}_gripper_worm_gear" type="revolute">
+      <limit lower="-15.7" upper="3.14" effort="${worm_joint_effort}" velocity="${worm_joint_velocity}"/>
+      <origin rpy="0.0 0.0 0.0" xyz="0.0 0.0 -0.00275"/>
+      <parent link="${prefix}_link7"/>
+      <child link="${prefix}_gripper_worm_gear"/>
+      <axis xyz="0.0 0.0 -1.0"/>
+      <dynamics damping="${joint_damping}" friction="${joint_friction}" />
     </joint>
-    <!-- Worm gear link -->
-    <link name="${prefix}_worm_gear">
-      <xacro:gripper_link_inertial mass="${worm_mass}" />
-      <visual name="${prefix}_worm_gear_visual">
+    <link name="${prefix}_gripper_gear_r">
+      <xacro:gripper_link_inertial mass="0.01" />
+      <visual>
         <material name="walkie_aluminum_polished" />
-        <origin rpy="0.0 0.0 -0.07392" xyz="0.0 0.0 0.00147" />
         <geometry>
-          <mesh
-                        filename="package://walkie_description/meshes/walkie-gripper/dae/Body1.522.dae"
-                        scale="0.01 0.01 0.01"
-                    />
+          <mesh filename="package://walkie_description/meshes/walkie-gripper/stl/Body1.113.stl" scale="1 1 1"/>
         </geometry>
       </visual>
     </link>
-    <!-- Worm gear joint (main controller) -->
-    <joint name="${prefix}_gripper_controller" type="revolute">
-      <limit
-                lower="-31.4"
-                upper="31.4"
-                effort="${worm_joint_effort}"
-                velocity="${worm_joint_velocity}"
-            />
-      <origin rpy="-3.14159 0.0 -3.14159" xyz="-0.00033 0.0013 0.00032" />
-      <parent link="${prefix}_gripper_base" />
-      <child link="${prefix}_worm_gear" />
-      <axis xyz="0.0 0.0 1.0" />
+    <joint name="${prefix}_gripper_gear_r" type="revolute">
+      <limit lower="-3.14" upper="3.14" effort="${joint_effort}" velocity="${joint_velocity}"/>
+      <mimic multiplier="0.1" offset="0" joint="${prefix}_gripper_worm_gear"/>
+      <origin rpy="0.0 0.0 0.0" xyz="-0.03240 -0.00100 -0.05335"/>
+      <parent link="${prefix}_link7"/>
+      <child link="${prefix}_gripper_gear_r"/>
+      <axis xyz="0.0 -1.0 0.0"/>
       <dynamics damping="${joint_damping}" friction="${joint_friction}" />
     </joint>
-    <!-- Right side links -->
-    <link name="${prefix}_gripper_right1">
-      <xacro:gripper_link_inertial mass="${link_mass}" />
-      <visual name="${prefix}_r_link1_visual">
+    <link name="${prefix}_gripper_gear_l">
+      <xacro:gripper_link_inertial mass="0.01" />
+      <visual>
         <material name="walkie_aluminum_polished" />
-        <origin rpy="0.0 0.0 0.1658" xyz="0.0 0.0 0.0" />
         <geometry>
-          <mesh
-                        filename="package://walkie_description/meshes/walkie-gripper/dae/Body1.415.dae"
-                        scale="0.01 0.01 0.01"
-                    />
+          <mesh filename="package://walkie_description/meshes/walkie-gripper/stl/Body1.007.stl" scale="1 1 1"/>
         </geometry>
       </visual>
     </link>
-    <link name="${prefix}_gripper_right2">
-      <xacro:gripper_link_inertial mass="${grip_mass}" />
-      <collision name="${prefix}_r_grip_collision">
-        <origin rpy="0.0 0.00006 0.0" xyz="-0.00864 0.04813 -0.00318" />
+    <joint name="${prefix}_gripper_gear_l" type="revolute">
+      <limit lower="-3.14" upper="3.14" effort="${joint_effort}" velocity="${joint_velocity}"/>
+      <mimic multiplier="-0.1" offset="0" joint="${prefix}_gripper_worm_gear"/>
+      <origin rpy="0.0 0.0 0.0" xyz="0.03240 -0.00100 -0.05335"/>
+      <parent link="${prefix}_link7"/>
+      <child link="${prefix}_gripper_gear_l"/>
+      <axis xyz="0.0 -1.0 0.0"/>
+      <dynamics damping="${joint_damping}" friction="${joint_friction}" />
+    </joint>
+    <link name="${prefix}_gripper_hand_r">
+      <xacro:gripper_link_inertial mass="0.015" />
+      <collision>
+        <origin rpy="0.0 0.0 0.0" xyz="-0.00904 0.0 -0.04823"/>
         <geometry>
-          <box size="0.03009 0.16753 0.01" />
+          <box size="0.03010 0.01000 0.16753"/>
         </geometry>
       </collision>
-      <visual name="${prefix}_r_grip_visual">
+      <visual>
         <material name="walkie_opaque_gold" />
-        <origin rpy="-1.5708 0.0 -0.00006" xyz="0.0 0.0 0.0" />
         <geometry>
-          <mesh
-                        filename="package://walkie_description/meshes/walkie-gripper/dae/Body1.411.dae"
-                        scale="0.01 0.01 0.01"
-                    />
+          <mesh filename="package://walkie_description/meshes/walkie-gripper/stl/Body1.123.stl" scale="1 1 1"/>
         </geometry>
       </visual>
     </link>
-    <link name="${prefix}_gripper_right3">
-      <xacro:gripper_link_inertial mass="${link_mass}" />
-      <visual name="${prefix}_r_link2_visual">
-        <material name="walkie_opaque_gray" />
-        <origin rpy="0.0 0.0 0.16896" xyz="0.0 0.0 0.0" />
+    <joint name="${prefix}_gripper_hand_r" type="revolute">
+      <limit lower="-3.14" upper="3.14" effort="${joint_effort}" velocity="${joint_velocity}"/>
+      <mimic multiplier="-1.0" offset="0" joint="${prefix}_gripper_gear_r"/>
+      <origin rpy="0.0 0.0 0.0" xyz="0.00896 0.00100 -0.06579"/>
+      <parent link="${prefix}_gripper_gear_r"/>
+      <child link="${prefix}_gripper_hand_r"/>
+      <axis xyz="0.0 -1.0 0.0"/>
+      <dynamics damping="${joint_damping}" friction="${joint_friction}" />
+    </joint>
+    <link name="${prefix}_gripper_hand_l">
+      <xacro:gripper_link_inertial mass="0.015" />
+      <collision>
+        <origin rpy="0.0 0.0 0.0" xyz="0.00904 0.0 -0.04823"/>
         <geometry>
-          <mesh
-                        filename="package://walkie_description/meshes/walkie-gripper/dae/Body1.405.dae"
-                        scale="0.01 0.01 0.01"
-                    />
+          <box size="0.03010 0.01000 0.16753"/>
+        </geometry>
+      </collision>
+      <visual>
+        <material name="walkie_opaque_gold" />
+        <geometry>
+          <mesh filename="package://walkie_description/meshes/walkie-gripper/stl/Body1.046.stl" scale="1 1 1"/>
         </geometry>
       </visual>
     </link>
-    <!-- Left side links -->
-    <link name="${prefix}_gripper_left1">
-      <xacro:gripper_link_inertial mass="${link_mass}" />
-      <visual name="${prefix}_l_link1_visual">
+    <joint name="${prefix}_gripper_hand_l" type="revolute">
+      <limit lower="-3.14" upper="3.14" effort="${joint_effort}" velocity="${joint_velocity}"/>
+      <mimic multiplier="-1.0" offset="0" joint="${prefix}_gripper_gear_l"/>
+      <origin rpy="0.0 0.0 0.0" xyz="-0.00896 0.00100 -0.06579"/>
+      <parent link="${prefix}_gripper_gear_l"/>
+      <child link="${prefix}_gripper_hand_l"/>
+      <axis xyz="0.0 -1.0 0.0"/>
+      <dynamics damping="${joint_damping}" friction="${joint_friction}" />
+    </joint>
+    <link name="${prefix}_gripper_connector_r">
+      <xacro:gripper_link_inertial mass="0.01" />
+      <visual>
         <material name="walkie_aluminum_polished" />
-        <origin rpy="0.0 0.0 0.1658" xyz="0.0 0.0 0.0" />
         <geometry>
-          <mesh
-                        filename="package://walkie_description/meshes/walkie-gripper/dae/Body1.007.dae"
-                        scale="-0.01 -0.01 -0.01"
-                    />
+          <mesh filename="package://walkie_description/meshes/walkie-gripper/stl/Body1.019.stl" scale="1 1 1"/>
         </geometry>
       </visual>
     </link>
-    <link name="${prefix}_gripper_left2">
-      <xacro:gripper_link_inertial mass="${grip_mass}" />
-      <collision name="${prefix}_l_grip_collision">
-        <origin rpy="0.0 0.0 0.0" xyz="0.00884 0.04813 -0.00318" />
+    <joint name="${prefix}_gripper_connector_r" type="revolute">
+      <limit lower="-3.14" upper="3.14" effort="${joint_effort}" velocity="${joint_velocity}"/>
+      <mimic multiplier="-1.0" offset="0" joint="${prefix}_gripper_hand_r"/>
+      <origin rpy="0.0 0.0 0.0" xyz="-0.01742 0.0 0.02955"/>
+      <parent link="${prefix}_gripper_hand_r"/>
+      <child link="${prefix}_gripper_connector_r"/>
+      <axis xyz="0.0 -1.0 0.0"/>
+      <dynamics damping="${joint_damping}" friction="${joint_friction}" />
+    </joint>
+    <link name="${prefix}_gripper_connector_l">
+      <xacro:gripper_link_inertial mass="0.01" />
+      <visual>
+        <material name="walkie_aluminum_polished" />
         <geometry>
-          <box size="0.03009 0.16753 0.01" />
-        </geometry>
-      </collision>
-      <visual name="${prefix}_l_grip_visual">
-        <material name="walkie_opaque_gold" />
-        <origin rpy="1.5708 -0.00006 0.00006" xyz="0.0 0.0 0.0" />
-        <geometry>
-          <mesh
-                        filename="package://walkie_description/meshes/walkie-gripper/dae/Body1.006.dae"
-                        scale="-0.01 -0.01 -0.01"
-                    />
+          <mesh filename="package://walkie_description/meshes/walkie-gripper/stl/Body1.003.stl" scale="1 1 1"/>
         </geometry>
       </visual>
     </link>
-    <link name="${prefix}_gripper_left3">
-      <xacro:gripper_link_inertial mass="${link_mass}" />
-      <visual name="${prefix}_l_link2_visual">
-        <material name="walkie_opaque_gray" />
-        <origin rpy="0.02363 0.13763 0.17059" xyz="0.0 0.0 0.0" />
-        <geometry>
-          <mesh
-                        filename="package://walkie_description/meshes/walkie-gripper/dae/Body1.005.dae"
-                        scale="-0.01 -0.01 -0.01"
-                    />
-        </geometry>
-      </visual>
-    </link>
-    <!-- Right side joints -->
-    <joint
-            name="${prefix}_gripper_base_to_${prefix}_gripper_right1"
-            type="revolute"
-        >
-      <limit
-                lower="-3.14"
-                upper="3.14"
-                effort="${joint_effort}"
-                velocity="${joint_velocity}"
-            />
-      <mimic
-                joint="${prefix}_gripper_controller"
-                multiplier="${-worm_gear_ratio}"
-                offset="0"
-            />
-      <origin rpy="1.5708 0.0 -3.14159" xyz="-0.0324 -0.00014 -0.0516" />
-      <parent link="${prefix}_gripper_base" />
-      <child link="${prefix}_gripper_right1" />
-      <axis xyz="0.0 0.0 1.0" />
-      <dynamics damping="${joint_damping}" friction="${joint_friction}" />
-    </joint>
-    <joint
-            name="${prefix}_gripper_right1_to_${prefix}_gripper_right2"
-            type="revolute"
-        >
-      <limit
-                lower="-3.14"
-                upper="3.14"
-                effort="${joint_effort}"
-                velocity="${joint_velocity}"
-            />
-      <mimic
-                joint="${prefix}_gripper_base_to_${prefix}_gripper_right1"
-                multiplier="-1.0"
-                offset="0"
-            />
-      <origin rpy="0.0 0.0 3.14159" xyz="-0.00901 -0.06579 0.00096" />
-      <parent link="${prefix}_gripper_right1" />
-      <child link="${prefix}_gripper_right2" />
-      <axis xyz="0.0 0.0 1.0" />
-      <dynamics damping="${joint_damping}" friction="${joint_friction}" />
-    </joint>
-    <joint
-            name="${prefix}_gripper_right2_to_${prefix}_gripper_right3"
-            type="revolute"
-        >
-      <limit
-                lower="-3.14"
-                upper="3.14"
-                effort="${joint_effort}"
-                velocity="${joint_velocity}"
-            />
-      <mimic
-                joint="${prefix}_gripper_right1_to_${prefix}_gripper_right2"
-                multiplier="-1.0"
-                offset="0"
-            />
-      <origin rpy="0.0 0.0 -3.14159" xyz="-0.01744 -0.02955 0.01103" />
-      <parent link="${prefix}_gripper_right2" />
-      <child link="${prefix}_gripper_right3" />
-      <axis xyz="0.0 0.0 1.0" />
-      <dynamics damping="${joint_damping}" friction="${joint_friction}" />
-    </joint>
-    <!-- Left side joints -->
-    <joint
-            name="${prefix}_gripper_base_to_${prefix}_gripper_left1"
-            type="revolute"
-        >
-      <limit
-                lower="-3.14"
-                upper="3.14"
-                effort="${joint_effort}"
-                velocity="${joint_velocity}"
-            />
-      <mimic
-                joint="${prefix}_gripper_base_to_${prefix}_gripper_right1"
-                multiplier="1.0"
-                offset="0"
-            />
-      <origin rpy="-1.5708 0.0 -3.14159" xyz="0.0324 -0.00014 -0.0516" />
-      <parent link="${prefix}_gripper_base" />
-      <child link="${prefix}_gripper_left1" />
-      <axis xyz="0.0 0.0 1.0" />
-      <dynamics damping="${joint_damping}" friction="${joint_friction}" />
-    </joint>
-    <joint
-            name="${prefix}_gripper_left1_to_${prefix}_gripper_left2"
-            type="revolute"
-        >
-      <limit
-                lower="-3.14"
-                upper="3.14"
-                effort="${joint_effort}"
-                velocity="${joint_velocity}"
-            />
-      <mimic
-                joint="${prefix}_gripper_base_to_${prefix}_gripper_left1"
-                multiplier="1.0"
-                offset="0"
-            />
-      <origin rpy="-3.14159 -0.00006 3.14159" xyz="0.00901 0.06579 -0.00096" />
-      <parent link="${prefix}_gripper_left1" />
-      <child link="${prefix}_gripper_left2" />
-      <axis xyz="0.0 0.0 1.0" />
-      <dynamics damping="${joint_damping}" friction="${joint_friction}" />
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
Commit message: feat: change collision mesh to simple geometries shape for optimize collision compute

File: urdf/walkie-arm/walkie_arm.urdf.xacro (robot description, xacro)
@@ -18,7 +18,7 @@
       </visual>
       <collision>
-        <origin rpy="0.0 0.0 0.0" xyz="0.07550 0.0 0.0" />
+        <origin rpy="1.57080 0.00000 1.57080" xyz="0.03350 0.00000 -0.00513"/>
         <geometry>
-          <mesh filename="package://walkie_description/meshes/walkie-arm/stl/Body1.267.stl" scale="1 1 1"/>
+          <cylinder radius="0.04838" length="0.08350"/>
         </geometry>
       </collision>
@@ -46,7 +46,7 @@
       </visual>
       <collision>
-        <origin rpy="0.0 0.0 0.0" xyz="0.04425 -0.03925 0.0" />
+        <origin rpy="-1.57080 1.57080 0.00000" xyz="0.04418 0.00000 -0.00000"/>
         <geometry>
-          <mesh filename="package://walkie_description/meshes/walkie-arm/stl/Body8.006.stl" scale="1 1 1"/>
+          <cylinder radius="0.04393" length="0.09802"/>
         </geometry>
       </collision>
@@ -73,7 +73,7 @@
       </visual>
       <collision>
-       <origin rpy="0.0 0.0 0.0" xyz="0.0 0.03925 -0.13525" />
+        <origin rpy="0.00000 0.00000 0.00000" xyz="-0.00000 0.03929 -0.12406"/>
         <geometry>
-          <mesh filename="package://walkie_description/meshes/walkie-arm/stl/Body2.006.stl" scale="1 1 1"/>
+          <cylinder radius="0.04469" length="0.15440"/>
         </geometry>
       </collision>
@@ -100,7 +100,7 @@
       </visual>
       <collision>
-        <origin rpy="0.0 0.0 0.0" xyz="0.03825 0.0 -0.11475" />
+        <origin rpy="-0.00000 1.57080 -0.00000" xyz="-0.00103 -0.00000 -0.11471"/>
         <geometry>
-          <mesh filename="package://walkie_description/meshes/walkie-arm/stl/Body1.266.stl" scale="1 1 1"/>
+          <cylinder radius="0.04497" length="0.09083"/>
         </geometry>
       </collision>
@@ -127,7 +127,7 @@
       </visual>
       <collision>
-        <origin rpy="0.0 0.0 0.0" xyz="-0.05962 0.0 -0.12200" />
+        <origin rpy="0.00000 0.00000 0.00000" xyz="-0.03467 -0.00059 -0.09265"/>
         <geometry>
-          <mesh filename="package://walkie_description/meshes/walkie-arm/stl/Body2.020.stl" scale="1 1 1"/>
+          <cylinder radius="0.03436" length="0.09152"/>
         </geometry>
       </collision>
@@ -154,7 +154,7 @@
       </visual>
       <collision>
-        <origin rpy="0.0 0.0 0.0" xyz="0.02037 -0.02800 -0.06500" />
+        <origin rpy="1.57080 0.00000 0.00000" xyz="0.02026 0.00000 -0.06561"/>
         <geometry>
-          <mesh filename="package://walkie_description/meshes/walkie-arm/stl/Body2.026.stl" scale="1 1 1"/>
+          <cylinder radius="0.03329" length="0.06786"/>
         </geometry>
       </collision>
@@ -181,7 +181,7 @@
       </visual>
       <collision>
-        <origin rpy="0.0 0.0 0.0" xyz="0.0 0.02800 -0.13825" />
+        <origin rpy="0.00000 0.00000 0.00000" xyz="-0.00000 0.02829 -0.08677"/>
         <geometry>
-          <mesh filename="package://walkie_description/meshes/walkie-arm/stl/Body1.259.stl" scale="1 1 1"/>
+          <cylinder radius="0.03852" length="0.10036"/>
         </geometry>
       </collision>

File: urdf/walkie-gripper/walkie_gripper.urdf.xacro (robot description, xacro)
@@ -30,5 +30,5 @@
     <link name="${prefix}_link7">
       <visual>
-        <material name="walkie_opaque_gold" />
+        <material name="walkie_aluminum_polished" />
         <origin rpy="0.0 0.0 0.0" xyz="0.0 0.02116 -0.03906" />
         <geometry>

Commit message: fix: invert axis of joint6

File: urdf/walkie-arm/walkie_arm.urdf.xacro (robot description, xacro)
@@ -165,5 +165,5 @@
     </link>
     <joint name="${prefix}_joint6" type="revolute">
-      <axis xyz="0.0 1.0 0.0" />
+      <axis xyz="0.0 -1.0 0.0" />
       <limit effort="${joint_effort}" lower="-1.57" upper="1.57" velocity="${joint_velocity}" />
       <parent link="${prefix}_link5" />
