Commit message: feat: update arm_ros2_control for real hardware, add external_gear_ratio for modified hardware interface

File: urdf/walkie-arm/arm_ros2_control.xacro (robot description, xacro)
@@ -46,38 +46,38 @@
     <xacro:if value="${use_global_config or hw_config['hardware_config'][prefix + '_joint1'] == target_type}">
       <xacro:configure_single_joint name="${prefix}_joint1" type="${target_type}"
-          can_id="${id_offset + 1}" gear_ratio="100.0" trq_limit="30" pole_pairs="14" />
+          can_id="${id_offset + 1}" gear_ratio="10.0" external_gear_ratio="10.0" pole_pairs="14" />
     </xacro:if>
     <xacro:if value="${use_global_config or hw_config['hardware_config'][prefix + '_joint2'] == target_type}">
       <xacro:configure_single_joint name="${prefix}_joint2" type="${target_type}"
-          can_id="${id_offset + 2}" gear_ratio="10.0" trq_limit="30" pole_pairs="14" />
+          can_id="${id_offset + 2}" gear_ratio="10.0" external_gear_ratio="10.0" pole_pairs="14" />
     </xacro:if>
     <xacro:if value="${use_global_config or hw_config['hardware_config'][prefix + '_joint3'] == target_type}">
       <xacro:configure_single_joint name="${prefix}_joint3" type="${target_type}"
-          can_id="${id_offset + 3}" gear_ratio="10.0" trq_limit="30" pole_pairs="14" />
+          can_id="${id_offset + 3}" gear_ratio="10.0" external_gear_ratio="10.0" pole_pairs="14" />
     </xacro:if>
     <xacro:if value="${use_global_config or hw_config['hardware_config'][prefix + '_joint4'] == target_type}">
       <xacro:configure_single_joint name="${prefix}_joint4" type="${target_type}"
-          can_id="${id_offset + 4}" gear_ratio="10.0" trq_limit="20" pole_pairs="14" />
+          can_id="${id_offset + 4}" gear_ratio="10.0" external_gear_ratio="10.0" pole_pairs="14" />
     </xacro:if>
     <xacro:if value="${use_global_config or hw_config['hardware_config'][prefix + '_joint5'] == target_type}">
       <xacro:configure_single_joint name="${prefix}_joint5" type="${target_type}"
-          can_id="${id_offset + 5}" gear_ratio="10.0" trq_limit="10" pole_pairs="14" />
+          can_id="${id_offset + 5}" gear_ratio="10.0" external_gear_ratio="1.0"  pole_pairs="14" />
     </xacro:if>
     <xacro:if value="${use_global_config or hw_config['hardware_config'][prefix + '_joint6'] == target_type}">
       <xacro:configure_single_joint name="${prefix}_joint6" type="${target_type}"
-          can_id="${id_offset + 6}" gear_ratio="10.0" trq_limit="10" pole_pairs="14" />
+          can_id="${id_offset + 6}" gear_ratio="10.0" external_gear_ratio="1.0"  pole_pairs="14" />
     </xacro:if>
     <xacro:if value="${use_global_config or hw_config['hardware_config'][prefix + '_joint7'] == target_type}">
       <xacro:configure_single_joint name="${prefix}_joint7" type="${target_type}"
-          can_id="${id_offset + 7}" gear_ratio="10.0" trq_limit="10" pole_pairs="14" />
+          can_id="${id_offset + 7}" gear_ratio="10.0" external_gear_ratio="1.0"  pole_pairs="14" />
     </xacro:if>
     <xacro:if value="${use_global_config or prefix + '_gripper_worm_gear_joint' in hw_config['hardware_config']}">
          <xacro:if value="${use_global_config or hw_config['hardware_config'][prefix + '_gripper_worm_gear_joint'] == target_type}">
             <xacro:configure_single_gripper name="${prefix}_gripper_worm_gear_joint" type="${target_type}"
-                can_id="${id_offset + 8}" gear_ratio="1.0" trq_limit="5" />
+                can_id="${id_offset + 8}" gear_ratio="10.0" external_gear_ratio="10.0" />
          </xacro:if>
     </xacro:if>
   </xacro:macro>
-  <xacro:macro name="configure_single_joint" params="name type can_id gear_ratio trq_limit pole_pairs">
+  <xacro:macro name="configure_single_joint" params="name type can_id gear_ratio external_gear_ratio pole_pairs">
     <joint name="${name}">
       <xacro:if value="${type == 'cubemars'}">
@@ -87,6 +87,6 @@
         <param name="kt">0.123</param>
         <param name="enc_off">0.0</param>
-        <param name="trq_limit">${trq_limit}</param>
         <param name="read_only">0</param>
+        <param name="external_gear_ratio">${external_gear_ratio}</param>
       </xacro:if>
       <command_interface name="position"/>
@@ -107,5 +107,5 @@
     </joint>
   </xacro:macro>
-  <xacro:macro name="configure_single_gripper" params="name type can_id gear_ratio trq_limit">
+  <xacro:macro name="configure_single_gripper" params="name type can_id gear_ratio external_gear_ratio">
     <joint name="${name}">
       <xacro:if value="${type == 'cubemars'}">
@@ -115,6 +115,6 @@
          <param name="kt">0.123</param>
          <param name="enc_off">0.0</param>
-         <param name="trq_limit">${trq_limit}</param>
          <param name="read_only">0</param>
+        <param name="external_gear_ratio">${external_gear_ratio}</param>
       </xacro:if>
       <command_interface name="position"/>

Commit message: feat: config for torque control

File: urdf/walkie-arm/arm_ros2_control.xacro (robot description, xacro)
@@ -117,5 +117,5 @@
          <param name="read_only">0</param>
         <param name="external_gear_ratio">${external_gear_ratio}</param>
-        <param name="trq_limit">1</param>
+        <param name="trq_limit">1.7</param>
         <param name="grasp_detect">1</param>
       </xacro:if>

File: urdf/walkie-arm/walkie_arm.urdf.xacro (robot description, xacro)
@@ -58,5 +58,5 @@
     <joint name="${prefix}_joint2" type="revolute">
       <axis xyz="0.0 1.0 0.0" />
-      <limit effort="${joint_effort}" lower="-3.14" upper="0.0" velocity="${joint_velocity}" />
+      <limit effort="${joint_effort}" lower="-3.14" upper="0.1" velocity="${joint_velocity}" />
       <parent link="${prefix}_link1" />
       <child link="${prefix}_link2" />
