Commit message: feat: roller

File: urdf/walkie/omni_wheel/gz_omni_wheel.urdf.xacro (robot description, xacro)
@@ -1,49 +1,171 @@
-<?xml version="1.0" ?>
-<robot xmlns:xacro="http://ros.org/wiki/xacro">
-  <xacro:include
-        filename="$(find walkie_description)/urdf/inertial_macros.xacro"
-    />
-  <xacro:include
-        filename="$(find walkie_description)/urdf/walkie/omni_wheel/omni_wheel.gazebo.xacro"
-    />
-  <xacro:include
-        filename="$(find walkie_description)/urdf/walkie/omni_wheel/omni_wheel.transmission.xacro"
-    />
-  <xacro:property name="wheel_thickness" value="0.05" />
-  <xacro:property name="wheel_radian" value="0.075" />
-  <xacro:property name="wheel_mass" value="0.05" />
-  <xacro:macro name="wheel_v0" params="prefix parent *joint_origin *joint_axis">
-    <joint name="${prefix}_wheel_joint" type="continuous">
-      <xacro:insert_block name="joint_origin" />
-      <parent link="${parent}" />
-      <child link="${prefix}_wheel_link" />
-      <limit effort="100" velocity="100" />
-      <dynamics damping="5.0" friction="0.5" />
-      <xacro:insert_block name="joint_axis" />
-    </joint>
-    <link name="${prefix}_wheel_link">
-        <visual>
-            <geometry>
-                <mesh
-                        filename="package://walkie_description/meshes/walkie/omni_wheel_optimize.dae"
-                        scale="1 1 1"
-                    />
-            </geometry>
-        </visual>
-        <xacro:inertial_cylinder
-                mass="${wheel_mass}"
-                length="${wheel_thickness}"
-                radius="${wheel_radian}"
-            >
-            <origin xyz="0 0 0" rpy="1.570796327 0 0" />
-        </xacro:inertial_cylinder>
-        <collision>
-            <origin xyz="0 0 0" rpy="1.570796327 0 0" />
-            <geometry>
-            <cylinder radius="${wheel_radian}" length="${wheel_thickness}" />
-            </geometry>
-        </collision>
-    </link>
-    <xacro:wheel_gazebo_v0 prefix="${prefix}" />
-  </xacro:macro>
+<?xml version="1.0"?>
+<robot name="omni_wheel" xmlns:xacro="http://ros.org/wiki/xacro">
+  <xacro:arg name="standalone" default="false" />
+  <xacro:arg name="prefix" default="wheel" />
+  <xacro:arg name="parent" default="base_link" />
+	<xacro:include
+    filename="$(find walkie_description)/urdf/inertial_macros.xacro"
+  />
+	<xacro:include
+    filename="$(find walkie_description)/urdf/walkie/omni_wheel/omni_wheel.gazebo.xacro"
+  />
+	<xacro:include
+    filename="$(find walkie_description)/urdf/walkie/omni_wheel/omni_wheel.transmission.xacro"
+  />
+	<xacro:include
+    filename="$(find walkie_description)/urdf/walkie/roller/gz_roller.urdf.xacro"
+  />
+	<xacro:property name="wheel_thickness" value="0.05" />
+	<xacro:property name="wheel_radian" value="0.075" />
+	<xacro:property name="wheel_mass" value="0.05" />
+	<xacro:macro name="wheel_v0" params="prefix parent *joint_origin *joint_axis">
+  	<joint name="${prefix}_wheel_joint" type="continuous">
+  		<xacro:insert_block name="joint_origin" />
+  		<parent link="${parent}" />
+  		<child link="${prefix}_wheel_link" />
+  		<limit effort="100" velocity="100" />
+  		<dynamics damping="5.0" friction="0.5" />
+  		<xacro:insert_block name="joint_axis" />
+  	</joint>
+  	<link name="${prefix}_wheel_link">
+  		<visual>
+  			<geometry>
+  				<mesh
+            filename="package://walkie_description/meshes/walkie/omni_wheel_optimize.dae"
+            scale="1 1 1"
+          />
+  			</geometry>
+  		</visual>
+  		<xacro:inertial_cylinder
+        mass="${wheel_mass}"
+        length="${wheel_thickness}"
+        radius="${wheel_radian}"
+      >
+  			<origin xyz="0 0 0" rpy="1.570796327 0 0" />
+  		</xacro:inertial_cylinder>
+  		<!-- <collision><origin xyz="0 0 0" rpy="1.570796327 0 0" /><geometry><cylinder radius="${wheel_radian}" length="${wheel_thickness}" /></geometry></collision> -->
+  	</link>
+  	<xacro:wheel_gazebo_v0 prefix="${prefix}" />
+  	<!-- Individual Roller Joint and Link Instantiations -->
+  	<xacro:roller prefix="${prefix}" num="1">
+  		<origin xyz="0.067000 -0.009500 0.000000" rpy="0.000000 -0.000000 0.000000" />
+  		<axis xyz="0.000000 0.000000 1.000000" />
+  	</xacro:roller>
+  	<xacro:roller prefix="${prefix}" num="2">
+  		<origin xyz="0.060365 -0.009500 0.029070" rpy="0.000000 -0.448799 0.000000" />
+  		<axis xyz="0.000000 0.000000 1.000000" />
+  	</xacro:roller>
+  	<xacro:roller prefix="${prefix}" num="3">
+  		<origin xyz="0.041774 -0.009500 0.052383" rpy="0.000000 -0.897598 0.000000" />
+  		<axis xyz="0.000000 0.000000 1.000000" />
+  	</xacro:roller>
+  	<xacro:roller prefix="${prefix}" num="4">
+  		<origin xyz="0.014909 -0.009500 0.065320" rpy="0.000000 -1.346398 0.000000" />
+  		<axis xyz="0.000000 0.000000 1.000000" />
+  	</xacro:roller>
+  	<xacro:roller prefix="${prefix}" num="5">
+  		<origin xyz="-0.014909 -0.009500 0.065320" rpy="0.000000 -1.795195 0.000000" />
+  		<axis xyz="0.000000 0.000000 1.000000" />
+  	</xacro:roller>
+  	<xacro:roller prefix="${prefix}" num="6">
+  		<origin xyz="-0.041774 -0.009500 0.052383" rpy="0.000000 -2.243994 0.000000" />
+  		<axis xyz="0.000000 0.000000 1.000000" />
+  	</xacro:roller>
+  	<xacro:roller prefix="${prefix}" num="7">
+  		<origin xyz="-0.060365 -0.009500 0.029070" rpy="0.000000 -2.692793 0.000000" />
+  		<axis xyz="0.000000 0.000000 1.000000" />
+  	</xacro:roller>
+  	<xacro:roller prefix="${prefix}" num="8">
+  		<origin xyz="-0.067000 -0.009500 0.000000" rpy="0.000000 -3.141593 0.000000" />
+  		<axis xyz="0.000000 0.000000 1.000000" />
+  	</xacro:roller>
+  	<xacro:roller prefix="${prefix}" num="9">
+  		<origin xyz="-0.060365 -0.009500 -0.029070" rpy="0.000000 -3.590392 0.000000" />
+  		<axis xyz="0.000000 0.000000 1.000000" />
+  	</xacro:roller>
+  	<xacro:roller prefix="${prefix}" num="10">
+  		<origin xyz="-0.041774 -0.009500 -0.052383" rpy="0.000000 -4.039191 0.000000" />
+  		<axis xyz="0.000000 0.000000 1.000000" />
+  	</xacro:roller>
+  	<xacro:roller prefix="${prefix}" num="11">
+  		<origin xyz="-0.014909 -0.009500 -0.065320" rpy="0.000000 -4.487990 0.000000" />
+  		<axis xyz="0.000000 0.000000 1.000000" />
+  	</xacro:roller>
+  	<xacro:roller prefix="${prefix}" num="12">
+  		<origin xyz="0.014909 -0.009500 -0.065320" rpy="0.000000 -4.936788 0.000000" />
+  		<axis xyz="0.000000 0.000000 1.000000" />
+  	</xacro:roller>
+  	<xacro:roller prefix="${prefix}" num="13">
+  		<origin xyz="0.041774 -0.009500 -0.052383" rpy="0.000000 -5.385587 0.000000" />
+  		<axis xyz="0.000000 0.000000 1.000000" />
+  	</xacro:roller>
+  	<xacro:roller prefix="${prefix}" num="14">
+  		<origin xyz="0.060365 -0.009500 -0.029070" rpy="0.000000 -5.834386 0.000000" />
+  		<axis xyz="0.000000 0.000000 1.000000" />
+  	</xacro:roller>
+  	<xacro:roller prefix="${prefix}" num="15">
+  		<origin xyz="0.065319 0.009500 0.014912" rpy="0.000000 -0.224449 0.000000" />
+  		<axis xyz="0.000000 0.000000 1.000000" />
+  	</xacro:roller>
+  	<xacro:roller prefix="${prefix}" num="16">
+  		<origin xyz="0.052381 0.009500 0.041776" rpy="0.000000 -0.673249 0.000000" />
+  		<axis xyz="0.000000 0.000000 1.000000" />
+  	</xacro:roller>
+  	<xacro:roller prefix="${prefix}" num="17">
+  		<origin xyz="0.029067 0.009500 0.060366" rpy="0.000000 -1.122048 0.000000" />
+  		<axis xyz="0.000000 0.000000 1.000000" />
+  	</xacro:roller>
+  	<xacro:roller prefix="${prefix}" num="18">
+  		<origin xyz="-0.000003 0.009500 0.067000" rpy="0.000000 -1.570847 0.000000" />
+  		<axis xyz="0.000000 0.000000 1.000000" />
+  	</xacro:roller>
+  	<xacro:roller prefix="${prefix}" num="19">
+  		<origin xyz="-0.029073 0.009500 0.060363" rpy="0.000000 -2.019644 0.000000" />
+  		<axis xyz="0.000000 0.000000 1.000000" />
+  	</xacro:roller>
+  	<xacro:roller prefix="${prefix}" num="20">
+  		<origin xyz="-0.052385 0.009500 0.041771" rpy="0.000000 -2.468444 0.000000" />
+  		<axis xyz="0.000000 0.000000 1.000000" />
+  	</xacro:roller>
+  	<xacro:roller prefix="${prefix}" num="21">
+  		<origin xyz="-0.065321 0.009500 0.014906" rpy="0.000000 -2.917243 0.000000" />
+  		<axis xyz="0.000000 0.000000 1.000000" />
+  	</xacro:roller>
+  	<xacro:roller prefix="${prefix}" num="22">
+  		<origin xyz="-0.065319 0.009500 -0.014912" rpy="0.000000 -3.366042 0.000000" />
+  		<axis xyz="0.000000 0.000000 1.000000" />
+  	</xacro:roller>
+  	<xacro:roller prefix="${prefix}" num="23">
+  		<origin xyz="-0.052381 0.009500 -0.041776" rpy="0.000000 -3.814841 0.000000" />
+  		<axis xyz="0.000000 0.000000 1.000000" />
+  	</xacro:roller>
+  	<xacro:roller prefix="${prefix}" num="24">
+  		<origin xyz="-0.029067 0.009500 -0.060366" rpy="0.000000 -4.263640 0.000000" />
+  		<axis xyz="0.000000 0.000000 1.000000" />
+  	</xacro:roller>
+  	<xacro:roller prefix="${prefix}" num="25">
+  		<origin xyz="0.000003 0.009500 -0.067000" rpy="0.000000 -4.712440 0.000000" />
+  		<axis xyz="0.000000 0.000000 1.000000" />
+  	</xacro:roller>
+  	<xacro:roller prefix="${prefix}" num="26">
+  		<origin xyz="0.029073 0.009500 -0.060363" rpy="0.000000 -5.161237 0.000000" />
+  		<axis xyz="0.000000 0.000000 1.000000" />
+  	</xacro:roller>
+  	<xacro:roller prefix="${prefix}" num="27">
+  		<origin xyz="0.052385 0.009500 -0.041771" rpy="0.000000 -5.610036 0.000000" />
+  		<axis xyz="0.000000 0.000000 1.000000" />
+  	</xacro:roller>
+  	<xacro:roller prefix="${prefix}" num="28">
+  		<origin xyz="0.065321 0.009500 -0.014906" rpy="0.000000 -6.058835 0.000000" />
+  		<axis xyz="0.000000 0.000000 1.000000" />
+  	</xacro:roller>
+	</xacro:macro>
+  <!-- Standalone Wheel Instantiation for testing & export -->
+  <xacro:if value="$(arg standalone)">
+    <link name="$(arg parent)" />
+    <xacro:wheel_v0 prefix="$(arg prefix)" parent="$(arg parent)">
+      <origin xyz="0 0 0" rpy="0 0 0" />
+      <axis xyz="0 1 0" />
+    </xacro:wheel_v0>
+  </xacro:if>
 </robot>

Commit message: Align sim/isaac drive geometry with real robot
Co-authored-by: Armmy2530 <42490759+Armmy2530@users.noreply.github.com>

File: urdf/walkie/omni_wheel/gz_omni_wheel.urdf.xacro (robot description, xacro)
@@ -11,5 +11,5 @@
     />
   <xacro:property name="wheel_thickness" value="0.05" />
-  <xacro:property name="wheel_radian" value="0.075" />
+  <xacro:property name="wheel_radius" value="0.076" />
   <xacro:property name="wheel_mass" value="0.05" />
   <xacro:macro name="wheel_v0" params="prefix parent *joint_origin *joint_axis">
@@ -34,5 +34,5 @@
                 mass="${wheel_mass}"
                 length="${wheel_thickness}"
-                radius="${wheel_radian}"
+                radius="${wheel_radius}"
             >
             <origin xyz="0 0 0" rpy="1.570796327 0 0" />
@@ -41,5 +41,5 @@
             <origin xyz="0 0 0" rpy="1.570796327 0 0" />
             <geometry>
-            <cylinder radius="${wheel_radian}" length="${wheel_thickness}" />
+            <cylinder radius="${wheel_radius}" length="${wheel_thickness}" />
             </geometry>
         </collision>
