Commit message: fix: update controller parameters

File: urdf/walkie/head/servo_camera.urdf.xacro (robot description, xacro)
@@ -19,6 +19,6 @@
       <parent link="${prefix}_servobase_link"/>
       <child link="${prefix}_servo_link"/>
-      <origin xyz="0 0 0" rpy="0 0 0"/> <axis xyz="1 0 0"/>
-      <limit lower="-1.5708" upper="1.5708" effort="1.0" velocity="1.0"/>
+      <origin xyz="0 0 0" rpy="0 0 0"/> <axis xyz="-1 0 0"/>
+      <limit lower="-0.384" upper="0.436" effort="10.0" velocity="1.0"/>
     </joint>
     <link name="${prefix}_servo_link">

File: urdf/walkie/ros2_control.xacro (robot description, xacro)
@@ -171,5 +171,5 @@
       <ros2_control name="HeadServoSystem" type="system">
         <hardware>
-          <plugin>topic_based_ros2_control/TopicBasedSystem</plugin>
+          <plugin>mock_components/GenericSystem</plugin>
           <param name="joint_commands_topic">/head_servo_joint_cmd</param>
           <param name="joint_states_topic">/head_servo_joint_states</param>

Commit message: feat: integrate zed camera model into walkie 1-arm head

File: urdf/walkie/head/servo_camera.urdf.xacro (robot description, xacro)
@@ -1,39 +1,79 @@
 <?xml version="1.0"?>
 <robot xmlns:xacro="http://ros.org/wiki/xacro">
+  <xacro:include filename="$(find zed_wrapper)/urdf/zed_macro.urdf.xacro" />
   <xacro:macro name="servo_v0" params="prefix parent *joint_origin">
+    <xacro:arg name="camera_name" default="zed_${prefix}"/>
+    <xacro:arg name="camera_model" default="zed2i" />
+    <xacro:arg name="use_zed_localization" default="false" />
     <joint name="${prefix}_servobase_joint" type="fixed">
-      <xacro:insert_block name="joint_origin"/>
-      <parent link="${parent}"/>
-      <child link="${prefix}_servobase_link"/>
+      <xacro:insert_block name="joint_origin" />
+      <parent link="${parent}" />
+      <child link="${prefix}_servobase_link" />
     </joint>
     <link name="${prefix}_servobase_link">
       <visual>
-        <origin xyz="0 0 0" rpy="0 0 0"/>
+        <origin xyz="0 0 0" rpy="0 0 0" />
         <geometry>
-          <mesh filename="package://walkie_description/meshes/walkie/ServoMountPlate.stl"  scale="0.001 0.001 0.001"/>
+          <mesh filename="package://walkie_description/meshes/walkie/ServoMountPlate.stl"
+            scale="0.001 0.001 0.001" />
         </geometry>
-        <material name="dark_grey"><color rgba="0.2 0.2 0.2 1"/></material>
+        <material name="dark_grey">
+          <color rgba="0.2 0.2 0.2 1" />
+        </material>
       </visual>
     </link>
     <joint name="${prefix}_servo_joint" type="revolute">
-      <parent link="${prefix}_servobase_link"/>
-      <child link="${prefix}_servo_link"/>
-      <origin xyz="0 0 0" rpy="0 0 0"/> <axis xyz="-1 0 0"/>
-      <limit lower="-0.384" upper="0.436" effort="10.0" velocity="1.0"/>
+      <parent link="${prefix}_servobase_link" />
+      <child link="${prefix}_servo_link" />
+      <origin xyz="0 0 0" rpy="0 0 0" />
+      <axis xyz="-1 0 0" />
+      <limit lower="-0.384" upper="0.436" effort="10.0" velocity="1.0" />
     </joint>
     <link name="${prefix}_servo_link">
       <visual>
-        <origin xyz="0 0 0" rpy="0 0 0"/>
+        <origin xyz="0 0 0" rpy="0 0 0" />
         <geometry>
-          <mesh filename="package://walkie_description/meshes/walkie/ServoCameraCase.stl"  scale="0.001 0.001 0.001"/>
+          <mesh filename="package://walkie_description/meshes/walkie/ServoCameraCase.stl"
+            scale="0.001 0.001 0.001" />
         </geometry>
       </visual>
       <collision>
-        <origin xyz="0.104 0 0" rpy="0 0 0"/>
+        <origin xyz="0.104 0 0" rpy="0 0 0" />
         <geometry>
-          <box size="0.208 0.039 0.039"/>
+          <box size="0.208 0.039 0.039" />
         </geometry>
       </collision>
     </link>
+    <xacro:zed_camera name="zed" model="$(arg camera_model)">
+      <!-- <gnss_origin /> -->
+       <origin xyz="0 0 0" rpy="0 0 0" />
+    </xacro:zed_camera>
+    <!-- <xacro:zed_camera name="zed" model="zed2i">
+      <origin xyz="0 0 0" rpy="0 0 0"/>
+    </xacro:zed_camera> -->
+    <!-- Zed Camera Mounting Joint -->
+    <!-- <joint name="${prefix}_zed_mounting_joint" type="fixed">
+      <parent link="${prefix}_servo_link" />
+      <child link="zed_camera_link" />
+      <origin xyz="0.098 -0.02 0" rpy="0 0 -1.5708" />
+    </joint> -->
+    <xacro:if value="$(arg use_zed_localization)">
+      <joint name="$(arg camera_name)_joint" type="fixed">
+        <parent link="$(arg camera_name)_camera_link" />
+        <child link="${prefix}_servo_link" />
+        <origin xyz="0.098 -0.02 -0.015" rpy="0 0 -1.5708" />
+        <!-- <origin
+          xyz="-0.12 0.0 -0.25"
+          rpy="0 0 0"
+        /> -->
+      </joint>
+    </xacro:if>
+    <xacro:unless value="$(arg use_zed_localization)">
+      <joint name="$(arg camera_name)_joint" type="fixed">
+        <parent link="${prefix}_servo_link" />
+        <child link="zed_camera_link" />
+        <origin xyz="0.098 -0.006 -0.015" rpy="0 0 -1.5708" />
+      </joint>
+    </xacro:unless>
   </xacro:macro>
 </robot>

Commit message: fix: correct camera collision origin and geometry offsets

File: urdf/walkie/head/servo_camera.urdf.xacro (robot description, xacro)
@@ -9,5 +9,5 @@
     <!-- ============ Servo Joint (tilt) ============ -->
     <joint name="${prefix}_servo_joint" type="revolute">
-      <limit lower="-3.14000" upper="3.14000" effort="0.00000" velocity="0.00000"/>
+      <limit lower="-0.785398163" upper="0.785398163" effort="0.00000" velocity="0.00000"/>
       <parent link="${parent}"/>
       <child link="${prefix}_servo_link"/>
@@ -23,7 +23,7 @@
       </visual>
       <collision>
-        <origin xyz="0.104 0 0" rpy="0 0 0"/>
+        <origin xyz="0.034 -0.056649 0" rpy="0 0 0"/>
         <geometry>
-          <box size="0.208 0.039 0.039"/>
+          <box size="0.186 0.044 0.040"/>
         </geometry>
       </collision>
