Commit message: fix: zed from path using file:// -> package://

File: urdf/walkie/depth_camera/zed/zed_macro.urdf.xacro (robot description, xacro)
@@ -1,3 +1,3 @@
-<?xml version="1.0"?>
+<?xml version="1.0" ?>
 <!--
 // Copyright 2025 Stereolabs
@@ -16,5 +16,5 @@
 -->
 <robot xmlns:xacro="http://wiki.ros.org/xacro">
-  <xacro:property name="M_PI" value="3.1415926535897931"/>
+  <xacro:property name="M_PI" value="3.1415926535897931" />
   <!--
     Parameters:
@@ -23,153 +23,160 @@
       - enable_gnss: if true enable the URDF link
   -->
-  <xacro:macro name="zed_camera" params="name=zed model=zed enable_gnss=false custom_baseline=0 *gnss_origin">
+  <xacro:macro
+        name="zed_camera"
+        params="name=zed model=zed enable_gnss=false custom_baseline=0 *gnss_origin"
+    >
     <xacro:if value="${model == 'zed'}">
-      <xacro:property name="baseline" value="0.12"/>
-      <xacro:property name="height" value="0.03"/>
-      <xacro:property name="bottom_slope" value="0.05"/>
-      <xacro:property name="screw_offset_x" value="0.0"/>
-      <xacro:property name="screw_offset_z" value="0.0"/>
-      <xacro:property name="optical_offset_x" value="-0.01"/>
-      <xacro:property name="mono" value="false"/>
-      <xacro:property name="mat" value="0.8 0.8 0.8 1.0"/>
+      <xacro:property name="baseline" value="0.12" />
+      <xacro:property name="height" value="0.03" />
+      <xacro:property name="bottom_slope" value="0.05" />
+      <xacro:property name="screw_offset_x" value="0.0" />
+      <xacro:property name="screw_offset_z" value="0.0" />
+      <xacro:property name="optical_offset_x" value="-0.01" />
+      <xacro:property name="mono" value="false" />
+      <xacro:property name="mat" value="0.8 0.8 0.8 1.0" />
     </xacro:if>
     <xacro:if value="${model == 'zedm'}">
-      <xacro:property name="baseline" value="0.063"/>
-      <xacro:property name="height" value="0.0265"/>
-      <xacro:property name="bottom_slope" value="0.0"/>
-      <xacro:property name="screw_offset_x" value="0.0"/>
-      <xacro:property name="screw_offset_z" value="0.0"/>
-      <xacro:property name="optical_offset_x" value="0.0"/>
-      <xacro:property name="mono" value="false"/>
-      <xacro:property name="mat" value="0 0 0 1.0"/>
+      <xacro:property name="baseline" value="0.063" />
+      <xacro:property name="height" value="0.0265" />
+      <xacro:property name="bottom_slope" value="0.0" />
+      <xacro:property name="screw_offset_x" value="0.0" />
+      <xacro:property name="screw_offset_z" value="0.0" />
+      <xacro:property name="optical_offset_x" value="0.0" />
+      <xacro:property name="mono" value="false" />
+      <xacro:property name="mat" value="0 0 0 1.0" />
     </xacro:if>
     <xacro:if value="${model == 'zed2'}">
-      <xacro:property name="baseline" value="0.12"/>
-      <xacro:property name="height" value="0.03"/>
-      <xacro:property name="bottom_slope" value="0.05"/>
-      <xacro:property name="screw_offset_x" value="0.0"/>
-      <xacro:property name="screw_offset_z" value="0.0"/>
-      <xacro:property name="optical_offset_x" value="-0.01"/>
-      <xacro:property name="mono" value="false"/>
-      <xacro:property name="mat" value="0.25 0.25 0.25 1.0"/>
+      <xacro:property name="baseline" value="0.12" />
+      <xacro:property name="height" value="0.03" />
+      <xacro:property name="bottom_slope" value="0.05" />
+      <xacro:property name="screw_offset_x" value="0.0" />
+      <xacro:property name="screw_offset_z" value="0.0" />
+      <xacro:property name="optical_offset_x" value="-0.01" />
+      <xacro:property name="mono" value="false" />
+      <xacro:property name="mat" value="0.25 0.25 0.25 1.0" />
     </xacro:if>
     <xacro:if value="${model == 'zed2i'}">
-      <xacro:property name="baseline" value="0.12"/>
-      <xacro:property name="height" value="0.03"/>
-      <xacro:property name="bottom_slope" value="0.0"/>
-      <xacro:property name="screw_offset_x" value="-0.01"/>
-      <xacro:property name="screw_offset_z" value="0.0"/>
-      <xacro:property name="optical_offset_x" value="-0.01"/>
-      <xacro:property name="mono" value="false"/>
-      <xacro:property name="mat" value="0.25 0.25 0.25 1.0"/>
+      <xacro:property name="baseline" value="0.12" />
+      <xacro:property name="height" value="0.03" />
+      <xacro:property name="bottom_slope" value="0.0" />
+      <xacro:property name="screw_offset_x" value="-0.01" />
+      <xacro:property name="screw_offset_z" value="0.0" />
+      <xacro:property name="optical_offset_x" value="-0.01" />
+      <xacro:property name="mono" value="false" />
+      <xacro:property name="mat" value="0.25 0.25 0.25 1.0" />
     </xacro:if>
     <xacro:if value="${model == 'zedx'}">
-      <xacro:property name="baseline" value="0.12"/>
-      <xacro:property name="height" value="0.032"/>
-      <xacro:property name="bottom_slope" value="0.0"/>
-      <xacro:property name="screw_offset_x" value="0.0"/>
-      <xacro:property name="screw_offset_z" value="-0.016"/>
-      <xacro:property name="optical_offset_x" value="-0.01"/>
-      <xacro:property name="mono" value="false"/>
-      <xacro:property name="mat" value="0.25 0.25 0.25 1.0"/>
+      <xacro:property name="baseline" value="0.12" />
+      <xacro:property name="height" value="0.032" />
+      <xacro:property name="bottom_slope" value="0.0" />
+      <xacro:property name="screw_offset_x" value="0.0" />
+      <xacro:property name="screw_offset_z" value="-0.016" />
+      <xacro:property name="optical_offset_x" value="-0.01" />
+      <xacro:property name="mono" value="false" />
+      <xacro:property name="mat" value="0.25 0.25 0.25 1.0" />
     </xacro:if>
     <xacro:if value="${model == 'zedxhdr'}">
-      <xacro:property name="baseline" value="0.12"/>
-      <xacro:property name="height" value="0.032"/>
-      <xacro:property name="bottom_slope" value="0.0"/>
-      <xacro:property name="screw_offset_x" value="0.0"/>
-      <xacro:property name="screw_offset_z" value="-0.016"/>
-      <xacro:property name="optical_offset_x" value="-0.01"/>
-      <xacro:property name="mono" value="false"/>
-      <xacro:property name="mat" value="0.25 0.25 0.25 1.0"/>
+      <xacro:property name="baseline" value="0.12" />
+      <xacro:property name="height" value="0.032" />
+      <xacro:property name="bottom_slope" value="0.0" />
+      <xacro:property name="screw_offset_x" value="0.0" />
+      <xacro:property name="screw_offset_z" value="-0.016" />
+      <xacro:property name="optical_offset_x" value="-0.01" />
+      <xacro:property name="mono" value="false" />
+      <xacro:property name="mat" value="0.25 0.25 0.25 1.0" />
     </xacro:if>
     <xacro:if value="${model == 'zedxm'}">
-      <xacro:property name="baseline" value="0.05"/>
-      <xacro:property name="height" value="0.032"/>
-      <xacro:property name="bottom_slope" value="0.0"/>
-      <xacro:property name="screw_offset_x" value="0.0"/>
-      <xacro:property name="screw_offset_z" value="-0.016"/>
-      <xacro:property name="optical_offset_x" value="-0.01"/>
-      <xacro:property name="mono" value="false"/>
-      <xacro:property name="mat" value="0.25 0.25 0.25 1.0"/>
+      <xacro:property name="baseline" value="0.05" />
+      <xacro:property name="height" value="0.032" />
+      <xacro:property name="bottom_slope" value="0.0" />
+      <xacro:property name="screw_offset_x" value="0.0" />
+      <xacro:property name="screw_offset_z" value="-0.016" />
+      <xacro:property name="optical_offset_x" value="-0.01" />
+      <xacro:property name="mono" value="false" />
+      <xacro:property name="mat" value="0.25 0.25 0.25 1.0" />
     </xacro:if>
     <xacro:if value="${model == 'zedxhdrmini'}">
-      <xacro:property name="baseline" value="0.05"/>
-      <xacro:property name="height" value="0.032"/>
-      <xacro:property name="bottom_slope" value="0.0"/>
-      <xacro:property name="screw_offset_x" value="0.0"/>
-      <xacro:property name="screw_offset_z" value="-0.016"/>
-      <xacro:property name="optical_offset_x" value="-0.01"/>
-      <xacro:property name="mono" value="false"/>
-      <xacro:property name="mat" value="0.25 0.25 0.25 1.0"/>
+      <xacro:property name="baseline" value="0.05" />
+      <xacro:property name="height" value="0.032" />
+      <xacro:property name="bottom_slope" value="0.0" />
+      <xacro:property name="screw_offset_x" value="0.0" />
+      <xacro:property name="screw_offset_z" value="-0.016" />
+      <xacro:property name="optical_offset_x" value="-0.01" />
+      <xacro:property name="mono" value="false" />
+      <xacro:property name="mat" value="0.25 0.25 0.25 1.0" />
     </xacro:if>
     <xacro:if value="${model == 'zedxhdrmax'}">
-      <xacro:property name="baseline" value="0.170"/>
-      <xacro:property name="height" value="0.032"/>
-      <xacro:property name="bottom_slope" value="0.0"/>
-      <xacro:property name="screw_offset_x" value="0.0"/>
-      <xacro:property name="screw_offset_z" value="-0.016"/>
-      <xacro:property name="optical_offset_x" value="-0.01"/>
-      <xacro:property name="mono" value="false"/>
-      <xacro:property name="mat" value="0.25 0.25 0.25 1.0"/>
+      <xacro:property name="baseline" value="0.170" />
+      <xacro:property name="height" value="0.032" />
+      <xacro:property name="bottom_slope" value="0.0" />
+      <xacro:property name="screw_offset_x" value="0.0" />
+      <xacro:property name="screw_offset_z" value="-0.016" />
+      <xacro:property name="optical_offset_x" value="-0.01" />
+      <xacro:property name="mono" value="false" />
+      <xacro:property name="mat" value="0.25 0.25 0.25 1.0" />
     </xacro:if>
     <xacro:if value="${model == 'virtual'}">
-      <xacro:property name="baseline" value="${custom_baseline}"/>
-      <xacro:property name="height" value="0.031"/>
-      <xacro:property name="bottom_slope" value="0.0"/>
-      <xacro:property name="screw_offset_x" value="0.00"/>
-      <xacro:property name="screw_offset_z" value="-0.0155"/>
-      <xacro:property name="optical_offset_x" value="0.0"/>
-      <xacro:property name="mono" value="false"/>
-      <xacro:property name="mat" value="0.25 0.25 0.25 1.0"/>
+      <xacro:property name="baseline" value="${custom_baseline}" />
+      <xacro:property name="height" value="0.031" />
+      <xacro:property name="bottom_slope" value="0.0" />
+      <xacro:property name="screw_offset_x" value="0.00" />
+      <xacro:property name="screw_offset_z" value="-0.0155" />
+      <xacro:property name="optical_offset_x" value="0.0" />
+      <xacro:property name="mono" value="false" />
+      <xacro:property name="mat" value="0.25 0.25 0.25 1.0" />
     </xacro:if>
     <xacro:if value="${model == 'zedxonegs'}">
-      <xacro:property name="baseline" value="0.0"/>
-      <xacro:property name="height" value="0.031"/>
-      <xacro:property name="bottom_slope" value="0.0"/>
-      <xacro:property name="screw_offset_x" value="0.0"/>
-      <xacro:property name="screw_offset_z" value="-0.0155"/>
-      <xacro:property name="optical_offset_x" value="0.0"/>
-      <xacro:property name="mono" value="true"/>
-      <xacro:property name="mat" value="0.25 0.25 0.25 1.0"/>
+      <xacro:property name="baseline" value="0.0" />
+      <xacro:property name="height" value="0.031" />
+      <xacro:property name="bottom_slope" value="0.0" />
+      <xacro:property name="screw_offset_x" value="0.0" />
+      <xacro:property name="screw_offset_z" value="-0.0155" />
+      <xacro:property name="optical_offset_x" value="0.0" />
+      <xacro:property name="mono" value="true" />
+      <xacro:property name="mat" value="0.25 0.25 0.25 1.0" />
     </xacro:if>
     <xacro:if value="${model == 'zedxone4k'}">
-      <xacro:property name="baseline" value="0.0"/>
-      <xacro:property name="height" value="0.031"/>
-      <xacro:property name="bottom_slope" value="0.0"/>
-      <xacro:property name="screw_offset_x" value="0.00"/>
-      <xacro:property name="screw_offset_z" value="-0.0155"/>
-      <xacro:property name="optical_offset_x" value="0.0"/>
-      <xacro:property name="mono" value="true"/>
-      <xacro:property name="mat" value="0.25 0.25 0.25 1.0"/>
+      <xacro:property name="baseline" value="0.0" />
+      <xacro:property name="height" value="0.031" />
+      <xacro:property name="bottom_slope" value="0.0" />
+      <xacro:property name="screw_offset_x" value="0.00" />
+      <xacro:property name="screw_offset_z" value="-0.0155" />
+      <xacro:property name="optical_offset_x" value="0.0" />
+      <xacro:property name="mono" value="true" />
+      <xacro:property name="mat" value="0.25 0.25 0.25 1.0" />
     </xacro:if>
     <xacro:if value="${model == 'zedxonehdr'}">
-      <xacro:property name="baseline" value="0.0"/>
-      <xacro:property name="height" value="0.025"/>
-      <xacro:property name="bottom_slope" value="0.0"/>
-      <xacro:property name="screw_offset_x" value="0.00"/>
-      <xacro:property name="screw_offset_z" value="-0.0125"/>
-      <xacro:property name="optical_offset_x" value="0.0"/>
-      <xacro:property name="mono" value="true"/>
-      <xacro:property name="mat" value="0.25 0.25 0.25 1.0"/>
+      <xacro:property name="baseline" value="0.0" />
+      <xacro:property name="height" value="0.025" />
+      <xacro:property name="bottom_slope" value="0.0" />
+      <xacro:property name="screw_offset_x" value="0.00" />
+      <xacro:property name="screw_offset_z" value="-0.0125" />
+      <xacro:property name="optical_offset_x" value="0.0" />
+      <xacro:property name="mono" value="true" />
+      <xacro:property name="mat" value="0.25 0.25 0.25 1.0" />
     </xacro:if>
     <!-- Camera mounting point (the threaded screw hole in the bottom) -->
-    <link name="${name}_camera_link"/>
+    <link name="${name}_camera_link" />
     <!-- Camera Center -->
     <link name="${name}_camera_center">
       <xacro:unless value="${model == 'virtual'}">
         <visual>
-          <origin xyz="${screw_offset_x} 0 ${screw_offset_z}" rpy="0 0 0"/>
+          <origin xyz="${screw_offset_x} 0 ${screw_offset_z}" rpy="0 0 0" />
           <geometry>
-            <mesh filename="file://$(find walkie_description)/meshes/walkie/depth_camera/zed/${model}.stl"/>
+            <mesh
+                            filename="package://walkie_description/meshes/walkie/depth_camera/zed/${model}.stl"
+                        />
           </geometry>
           <material name="zed_mat">
-            <color rgba="${mat}"/>
+            <color rgba="${mat}" />
           </material>
         </visual>
         <collision>
-          <origin xyz="${screw_offset_x} 0 ${screw_offset_z}" rpy="0 0 0"/>
+          <origin xyz="${screw_offset_x} 0 ${screw_offset_z}" rpy="0 0 0" />
           <geometry>
-            <mesh filename="file://$(find walkie_description)/meshes/walkie/depth_camera/zed/${model}.stl"/>
+            <mesh
+                            filename="package://walkie_description/meshes/walkie/depth_camera/zed/${model}.stl"
+                        />
           </geometry>
         </collision>
@@ -177,7 +184,7 @@
     </link>
     <joint name="${name}_camera_center_joint" type="fixed">
-      <parent link="${name}_camera_link"/>
-      <child link="${name}_camera_center"/>
-      <origin xyz="0 0 ${height/2}" rpy="0 ${bottom_slope} 0"/>
+      <parent link="${name}_camera_link" />
+      <child link="${name}_camera_center" />
+      <origin xyz="0 0 ${height/2}" rpy="0 ${bottom_slope} 0" />
     </joint>
     <xacro:unless value="${mono}">
@@ -186,16 +193,20 @@
         <xacro:if value="${model == 'virtual'}">
           <visual>
-            <origin xyz="0 0 0" rpy="0 0 0"/>
+            <origin xyz="0 0 0" rpy="0 0 0" />
             <geometry>
-              <mesh filename="file://$(find walkie_description)/meshes/walkie/depth_camera/zed/${model}.stl"/>
+              <mesh
+                                filename="package://walkie_description/meshes/walkie/depth_camera/zed/${model}.stl"
+                            />
             </geometry>
             <material name="zed_mat">
-              <color rgba="${mat}"/>
+              <color rgba="${mat}" />
             </material>
           </visual>
           <collision>
-            <origin xyz="0 0 0" rpy="0 0 0"/>
+            <origin xyz="0 0 0" rpy="0 0 0" />
             <geometry>
-              <mesh filename="file://$(find walkie_description)/meshes/walkie/depth_camera/zed/${model}.stl"/>
+              <mesh
+                                filename="package://walkie_description/meshes/walkie/depth_camera/zed/${model}.stl"
+                            />
             </geometry>
           </collision>
@@ -203,13 +214,13 @@
       </link>
       <joint name="${name}_left_camera_joint" type="fixed">
-        <parent link="${name}_camera_center"/>
-        <child link="${name}_left_camera_frame"/>
-        <origin xyz="${optical_offset_x} ${baseline/2} 0" rpy="0 0 0"/>
-      </joint>
-      <link name="${name}_left_camera_frame_optical"/>
+        <parent link="${name}_camera_center" />
+        <child link="${name}_left_camera_frame" />
+        <origin xyz="${optical_offset_x} ${baseline/2} 0" rpy="0 0 0" />
+      </joint>
+      <link name="${name}_left_camera_frame_optical" />
       <joint name="${name}_left_camera_optical_joint" type="fixed">
-        <origin xyz="0 0 0" rpy="-${M_PI/2} 0.0 -${M_PI/2}"/>
-        <parent link="${name}_left_camera_frame"/>
-        <child link="${name}_left_camera_frame_optical"/>
+        <origin xyz="0 0 0" rpy="-${M_PI/2} 0.0 -${M_PI/2}" />
+        <parent link="${name}_left_camera_frame" />
+        <child link="${name}_left_camera_frame_optical" />
       </joint>
       <!-- Right Camera -->
@@ -217,16 +228,20 @@
         <xacro:if value="${model == 'virtual'}">
           <visual>
-            <origin xyz="0 0 0" rpy="0 0 0"/>
+            <origin xyz="0 0 0" rpy="0 0 0" />
             <geometry>
-              <mesh filename="file://$(find walkie_description)/meshes/walkie/depth_camera/zed/${model}.stl"/>
+              <mesh
+                                filename="package://walkie_description/meshes/walkie/depth_camera/zed/${model}.stl"
+                            />
             </geometry>
             <material name="zed_mat">
-              <color rgba="${mat}"/>
+              <color rgba="${mat}" />
             </material>
           </visual>
           <collision>
-            <origin xyz="0 0 0" rpy="0 0 0"/>
+            <origin xyz="0 0 0" rpy="0 0 0" />
             <geometry>
-              <mesh filename="file://$(find walkie_description)/meshes/walkie/depth_camera/zed/${model}.stl"/>
+              <mesh
+                                filename="package://walkie_description/meshes/walkie/depth_camera/zed/${model}.stl"
+                            />
             </geometry>
           </collision>
@@ -234,39 +249,39 @@
       </link>
       <joint name="${name}_right_camera_joint" type="fixed">
-        <parent link="${name}_camera_center"/>
-        <child link="${name}_right_camera_frame"/>
-        <origin xyz="${optical_offset_x} -${baseline/2} 0" rpy="0 0 0"/>
-      </joint>
-      <link name="${name}_right_camera_frame_optical"/>
+        <parent link="${name}_camera_center" />
+        <child link="${name}_right_camera_frame" />
+        <origin xyz="${optical_offset_x} -${baseline/2} 0" rpy="0 0 0" />
+      </joint>
+      <link name="${name}_right_camera_frame_optical" />
       <joint name="${name}_right_camera_optical_joint" type="fixed">
-        <origin xyz="0 0 0" rpy="-${M_PI/2} 0.0 -${M_PI/2}"/>
-        <parent link="${name}_right_camera_frame"/>
-        <child link="${name}_right_camera_frame_optical"/>
+        <origin xyz="0 0 0" rpy="-${M_PI/2} 0.0 -${M_PI/2}" />
+        <parent link="${name}_right_camera_frame" />
+        <child link="${name}_right_camera_frame_optical" />
       </joint>
       <!-- ZED2 Sensors -->
       <xacro:if value="${model == 'zed2'}">
-        <link name="${name}_mag_link"/>
+        <link name="${name}_mag_link" />
         <joint name="${name}_mag_joint" type="fixed">
-          <parent link="${name}_camera_center"/>
-          <child link="${name}_mag_link"/>
-          <origin xyz="0 0 0" rpy="0 0 0"/>
+          <parent link="${name}_camera_center" />
+          <child link="${name}_mag_link" />
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