Commit message: feat:wristcam_link

File: urdf/openarm/ee/openarm_hand.xacro (robot description, xacro)
@@ -70,4 +70,20 @@
       <mimic joint="${ee_prefix}finger_joint1" />
     </joint>
+    <link name="${ee_prefix}wristcam_bracket">
+      <visual name="${ee_prefix}wristcam_bracket_visual">
+        <origin xyz="0.0095 0 -0.0055" rpy="3.125 -1.57 0" />
+        <geometry>
+          <mesh filename="package://${description_pkg}/meshes/openarm/arm/${arm_type}/visual/wristcam_bracket.stl" scale="0.001 0.001 0.001" />
+        </geometry>
+        <material name="wristcam_bracket_material">
+          <color rgba="0.2 0.2 0.2 1.0" />
+        </material>
+      </visual>
+    </link>
+    <joint name="${ee_prefix}wristcam_bracket_joint" type="fixed">
+      <parent link="${ee_prefix}hand" />
+      <child link="${ee_prefix}wristcam_bracket" />
+      <origin xyz="0 0 0" rpy="0 0 0 " />
+    </joint>
   </xacro:macro>
 </robot>

Commit message: feat:wristcam_collision

File: urdf/openarm/ee/openarm_hand.xacro (robot description, xacro)
@@ -80,4 +80,10 @@
         </material>
       </visual>
+      <collision name="${ee_prefix}wristcam_bracket_collision">
+        <origin xyz="0.0095 0 -0.0055" rpy="3.125 -1.57 0" />
+        <geometry>
+          <mesh filename="package://${description_pkg}/meshes/openarm/arm/${arm_type}/visual/wristcam_bracket.stl" scale="0.001 0.001 0.001" />
+        </geometry>
+      </collision>
     </link>
     <joint name="${ee_prefix}wristcam_bracket_joint" type="fixed">
