Commit message: feat:optimize collision model

File: urdf/openarm/ee/openarm_hand.xacro (robot description, xacro)
@@ -75,5 +75,5 @@
         <origin xyz="0.0095 0 -0.0055" rpy="3.125 -1.57 0" />
         <geometry>
-          <mesh filename="package://${description_pkg}/meshes/openarm/arm/${arm_type}/visual/wristcam_bracket.stl" scale="0.001 0.001 0.001" />
+          <mesh filename="package://${description_pkg}/meshes/openarm/ee/${ee_type}/visual/wristcam_bracket.stl" scale="0.001 0.001 0.001" />
         </geometry>
         <material name="wristcam_bracket_material">
@@ -84,5 +84,5 @@
         <origin xyz="0.0095 0 -0.0055" rpy="3.125 -1.57 0" />
         <geometry>
-          <mesh filename="package://${description_pkg}/meshes/openarm/arm/${arm_type}/visual/wristcam_bracket.stl" scale="0.001 0.001 0.001" />
+          <mesh filename="package://${description_pkg}/meshes/openarm/ee/${ee_type}/collision/wristcam_bracket.stl" scale="0.001 0.001 0.001" />
         </geometry>
       </collision>

File: urdf/walkie/depth_camera/zed/zed_macro.urdf.xacro (robot description, xacro)
@@ -25,5 +25,5 @@
   <xacro:macro
         name="zed_camera"
-        params="name=zed model=zed enable_gnss=false custom_baseline=0 *gnss_origin"
+        params="name=zed model=zed enable_gnss=false custom_baseline=0 enable_collision=true *gnss_origin"
     >
     <xacro:if value="${model == 'zed'}">
@@ -173,12 +173,14 @@
           </material>
         </visual>
-        <collision>
-          <origin xyz="${screw_offset_x} 0 ${screw_offset_z}" rpy="0 0 0" />
-          <geometry>
-            <mesh
-                            filename="package://walkie_description/meshes/walkie/depth_camera/zed/${model}.stl"
-                        />
-          </geometry>
-        </collision>
+        <xacro:if value="${enable_collision}">
+          <collision>
+            <origin xyz="${screw_offset_x} 0 ${screw_offset_z}" rpy="0 0 0" />
+            <geometry>
+              <mesh
+                              filename="package://walkie_description/meshes/walkie/depth_camera/zed/${model}.stl"
+                          />
+            </geometry>
+          </collision>
+        </xacro:if>
       </xacro:unless>
     </link>
@@ -203,12 +205,14 @@
             </material>
           </visual>
-          <collision>
-            <origin xyz="0 0 0" rpy="0 0 0" />
-            <geometry>
-              <mesh
-                                filename="package://walkie_description/meshes/walkie/depth_camera/zed/${model}.stl"
-                            />
-            </geometry>
-          </collision>
+          <xacro:if value="${enable_collision}">
+            <collision>
+              <origin xyz="0 0 0" rpy="0 0 0" />
+              <geometry>
+                <mesh
+                                  filename="package://walkie_description/meshes/walkie/depth_camera/zed/${model}.stl"
+                              />
+              </geometry>
+            </collision>
+          </xacro:if>
         </xacro:if>
       </link>
@@ -238,12 +242,14 @@
             </material>
           </visual>
-          <collision>
-            <origin xyz="0 0 0" rpy="0 0 0" />
-            <geometry>
-              <mesh
-                                filename="package://walkie_description/meshes/walkie/depth_camera/zed/${model}.stl"
-                            />
-            </geometry>
-          </collision>
+          <xacro:if value="${enable_collision}">
+            <collision>
+              <origin xyz="0 0 0" rpy="0 0 0" />
+              <geometry>
+                <mesh
+                                  filename="package://walkie_description/meshes/walkie/depth_camera/zed/${model}.stl"
+                              />
+              </geometry>
+            </collision>
+          </xacro:if>
         </xacro:if>
       </link>

File: urdf/walkie/head/servo_camera.urdf.xacro (robot description, xacro)
@@ -25,5 +25,5 @@
         <origin xyz="0 0 0" rpy="0 0 0"/>
         <geometry>
-          <mesh filename="package://walkie_description/meshes/walkie/HeadCameraMount_simple.stl"/>
+          <mesh filename="package://walkie_description/meshes/walkie/HeadCameraMount_collision.stl"/>
         </geometry>
       </collision>
@@ -34,5 +34,5 @@
     </link>
     <!-- ============ ZED Camera Body ============ -->
-    <xacro:zed_camera name="$(arg camera_name)" model="$(arg camera_model)">
+    <xacro:zed_camera name="$(arg camera_name)" model="$(arg camera_model)" enable_collision="false">
       <origin xyz="0 0 0" rpy="0 0 0"/>
     </xacro:zed_camera>
