Commit message: feat:lift-joint-param

File: urdf/walkie/depth_camera/d415/d415.urdf.xacro (robot description, xacro)
@@ -150,19 +150,4 @@
           <visualize>1</visualize>
           <gz_frame_id>${name}_color_optical_frame</gz_frame_id>
-          <plugin name="${name}_color_controller" filename="libgazebo_ros_camera.so">
-            <alwaysOn>true</alwaysOn>
-            <updateRate>0.0</updateRate>
-            <cameraName>${name}/color/</cameraName>
-            <imageTopicName>image_raw</imageTopicName>
-            <cameraInfoTopicName>camera_info</cameraInfoTopicName>
-            <frameName>${name}_color_optical_frame</frameName>
-            <!--<hackBaseline>0.07</hackBaseline>-->
-            <hackBaseline>0.0</hackBaseline>
-            <distortionK1>0.0</distortionK1>
-            <distortionK2>0.0</distortionK2>
-            <distortionK3>0.0</distortionK3>
-            <distortionT1>0.0</distortionT1>
-            <distortionT2>0.0</distortionT2>
-          </plugin>
         </sensor>
       </xacro:if>
@@ -193,19 +178,4 @@
           <update_rate>${updaterate}</update_rate>
           <visualize>0</visualize>
-          <plugin name="{name}_left_ir_controller" filename="libgazebo_ros_camera.so">
-            <alwaysOn>true</alwaysOn>
-            <updateRate>0.0</updateRate>
-            <cameraName>${name}/left_ir/</cameraName>
-            <imageTopicName>image_raw</imageTopicName>
-            <cameraInfoTopicName>camera_info</cameraInfoTopicName>
-            <frameName>${name}_left_ir_optical_frame</frameName>
-            <!--<hackBaseline>0.07</hackBaseline>-->
-            <hackBaseline>0.0</hackBaseline>
-            <distortionK1>0.0</distortionK1>
-            <distortionK2>0.0</distortionK2>
-            <distortionK3>0.0</distortionK3>
-            <distortionT1>0.0</distortionT1>
-            <distortionT2>0.0</distortionT2>
-          </plugin>
         </sensor>
         <sensor name="${name}_right_ired_sensor" type="camera">
@@ -234,19 +204,4 @@
           <update_rate>${updaterate}</update_rate>
           <visualize>0</visualize>
-          <plugin name="{name}_right_ir_controller" filename="libgazebo_ros_camera.so">
-            <alwaysOn>true</alwaysOn>
-            <updateRate>0.0</updateRate>
-            <cameraName>${name}/right_ir/</cameraName>
-            <imageTopicName>image_raw</imageTopicName>
-            <cameraInfoTopicName>camera_info</cameraInfoTopicName>
-            <frameName>${name}_right_ir_optical_frame</frameName>
-            <!--<hackBaseline>0.07</hackBaseline>-->
-            <hackBaseline>0.0</hackBaseline>
-            <distortionK1>0.0</distortionK1>
-            <distortionK2>0.0</distortionK2>
-            <distortionK3>0.0</distortionK3>
-            <distortionT1>0.0</distortionT1>
-            <distortionT2>0.0</distortionT2>
-          </plugin>
         </sensor>
       </xacro:if>
@@ -279,21 +234,4 @@
           <topic>${name}_depth/image</topic>
           <gz_frame_id>${name}_depth_frame</gz_frame_id>
-          <plugin name="{name}_depth_controller" filename="libgazebo_ros_camera.so">
-            <alwaysOn>true</alwaysOn>
-            <updateRate>0.0</updateRate>
-            <cameraName>${name}/depth/</cameraName>
-            <imageTopicName>image_raw</imageTopicName>
-            <cameraInfoTopicName>camera_info</cameraInfoTopicName>
-            <frameName>${name}_depth_optical_frame</frameName>
-            <hackBaseline>0.07</hackBaseline>
-            <!-- <hackBaseline>0.0</hackBaseline> -->
-            <distortionK1>0.0</distortionK1>
-            <distortionK2>0.0</distortionK2>
-            <distortionK3>0.0</distortionK3>
-            <distortionT1>0.0</distortionT1>
-            <distortionT2>0.0</distortionT2>
-            <min_depth>0.1</min_depth>
-            <max_depth>100.0</max_depth>
-          </plugin>
         </sensor>
       </xacro:if>

File: urdf/walkie/lift/lift.urdf.xacro (robot description, xacro)
@@ -4,5 +4,5 @@
     <joint name="${prefix}_joint" type="prismatic">
         <xacro:insert_block name="joint_origin"/>
-        <limit lower="-0.506" upper="0.00000" effort="0.00000" velocity="0.00000"/>
+        <limit lower="-0.506" upper="0.00000" effort="100.0" velocity="0.1"/>
         <parent link="${parent}"/>
         <child link="${prefix}_link"/>

File: urdf/walkie/ros2_control.xacro (robot description, xacro)
@@ -93,5 +93,10 @@
             <param name="max">0.00000</param>
           </command_interface>
-          <state_interface name="position" />
+          <state_interface name="position">
+            <param name="initial_value">0.0</param>
+          </state_interface>
+          <state_interface name="velocity">
+            <param name="initial_value">0.0</param>
+          </state_interface>
         </joint>
         <xacro:position_arm_joint joint_name="openarm_left_joint1" />
