Commit message: feat:openarm-cofig + lift

File: urdf/walkie/lift/lift.urdf.xacro (robot description, xacro)
@@ -4,5 +4,5 @@
     <joint name="${prefix}_joint" type="prismatic">
         <xacro:insert_block name="joint_origin"/>
-        <limit lower="-0.51510" upper="0.00000" effort="0.00000" velocity="0.00000"/>
+        <limit lower="-0.506" upper="0.00000" effort="0.00000" velocity="0.00000"/>
         <parent link="${parent}"/>
         <child link="${prefix}_link"/>

File: urdf/walkie/ros2_control.xacro (robot description, xacro)
@@ -295,4 +295,16 @@
         </joint>
       </ros2_control>
+      <ros2_control name="LiftSystem" type="system">
+        <hardware>
+          <plugin>mock_components/GenericSystem</plugin>
+        </hardware>
+        <joint name="lift_joint">
+          <command_interface name="position">
+            <param name="min">-0.51510</param>
+            <param name="max">0.00000</param>
+          </command_interface>
+          <state_interface name="position" />
+        </joint>
+      </ros2_control>
       <ros2_control name="ArmSystem" type="system">
         <hardware>

Commit message: feat:preview-lift-rviz

File: urdf/walkie/lift/lift.urdf.xacro (robot description, xacro)
@@ -4,5 +4,5 @@
     <joint name="${prefix}_joint" type="prismatic">
         <xacro:insert_block name="joint_origin"/>
-        <limit lower="0.000" upper="0.743" effort="1000.0" velocity="0.1"/>
+        <limit lower="0.000" upper="0.7435" effort="1000.0" velocity="0.1"/>
         <parent link="${parent}"/>
         <child link="${prefix}_link"/>

Commit message: fix:mimic finger

File: urdf/walkie/lift/lift.urdf.xacro (robot description, xacro)
@@ -4,5 +4,5 @@
     <joint name="${prefix}_joint" type="prismatic">
         <xacro:insert_block name="joint_origin"/>
-        <limit lower="0.000" upper="0.7435" effort="1000.0" velocity="0.1"/>
+        <limit lower="0.000" upper="0.7435" effort="10000.0" velocity="0.1"/>
         <parent link="${parent}"/>
         <child link="${prefix}_link"/>

File: urdf/walkie/ros2_control.xacro (robot description, xacro)
@@ -175,5 +175,17 @@
         <xacro:position_arm_joint joint_name="openarm_right_joint7" />
         <xacro:position_arm_joint joint_name="openarm_left_finger_joint1" />
+        <joint name="openarm_left_finger_joint2">
+          <param name="mimic">openarm_left_finger_joint1</param>
+          <param name="multiplier">1.0</param>
+          <state_interface name="position" />
+          <state_interface name="velocity" />
+        </joint>
         <xacro:position_arm_joint joint_name="openarm_right_finger_joint1" />
+        <joint name="openarm_right_finger_joint2">
+          <param name="mimic">openarm_right_finger_joint1</param>
+          <param name="multiplier">1.0</param>
+          <state_interface name="position" />
+          <state_interface name="velocity" />
+        </joint>
       </ros2_control>
     </xacro:if>

Commit message: fix:conflict remain

File: urdf/walkie/lift/lift.urdf.xacro (robot description, xacro)
@@ -4,9 +4,5 @@
     <joint name="${prefix}_joint" type="prismatic">
         <xacro:insert_block name="joint_origin"/>
-<<<<<<< HEAD
-        <limit lower="0.000" upper="0.7435" effort="1000.0" velocity="0.1"/>
-=======
         <limit lower="0.000" upper="0.7435" effort="10000.0" velocity="0.1"/>
->>>>>>> test/real-bringup
         <parent link="${parent}"/>
         <child link="${prefix}_link"/>
