Commit message: fix(urdf): raise lift joint lower limit to 0.08 m

File: urdf/walkie/lift/lift.urdf.xacro (robot description, xacro)
@@ -4,5 +4,5 @@
     <joint name="${prefix}_joint" type="prismatic">
         <xacro:insert_block name="joint_origin"/>
-        <limit lower="0.000" upper="0.7435" effort="10000.0" velocity="0.1"/>
+        <limit lower="0.080" upper="0.7435" effort="10000.0" velocity="0.1"/>
         <parent link="${parent}"/>
         <child link="${prefix}_link"/>

File: urdf/walkie/ros2_control.xacro (robot description, xacro)
@@ -383,5 +383,5 @@
         <joint name="lift_joint">
           <command_interface name="position">
-            <param name="min">0.00000</param>
+            <param name="min">0.08000</param>
             <param name="max">0.74350</param>
           </command_interface>
