Commit message: add real hardware ros2 control urdf config

File: urdf/walkie/ros2_control.xacro (robot description, xacro)
@@ -2,4 +2,5 @@
 <robot xmlns:xacro="http://www.ros.org/wiki/xacro">
   <xacro:macro name="ros2_control" params="ros2_control">
+    <!-- Simulation - Gazebo based ros2_control -->
     <xacro:if value="${ros2_control == 'gazebo'}">
       <ros2_control name="GazeboSimSystem" type="system">
@@ -41,12 +42,8 @@
       </ros2_control>
     </xacro:if>
+    <!-- Issac Sim/ MicroROS : Topic based ros2_control -->
     <xacro:if value="${ros2_control == 'topic_base'}">
       <ros2_control name="topic_base_controller" type="system">
         <hardware>
-          <plugin>topic_based_ros2_control/TopicBasedSystem</plugin>
-          <param name="joint_commands_topic">/drivebase_joint_cmd</param>
-          <param name="joint_states_topic">/drivebase_joint_states</param>
-          <!-- <param name="sum_wrapped_joint_states">true</param> -->
-          <param name="trigger_joint_command_threshold">-1.0</param>
         </hardware>
         <joint name="fl_wheel_joint">
@@ -84,4 +81,101 @@
       </ros2_control>
     </xacro:if>
+    <!-- Real Hardware : real_robot based ros2_control -->
+    <xacro:if value="${ros2_control == 'real_robot'}">
+      <ros2_control name="topic_base_controller" type="system">
+        <hardware>
+          <plugin>cubemars_hardware/CubeMarsSystemHardware</plugin>
+          <param name="can_interface">can0</param>
+        </hardware>
+        <joint name="fl_wheel_joint">
+          <param name="can_id">1</param>
+          <param name="pole_pairs">14</param>
+          <param name="gear_ratio">10</param>
+          <param name="kt">0.123</param>
+          <param name="enc_off">0.0</param>
+          <param name="trq_limit">30</param>
+          <xacro:if value="${read_only}">
+            <param name="read_only">1</param>
+          </xacro:if>
+          <command_interface name="position" />
+          <command_interface name="velocity">
+            <param name="min"> -16.00</param>
+            <param name="max"> 16.00</param>
+          </command_interface>
+          <command_interface name="acceleration" />
+          <command_interface name="effort" />
+          <state_interface name="position" />
+          <state_interface name="velocity" />
+          <state_interface name="effort" />
+          <state_interface name="temperature" />
+        </joint>
+        <joint name="fr_wheel_joint">
+          <param name="can_id">2</param>
+          <param name="pole_pairs">14</param>
+          <param name="gear_ratio">10</param>
+          <param name="kt">0.123</param>
+          <param name="enc_off">0.0</param>
+          <param name="trq_limit">30</param>
+          <xacro:if value="${read_only}">
+            <param name="read_only">1</param>
+          </xacro:if>
+          <command_interface name="position" />
+          <command_interface name="velocity">
+            <param name="min"> -16.00</param>
+            <param name="max"> 16.00</param>
+          </command_interface>
+          <command_interface name="acceleration" />
+          <command_interface name="effort" />
+          <state_interface name="position" />
+          <state_interface name="velocity" />
+          <state_interface name="effort" />
+          <state_interface name="temperature" />
+        </joint>
+        <joint name="br_wheel_joint">
+          <param name="can_id">3</param>
+          <param name="pole_pairs">14</param>
+          <param name="gear_ratio">10</param>
+          <param name="kt">0.123</param>
+          <param name="enc_off">0.0</param>
+          <param name="trq_limit">30</param>
+          <xacro:if value="${read_only}">
+            <param name="read_only">1</param>
+          </xacro:if>
+          <command_interface name="position" />
+          <command_interface name="velocity">
+            <param name="min"> -16.00</param>
+            <param name="max"> 16.00</param>
+          </command_interface>
+          <command_interface name="acceleration" />
+          <command_interface name="effort" />
+          <state_interface name="position" />
+          <state_interface name="velocity" />
+          <state_interface name="effort" />
+          <state_interface name="temperature" />
+        </joint>
+        <joint name="bl_wheel_joint">
+          <param name="can_id">4</param>
+          <param name="pole_pairs">14</param>
+          <param name="gear_ratio">10</param>
+          <param name="kt">0.123</param>
+          <param name="enc_off">0.0</param>
+          <param name="trq_limit">30</param>
+          <xacro:if value="${read_only}">
+            <param name="read_only">1</param>
+          </xacro:if>
+          <command_interface name="position" />
+          <command_interface name="velocity">
+            <param name="min"> -16.00</param>
+            <param name="max"> 16.00</param>
+          </command_interface>
+          <command_interface name="acceleration" />
+          <command_interface name="effort" />
+          <state_interface name="position" />
+          <state_interface name="velocity" />
+          <state_interface name="effort" />
+          <state_interface name="temperature" />
+        </joint>
+      </ros2_control>
+    </xacro:if>
     <gazebo>
       <plugin name="gz_ros2_control::GazeboSimROS2ControlPlugin"

Commit message: feat: add ros2_control for servo joint

File: urdf/walkie/ros2_control.xacro (robot description, xacro)
@@ -169,4 +169,15 @@
         </joint>
       </ros2_control>
+      <ros2_control name="HeadServoSystem" type="system">
+        <hardware>
+          <plugin>topic_based_ros2_control/TopicBasedSystem</plugin>
+          <param name="joint_commands_topic">/head_servo_joint_cmd</param>
+          <param name="joint_states_topic">/head_servo_joint_states</param>
+        </hardware>
+        <joint name="head_servo_joint">
+          <command_interface name="position" />
+          <state_interface name="position" />
+        </joint>
+      </ros2_control>
     </xacro:if>
     <gazebo>

Commit message: feat: add mock hardware for launching without robot for testing software separately w/o full system

File: urdf/walkie/ros2_control.xacro (robot description, xacro)
@@ -1,5 +1,52 @@
-<?xml version="1.0"?>
+<?xml version="1.0" ?>
 <robot xmlns:xacro="http://www.ros.org/wiki/xacro">
   <xacro:macro name="ros2_control" params="ros2_control">
+    <!-- Mock hardware -->
+    <xacro:if value="${ros2_control == 'mock'}">
+        <ros2_control name="MockSystem" type="system">
+        <hardware>
+            <plugin>mock_components/GenericSystem</plugin>
+        </hardware>
+        <joint name="fl_wheel_joint">
+            <command_interface name="velocity">
+            <param name="min"> -3.14</param>
+            <param name="max"> 3.14</param>
+            </command_interface>
+            <state_interface name="velocity" />
+            <state_interface name="position" />
+        </joint>
+        <joint name="fr_wheel_joint">
+            <command_interface name="velocity">
+            <param name="min"> -3.14</param>
+            <param name="max"> 3.14</param>
+            </command_interface>
+            <state_interface name="velocity" />
+            <state_interface name="position" />
+        </joint>
+        <joint name="br_wheel_joint">
+            <command_interface name="velocity">
+            <param name="min"> -3.14</param>
+            <param name="max"> 3.14</param>
+            </command_interface>
+            <state_interface name="velocity" />
+            <state_interface name="position" />
+        </joint>
+        <joint name="bl_wheel_joint">
+            <command_interface name="velocity">
+            <param name="min"> -3.14</param>
+            <param name="max"> 3.14</param>
+            </command_interface>
+            <state_interface name="velocity" />
+            <state_interface name="position" />
+        </joint>
+        <joint name="head_servo_joint">
+            <command_interface name="position">
+            <param name="min"> -1.54</param>
+            <param name="max"> 1.54</param>
+            </command_interface>
+            <state_interface name="position" />
+        </joint>
+        </ros2_control>
+    </xacro:if>
     <!-- Simulation - Gazebo based ros2_control -->
     <xacro:if value="${ros2_control == 'gazebo'}">
@@ -190,8 +237,9 @@
     <gazebo>
       <plugin
-        name="gz_ros2_control::GazeboSimROS2ControlPlugin"
-        filename="libgz_ros2_control-system.so"
-      >
-        <parameters>$(find walkie_description)/config/ros2_controller/sim_controllers.yaml</parameters>
+                name="gz_ros2_control::GazeboSimROS2ControlPlugin"
+                filename="libgz_ros2_control-system.so"
+            >
+        <parameters
+                >$(find walkie_description)/config/ros2_controller/sim_controllers.yaml</parameters>
       </plugin>
     </gazebo>
