Commit message: feat: add isaac sim ros2 control support

File: urdf/walkie/ros2_control.xacro (robot description, xacro)
@@ -8,4 +8,6 @@
         <param name="max">${vel_max}</param>
       </command_interface>
+      <command_interface name="position" />
+      <command_interface name="effort" />
       <state_interface name="velocity" />
       <state_interface name="position" />
@@ -16,4 +18,6 @@
     <joint name="${joint_name}">
       <command_interface name="position" />
+      <command_interface name="velocity" />
+      <command_interface name="effort" />
       <state_interface name="position">
         <param name="initial_value">0.0</param>
@@ -26,7 +30,7 @@
   <!-- Sub-macro: CubeMars wheel joint (real_robot) -->
   <xacro:macro
-    name="cubemars_wheel_joint"
-    params="name can_id pole_pairs gear_ratio kt enc_off trq_limit read_only vel_min=-16 vel_max=16"
-  >
+        name="cubemars_wheel_joint"
+        params="name can_id pole_pairs gear_ratio kt enc_off trq_limit read_only vel_min=-16 vel_max=16"
+    >
     <joint name="${name}">
       <param name="can_id">${can_id}</param>
@@ -58,23 +62,23 @@
         </hardware>
         <xacro:wheel_velocity_joint
-          name="fl_wheel_joint"
-          vel_min="-3.14"
-          vel_max="3.14"
-        />
-        <xacro:wheel_velocity_joint
-          name="fr_wheel_joint"
-          vel_min="-3.14"
-          vel_max="3.14"
-        />
-        <xacro:wheel_velocity_joint
-          name="br_wheel_joint"
-          vel_min="-3.14"
-          vel_max="3.14"
-        />
-        <xacro:wheel_velocity_joint
-          name="bl_wheel_joint"
-          vel_min="-3.14"
-          vel_max="3.14"
-        />
+                    name="fl_wheel_joint"
+                    vel_min="-3.14"
+                    vel_max="3.14"
+                />
+        <xacro:wheel_velocity_joint
+                    name="fr_wheel_joint"
+                    vel_min="-3.14"
+                    vel_max="3.14"
+                />
+        <xacro:wheel_velocity_joint
+                    name="br_wheel_joint"
+                    vel_min="-3.14"
+                    vel_max="3.14"
+                />
+        <xacro:wheel_velocity_joint
+                    name="bl_wheel_joint"
+                    vel_min="-3.14"
+                    vel_max="3.14"
+                />
         <joint name="head_servo_joint">
           <command_interface name="position">
@@ -116,23 +120,23 @@
         </hardware>
         <xacro:wheel_velocity_joint
-          name="fl_wheel_joint"
-          vel_min="-3.14"
-          vel_max="3.14"
-        />
-        <xacro:wheel_velocity_joint
-          name="fr_wheel_joint"
-          vel_min="-3.14"
-          vel_max="3.14"
-        />
-        <xacro:wheel_velocity_joint
-          name="br_wheel_joint"
-          vel_min="-3.14"
-          vel_max="3.14"
-        />
-        <xacro:wheel_velocity_joint
-          name="bl_wheel_joint"
-          vel_min="-3.14"
-          vel_max="3.14"
-        />
+                    name="fl_wheel_joint"
+                    vel_min="-3.14"
+                    vel_max="3.14"
+                />
+        <xacro:wheel_velocity_joint
+                    name="fr_wheel_joint"
+                    vel_min="-3.14"
+                    vel_max="3.14"
+                />
+        <xacro:wheel_velocity_joint
+                    name="br_wheel_joint"
+                    vel_min="-3.14"
+                    vel_max="3.14"
+                />
+        <xacro:wheel_velocity_joint
+                    name="bl_wheel_joint"
+                    vel_min="-3.14"
+                    vel_max="3.14"
+                />
         <joint name="head_servo_joint">
           <command_interface name="position">
@@ -171,26 +175,64 @@
       <ros2_control name="TopicBaseSystem" type="system">
         <hardware>
-        </hardware>
-        <xacro:wheel_velocity_joint
-          name="fl_wheel_joint"
-          vel_min="-16"
-          vel_max="16"
-        />
-        <xacro:wheel_velocity_joint
-          name="fr_wheel_joint"
-          vel_min="-16"
-          vel_max="16"
-        />
-        <xacro:wheel_velocity_joint
-          name="br_wheel_joint"
-          vel_min="-16"
-          vel_max="16"
-        />
-        <xacro:wheel_velocity_joint
-          name="bl_wheel_joint"
-          vel_min="-16"
-          vel_max="16"
-        />
-      </ros2_control>
+            <plugin>topic_based_ros2_control/TopicBasedSystem</plugin>
+            <param name="joint_commands_topic">/isaac_joint_commands</param>
+            <param name="joint_states_topic">/isaac_joint_states</param>
+            <!-- <param name="sum_wrapped_joint_states">true</param> -->
+        </hardware>
+        <xacro:wheel_velocity_joint
+                    name="fl_wheel_joint"
+                    vel_min="-16"
+                    vel_max="16"
+                />
+        <xacro:wheel_velocity_joint
+                    name="fr_wheel_joint"
+                    vel_min="-16"
+                    vel_max="16"
+                />
+        <xacro:wheel_velocity_joint
+                    name="br_wheel_joint"
+                    vel_min="-16"
+                    vel_max="16"
+                />
+        <xacro:wheel_velocity_joint
+                    name="bl_wheel_joint"
+                    vel_min="-16"
+                    vel_max="16"
+                />
+        <joint name="head_servo_joint">
+            <command_interface name="velocity" />
+            <command_interface name="effort" />
+            <command_interface name="position">
+                <param name="min">-1.54</param>
+                <param name="max">1.54</param>
+            </command_interface>
+            <state_interface name="position" />
+        </joint>
+        <joint name="lift_joint">
+            <command_interface name="velocity" />
+            <command_interface name="effort" />
+            <command_interface name="position">
+                <param name="min">-0.51510</param>
+                <param name="max">0.00000</param>
+            </command_interface>
+            <state_interface name="position" />
+        </joint>
+        <xacro:position_arm_joint joint_name="openarm_left_joint1" />
+        <xacro:position_arm_joint joint_name="openarm_left_joint2" />
+        <xacro:position_arm_joint joint_name="openarm_left_joint3" />
+        <xacro:position_arm_joint joint_name="openarm_left_joint4" />
+        <xacro:position_arm_joint joint_name="openarm_left_joint5" />
+        <xacro:position_arm_joint joint_name="openarm_left_joint6" />
+        <xacro:position_arm_joint joint_name="openarm_left_joint7" />
+        <xacro:position_arm_joint joint_name="openarm_right_joint1" />
+        <xacro:position_arm_joint joint_name="openarm_right_joint2" />
+        <xacro:position_arm_joint joint_name="openarm_right_joint3" />
+        <xacro:position_arm_joint joint_name="openarm_right_joint4" />
+        <xacro:position_arm_joint joint_name="openarm_right_joint5" />
+        <xacro:position_arm_joint joint_name="openarm_right_joint6" />
+        <xacro:position_arm_joint joint_name="openarm_right_joint7" />
+        <xacro:position_arm_joint joint_name="openarm_left_finger_joint1" />
+        <xacro:position_arm_joint joint_name="openarm_right_finger_joint1" />
+        </ros2_control>
     </xacro:if>
     <!-- Real Hardware : real_robot based ros2_control -->
@@ -202,43 +244,43 @@
         </hardware>
         <xacro:cubemars_wheel_joint
-          name="fl_wheel_joint"
-          can_id="3"
-          pole_pairs="14"
-          gear_ratio="10"
-          kt="0.123"
-          enc_off="0.0"
-          trq_limit="30"
-          read_only="0"
-        />
+                    name="fl_wheel_joint"
+                    can_id="3"
+                    pole_pairs="14"
+                    gear_ratio="10"
+                    kt="0.123"
+                    enc_off="0.0"
+                    trq_limit="30"
+                    read_only="0"
+                />
         <xacro:cubemars_wheel_joint
-          name="fr_wheel_joint"
-          can_id="1"
-          pole_pairs="14"
-          gear_ratio="10"
-          kt="0.123"
-          enc_off="0.0"
-          trq_limit="30"
-          read_only="0"
-        />
+                    name="fr_wheel_joint"
+                    can_id="1"
+                    pole_pairs="14"
+                    gear_ratio="10"
+                    kt="0.123"
+                    enc_off="0.0"
+                    trq_limit="30"
+                    read_only="0"
+                />
         <xacro:cubemars_wheel_joint
-          name="br_wheel_joint"
-          can_id="4"
-          pole_pairs="14"
-          gear_ratio="10"
-          kt="0.123"
-          enc_off="0.0"
-          trq_limit="30"
-          read_only="0"
-        />
+                    name="br_wheel_joint"
+                    can_id="4"
+                    pole_pairs="14"
+                    gear_ratio="10"
+                    kt="0.123"
+                    enc_off="0.0"
+                    trq_limit="30"
+                    read_only="0"
+                />
         <xacro:cubemars_wheel_joint
-          name="bl_wheel_joint"
-          can_id="2"
-          pole_pairs="14"
-          gear_ratio="10"
-          kt="0.123"
-          enc_off="0.0"
-          trq_limit="30"
-          read_only="0"
-        />
+                    name="bl_wheel_joint"
+                    can_id="2"
+                    pole_pairs="14"
+                    gear_ratio="10"
+                    kt="0.123"
+                    enc_off="0.0"
+                    trq_limit="30"
+                    read_only="0"
+                />
       </ros2_control>
       <ros2_control name="HeadServoSystem" type="system">
@@ -279,9 +321,9 @@
       <gazebo>
         <plugin
-          name="gz_ros2_control::GazeboSimROS2ControlPlugin"
-          filename="libgz_ros2_control-system.so"
-        >
+                    name="gz_ros2_control::GazeboSimROS2ControlPlugin"
+                    filename="libgz_ros2_control-system.so"
+                >
           <parameters
-          >$(find walkie_description)/config/ros2_controller/sim_controllers.yaml</parameters>
+                    >$(find walkie_description)/config/ros2_controller/sim_controllers.yaml</parameters>
         </plugin>
       </gazebo>

Commit message: feat: add unitree lidar urdf

File: urdf/walkie/ros2_control.xacro (robot description, xacro)
@@ -293,12 +293,32 @@
       <ros2_control name="HeadServoSystem" type="system">
         <hardware>
-          <plugin>mock_components/GenericSystem</plugin>
-          <param name="joint_commands_topic">/head_servo_joint_cmd</param>
-          <param name="joint_states_topic">/head_servo_joint_states</param>
+          <plugin>dynamixel_hardware_interface/DynamixelHardware</plugin>
+          <param name="port_name">/dev/ttyUSB0</param>
+          <param name="baud_rate">57600</param>
+          <param name="number_of_joints">1</param>
+          <param name="number_of_transmissions">1</param>
+          <param name="dynamixel_model_folder">/param/dxl_model</param>
         </hardware>
         <joint name="head_servo_joint">
-          <command_interface name="position" />
-          <state_interface name="position" />
-        </joint>
+          <command_interface name="position">
+            <param name="min">-0.7854</param>
+            <param name="max">0.7854</param>
+          </command_interface>
+          <state_interface name="position"/>
+          <state_interface name="velocity"/>
+          <state_interface name="effort"/>
+        </joint>
+        <gpio name="head_servo_joint">
+          <param name="type">dxl</param>
+          <param name="ID">2</param>
+          <command_interface name="Goal Position"/>
+          <state_interface name="Present Position"/>
+          <state_interface name="Present Velocity"/>
+          <state_interface name="Present Load"/>
+          <param name="Position P Gain">800</param>
+          <param name="Position I Gain">100</param>
+          <param name="Position D Gain">100</param>
+          <param name="Drive Mode">0</param>
+        </gpio>
       </ros2_control>
       <ros2_control name="LiftSystem" type="system">

Commit message: feat(description): integrate openarm real hardware configuration
Updates the main robot URDF and ros2_control configuration to support the bimanual arms on the real robot.

NOTE: This configuration currently breaks simulation pipelines. The robot compiles and runs successfully on physical hardware, but additional gazebo/mock matching configurations are required to restore simulation functionality.

File: urdf/walkie/ros2_control.xacro (robot description, xacro)
@@ -24,4 +24,7 @@
       </state_interface>
       <state_interface name="velocity">
+        <param name="initial_value">0.0</param>
+      </state_interface>
+      <state_interface name="effort">
         <param name="initial_value">0.0</param>
       </state_interface>
@@ -54,5 +57,34 @@
     </joint>
   </xacro:macro>
-  <xacro:macro name="ros2_control" params="ros2_control">
+  <!-- Global helper macro to configure real arm hardware joints cleanly -->
+  <xacro:macro name="configure_joint" params="joint_name initial_position">
+    <joint name="${joint_name}">
+      <command_interface name="position"/>
+      <command_interface name="velocity"/>
+      <command_interface name="effort"/>
+      <state_interface name="position">
+        <param name="initial_value">${initial_position}</param>
+      </state_interface>
+      <state_interface name="velocity">
+        <param name="initial_value">0.0</param>
+      </state_interface>
+      <state_interface name="effort">
+        <param name="initial_value">0.0</param>
+      </state_interface>
+    </joint>
+  </xacro:macro>
+  <!-- Main Macro Declaration (ros2_control included back into parameters list) -->
+  <xacro:macro name="ros2_control"
+            params="ros2_control
+                arm_type:=^|openarm
+                control_gains:=^|{}
+                left_can_interface:=^|can1
+                right_can_interface:=^|can0
+                use_fake_hardware:=^|true
+                fake_sensor_commands:=^|false
+                hand:=^|false
+                left_arm_prefix:=^|left_
+                right_arm_prefix:=^|right_
+                can_fd:=^|true">
     <!-- Mock hardware -->
     <xacro:if value="${ros2_control == 'mock'}">
@@ -241,5 +273,5 @@
         <xacro:position_arm_joint joint_name="openarm_left_finger_joint1" />
         <xacro:position_arm_joint joint_name="openarm_right_finger_joint1" />
-        </ros2_control>
+      </ros2_control>
     </xacro:if>
     <!-- Real Hardware : real_robot based ros2_control -->
@@ -248,5 +280,5 @@
         <hardware>
           <plugin>cubemars_hardware/CubeMarsSystemHardware</plugin>
-          <param name="can_interface">can0</param>
+          <param name="can_interface">can2</param>
         </hardware>
         <xacro:cubemars_wheel_joint
@@ -299,4 +331,5 @@
           <param name="number_of_transmissions">1</param>
           <param name="dynamixel_model_folder">/param/dxl_model</param>
+          <param name="disable_torque_at_init">true</param>
         </hardware>
         <joint name="head_servo_joint">
@@ -331,27 +364,11 @@
             <param name="max">0.74300</param>
           </command_interface>
-          <state_interface name="position" />
-        </joint>
-      </ros2_control>
-      <ros2_control name="ArmSystem" type="system">
-        <hardware>
-          <plugin>mock_components/GenericSystem</plugin>
-        </hardware>
-        <xacro:position_arm_joint joint_name="openarm_left_joint1" />
-        <xacro:position_arm_joint joint_name="openarm_left_joint2" />
-        <xacro:position_arm_joint joint_name="openarm_left_joint3" />
-        <xacro:position_arm_joint joint_name="openarm_left_joint4" />
-        <xacro:position_arm_joint joint_name="openarm_left_joint5" />
-        <xacro:position_arm_joint joint_name="openarm_left_joint6" />
-        <xacro:position_arm_joint joint_name="openarm_left_joint7" />
-        <xacro:position_arm_joint joint_name="openarm_right_joint1" />
-        <xacro:position_arm_joint joint_name="openarm_right_joint2" />
-        <xacro:position_arm_joint joint_name="openarm_right_joint3" />
-        <xacro:position_arm_joint joint_name="openarm_right_joint4" />
-        <xacro:position_arm_joint joint_name="openarm_right_joint5" />
-        <xacro:position_arm_joint joint_name="openarm_right_joint6" />
-        <xacro:position_arm_joint joint_name="openarm_right_joint7" />
-        <xacro:position_arm_joint joint_name="openarm_left_finger_joint1" />
-        <xacro:position_arm_joint joint_name="openarm_right_finger_joint1" />
+          <state_interface name="position">
+            <param name="initial_value">0.0</param>
+          </state_interface>
+          <state_interface name="velocity">
+            <param name="initial_value">0.0</param>
+          </state_interface>
+        </joint>
       </ros2_control>
     </xacro:if>

Commit message: fix:mimic finger

File: urdf/walkie/ros2_control.xacro (robot description, xacro)
@@ -211,5 +211,17 @@
         <xacro:position_arm_joint joint_name="openarm_right_joint7" />
         <xacro:position_arm_joint joint_name="openarm_left_finger_joint1" />
+        <joint name="openarm_left_finger_joint2">
+          <param name="mimic">openarm_left_finger_joint1</param>
+          <param name="multiplier">1.0</param>
+          <state_interface name="position" />
+          <state_interface name="velocity" />
+        </joint>
         <xacro:position_arm_joint joint_name="openarm_right_finger_joint1" />
+        <joint name="openarm_right_finger_joint2">
+          <param name="mimic">openarm_right_finger_joint1</param>
+          <param name="multiplier">1.0</param>
+          <state_interface name="position" />
+          <state_interface name="velocity" />
+        </joint>
       </ros2_control>
     </xacro:if>

Commit message: fix:init value

File: urdf/walkie/ros2_control.xacro (robot description, xacro)
@@ -15,5 +15,5 @@
   </xacro:macro>
   <!-- Sub-macro: Position-controlled arm joint (mock/gazebo/topic_base) -->
-  <xacro:macro name="position_arm_joint" params="joint_name">
+  <xacro:macro name="position_arm_joint" params="joint_name initial_position:=^|0.0">
     <joint name="${joint_name}">
       <command_interface name="position" />
@@ -21,5 +21,5 @@
       <command_interface name="effort" />
       <state_interface name="position">
-        <param name="initial_value">0.0</param>
+        <param name="initial_value">${initial_position}</param>
       </state_interface>
       <state_interface name="velocity">
@@ -132,15 +132,15 @@
           </state_interface>
         </joint>
-        <xacro:position_arm_joint joint_name="openarm_left_joint1" />
+        <xacro:position_arm_joint joint_name="openarm_left_joint1" initial_position="0.2618" />
         <xacro:position_arm_joint joint_name="openarm_left_joint2" />
         <xacro:position_arm_joint joint_name="openarm_left_joint3" />
-        <xacro:position_arm_joint joint_name="openarm_left_joint4" />
+        <xacro:position_arm_joint joint_name="openarm_left_joint4" initial_position="0.2618" />
         <xacro:position_arm_joint joint_name="openarm_left_joint5" />
         <xacro:position_arm_joint joint_name="openarm_left_joint6" />
         <xacro:position_arm_joint joint_name="openarm_left_joint7" />
-        <xacro:position_arm_joint joint_name="openarm_right_joint1" />
+        <xacro:position_arm_joint joint_name="openarm_right_joint1" initial_position="-0.2618" />
         <xacro:position_arm_joint joint_name="openarm_right_joint2" />
         <xacro:position_arm_joint joint_name="openarm_right_joint3" />
-        <xacro:position_arm_joint joint_name="openarm_right_joint4" />
+        <xacro:position_arm_joint joint_name="openarm_right_joint4" initial_position="0.2618" />
         <xacro:position_arm_joint joint_name="openarm_right_joint5" />
         <xacro:position_arm_joint joint_name="openarm_right_joint6" />
@@ -192,15 +192,15 @@
           </state_interface>
         </joint>
-        <xacro:position_arm_joint joint_name="openarm_left_joint1" />
+        <xacro:position_arm_joint joint_name="openarm_left_joint1" initial_position="0.2618" />
         <xacro:position_arm_joint joint_name="openarm_left_joint2" />
         <xacro:position_arm_joint joint_name="openarm_left_joint3" />
-        <xacro:position_arm_joint joint_name="openarm_left_joint4" />
+        <xacro:position_arm_joint joint_name="openarm_left_joint4" initial_position="0.2618" />
         <xacro:position_arm_joint joint_name="openarm_left_joint5" />
         <xacro:position_arm_joint joint_name="openarm_left_joint6" />
         <xacro:position_arm_joint joint_name="openarm_left_joint7" />
-        <xacro:position_arm_joint joint_name="openarm_right_joint1" />
+        <xacro:position_arm_joint joint_name="openarm_right_joint1" initial_position="-0.2618" />
         <xacro:position_arm_joint joint_name="openarm_right_joint2" />
         <xacro:position_arm_joint joint_name="openarm_right_joint3" />
-        <xacro:position_arm_joint joint_name="openarm_right_joint4" />
+        <xacro:position_arm_joint joint_name="openarm_right_joint4" initial_position="0.2618" />
         <xacro:position_arm_joint joint_name="openarm_right_joint5" />
         <xacro:position_arm_joint joint_name="openarm_right_joint6" />
@@ -269,15 +269,15 @@
             <state_interface name="position" />
         </joint>
-        <xacro:position_arm_joint joint_name="openarm_left_joint1" />
+        <xacro:position_arm_joint joint_name="openarm_left_joint1" initial_position="0.2618" />
         <xacro:position_arm_joint joint_name="openarm_left_joint2" />
         <xacro:position_arm_joint joint_name="openarm_left_joint3" />
-        <xacro:position_arm_joint joint_name="openarm_left_joint4" />
+        <xacro:position_arm_joint joint_name="openarm_left_joint4" initial_position="0.2618" />
         <xacro:position_arm_joint joint_name="openarm_left_joint5" />
         <xacro:position_arm_joint joint_name="openarm_left_joint6" />
         <xacro:position_arm_joint joint_name="openarm_left_joint7" />
-        <xacro:position_arm_joint joint_name="openarm_right_joint1" />
+        <xacro:position_arm_joint joint_name="openarm_right_joint1" initial_position="-0.2618" />
         <xacro:position_arm_joint joint_name="openarm_right_joint2" />
         <xacro:position_arm_joint joint_name="openarm_right_joint3" />
-        <xacro:position_arm_joint joint_name="openarm_right_joint4" />
+        <xacro:position_arm_joint joint_name="openarm_right_joint4" initial_position="0.2618" />
         <xacro:position_arm_joint joint_name="openarm_right_joint5" />
         <xacro:position_arm_joint joint_name="openarm_right_joint6" />
