Commit message: fix(description): add base collision box for arm clearance
Co-Authored-By: Claude Opus 4.8 (1M context) <noreply@anthropic.com>

File: urdf/walkie/base/base.urdf.xacro (robot description, xacro)
@@ -33,4 +33,10 @@
         </geometry>
       </collision>
+      <collision>
+        <origin xyz="0 0.07 0.845" rpy="0 0 0"/>
+        <geometry>
+          <box size="0.46 0.07 1.04"/>
+        </geometry>
+      </collision>
       <xacro:inertial_cylinder mass="${base_mass}" length="${bass_thickness}" radius="${base_radian}">
         <origin xyz="0 0 0" rpy="0 0 0"/>
