Commit message: fix: delete scale for new optimized mesh file

File: urdf/walkie/base/base.urdf.xacro (robot description, xacro)
@@ -17,20 +17,20 @@
         <geometry>
           <!-- <mesh filename="package://walkie_description/meshes/walkie/base_link.dae"/> -->
-          <mesh filename="package://walkie_description/meshes/walkie/base_link2.stl" scale="0.001 0.001 0.001"/>
+          <mesh filename="package://walkie_description/meshes/walkie/base_link2.stl"/>
         </geometry>
         <material name="grey"/>
       </visual>
       <collision>
-        <origin xyz="0 0 0.165" rpy="0 0 0" />
-          <geometry>
-            <cylinder radius="0.3" length="0.33"/>
+        <origin xyz="0 0 0.165" rpy="0 0 0"/>
+        <geometry>
+          <cylinder radius="0.3" length="0.33"/>
           <!-- <mesh filename="package://walkie_description/meshes/walkie/base_link_collision.stl"/> -->
-          </geometry>
+        </geometry>
       </collision>
       <collision>
-        <origin xyz="0 0 0.615" rpy="0 0 0" />
-            <geometry>
-              <box size="0.32 0.2 0.57" />
-            </geometry>
+        <origin xyz="0 0 0.615" rpy="0 0 0"/>
+        <geometry>
+          <box size="0.32 0.2 0.57"/>
+        </geometry>
       </collision>
       <xacro:inertial_cylinder mass="${base_mass}" length="${bass_thickness}" radius="${base_radian}">

Commit message: feat: update collision geometry

File: urdf/walkie/base/base.urdf.xacro (robot description, xacro)
@@ -27,10 +27,10 @@
         </geometry>
       </collision>
-      <!-- <collision>
-        <origin xyz="0 0 0.605" rpy="0 0 0"/>
+      <collision>
+        <origin xyz="0 0.07 0.725" rpy="0 0 0"/>
         <geometry>
-          <box size="0.3 0.19 0.54"/>
+          <box size="0.196 0.18 0.80"/>
         </geometry>
-      </collision> -->
+      </collision>
       <xacro:inertial_cylinder mass="${base_mass}" length="${bass_thickness}" radius="${base_radian}">
         <origin xyz="0 0 0" rpy="0 0 0"/>

File: urdf/walkie/lift/lift.urdf.xacro (robot description, xacro)
@@ -16,8 +16,21 @@
             <material name="grey"/>
         </visual>
-        <collision name="lift_collision">
+        <!-- <collision name="lift_collision">
             <origin rpy="0.00000 0.00000 -0.00000" xyz="-0.00000 -0.08773 0.09614"/>
             <geometry>
                 <box size="0.34666 0.35267 0.18936"/>
+            </geometry>
+        </collision> -->
+        <collision name="top_bar">
+            <origin xyz="0 0 0.122" rpy="0 0 0"/>
+            <geometry>
+            <box size="0.346 0.174 0.132"/>
+            </geometry>
+        </collision>
+        <!-- Vertical stem -->
+        <collision name="stem">
+            <origin xyz="0 -0.172 0.122" rpy="0 0 0"/>
+            <geometry>
+            <box size="0.190 0.190 0.132"/>
             </geometry>
         </collision>

Commit message: fix(urdf): update robot collision meshes and openarm config

File: urdf/walkie/base/base.urdf.xacro (robot description, xacro)
@@ -34,7 +34,7 @@
       </collision>
       <collision>
-        <origin xyz="0 0.07 0.845" rpy="0 0 0"/>
+        <origin xyz="-0.115 0.07 0.845" rpy="0 0 0"/>
         <geometry>
-          <box size="0.46 0.07 1.04"/>
+          <box size="0.23 0.07 1.04"/>
         </geometry>
       </collision>
