Commit message: feat: optimize mesh file by post-processing on blender using decimate modifier

File: urdf/walkie/base/base.urdf.xacro (robot description, xacro)
@@ -17,5 +17,5 @@
         <origin xyz="0 0 0" rpy="0 0 0"/>
         <geometry>
-          <mesh filename="package://walkie_description/meshes/walkie/base_link.stl"/>
+          <mesh filename="package://walkie_description/meshes/walkie/base_link_simple.stl"/>
         </geometry>
         <material name="grey"/>

File: urdf/walkie/head/servo_camera.urdf.xacro (robot description, xacro)
@@ -19,5 +19,5 @@
         <origin xyz="0 0 0" rpy="0 0 0"/>
         <geometry>
-          <mesh filename="package://walkie_description/meshes/walkie/HeadCameraMount.stl"/>
+          <mesh filename="package://walkie_description/meshes/walkie/HeadCameraMount_simple.stl"/>
         </geometry>
       </visual>
@@ -25,5 +25,5 @@
         <origin xyz="0 0 0" rpy="0 0 0"/>
         <geometry>
-          <mesh filename="package://walkie_description/meshes/walkie/HeadCameraMount.stl"/>
+          <mesh filename="package://walkie_description/meshes/walkie/HeadCameraMount_simple.stl"/>
         </geometry>
       </collision>
@@ -44,5 +44,4 @@
         <camera name="${prefix}_left">
           <horizontal_fov>1.9199</horizontal_fov>
-          <!-- ZED2i: 110 deg -->
           <image>
             <width>1920</width>

File: urdf/walkie/lift/lift.urdf.xacro (robot description, xacro)
@@ -12,5 +12,5 @@
         <visual name="lift">
             <geometry>
-                <mesh filename="package://walkie_description/meshes/walkie/Lift.stl"/>
+                <mesh filename="package://walkie_description/meshes/walkie/Lift_simple.stl"/>
             </geometry>
             <material name="grey"/>
