Commit message: fix(openarm): remove negative collision scales, re-bake link3 transform, and clean xacro
- Re-bake transform on modified link3.dae with identity scene matrix for Isaac Sim compatibility
- Add pre-mirrored collision meshes (linkX_symp_inv.stl and finger_inv.stl) with positive scale
- Select _symp_inv collision meshes dynamically when reflect == -1 in openarm_macro.xacro
- Update right_finger collision in openarm_hand.xacro to use finger_inv.stl with positive scale
- Preserve original OpenArm v1.0 link3 visual and collision meshes
- Remove stray backtick character in openarm_macro.xacro

File: urdf/openarm/arm/openarm_macro.xacro (robot description, xacro)
@@ -23,4 +23,5 @@
     <!-- <xacro:property name="prefix" value="${'' if no_prefix else arm_prefix + arm_type + '_'}" /> -->
     <xacro:property name="prefix" value="${'' if no_prefix else 'openarm' + '_' +  arm_prefix}" />
+    <xacro:property name="collision_mesh" value="${name + '_symp_inv.stl' if reflect == -1 else name + '_symp.stl'}" />
     <link name="${prefix}${name}">
       <visual name="${prefix}${name}_visual">
@@ -33,8 +34,7 @@
         <xacro:openarm-kinematics-link config="${kinematics_link}" name="${name}" />
         <geometry>
-          <mesh filename="package://${description_pkg}/meshes/openarm/arm/${arm_type}/collision/${name}_symp.stl" scale="0.001 ${0.001*reflect} 0.001" />
-          <!-- <mesh filename="package://${description_pkg}/meshes/arm/${arm_type}/collision/${name}.stl" scale="0.001 0.001 0.001" /> -->
+          <mesh filename="package://${description_pkg}/meshes/openarm/arm/${arm_type}/collision/${collision_mesh}" scale="0.001 0.001 0.001" />
         </geometry>
-      </collision>`
+      </collision>
       <xacro:openarm-inertials name="${name}" inertials="${inertials}" reflect="${reflect}" />
     </link>

File: urdf/openarm/ee/openarm_hand.xacro (robot description, xacro)
@@ -50,5 +50,5 @@
         <xacro:openarm-ee-kinematics-link config="${ee_kinematics_link}" name="right_finger" />
         <geometry>
-          <mesh filename="package://${description_pkg}/meshes/openarm/ee/${ee_type}/collision/finger.stl" scale="0.001 -0.001 0.001" />
+          <mesh filename="package://${description_pkg}/meshes/openarm/ee/${ee_type}/collision/finger_inv.stl" scale="0.001 0.001 0.001" />
         </geometry>
       </collision>

Commit message: docs(openarm): add pre-mirrored visual meshes and simulation collider compatibility notes
- Add pre-mirrored visual meshes (link0-7_inv.dae/stl and finger_inv.dae/stl)
- Clean up obsolete left_symp collision files
- Update openarm_macro.xacro and openarm_hand.xacro with compatibility comments
- Document negative scale reflection issues across PhysX-based platforms (SAPIEN, Isaac Sim, O3DE) in readme.md

File: urdf/openarm/arm/openarm_macro.xacro (robot description, xacro)
@@ -23,4 +23,8 @@
     <!-- <xacro:property name="prefix" value="${'' if no_prefix else arm_prefix + arm_type + '_'}" /> -->
     <xacro:property name="prefix" value="${'' if no_prefix else 'openarm' + '_' +  arm_prefix}" />
+    <!-- Pre-mirrored meshes (_inv.dae, _symp_inv.stl) with positive scale are used instead of
+         negative scaling (e.g. scale="... -0.001 ...") to prevent PhysX/engine cooking failures
+         in SAPIEN, Isaac Sim, and O3DE (see readme.md). -->
+    <xacro:property name="visual_mesh" value="${name + '_inv.dae' if reflect == -1 else name + '.dae'}" />
     <xacro:property name="collision_mesh" value="${name + '_symp_inv.stl' if reflect == -1 else name + '_symp.stl'}" />
     <link name="${prefix}${name}">
@@ -28,5 +32,5 @@
         <xacro:openarm-kinematics-link config="${kinematics_link}" name="${name}" />
         <geometry>
-          <mesh filename="package://${description_pkg}/meshes/openarm/arm/${arm_type}/visual/${name}.dae" scale="0.001 ${0.001*reflect} 0.001" />
+          <mesh filename="package://${description_pkg}/meshes/openarm/arm/${arm_type}/visual/${visual_mesh}" scale="0.001 0.001 0.001" />
         </geometry>
       </visual>

File: urdf/openarm/ee/openarm_hand.xacro (robot description, xacro)
@@ -41,8 +41,9 @@
     </link>
     <link name="${ee_prefix}right_finger">
+      <!-- Pre-mirrored finger_inv meshes with positive scale prevent PhysX cooking failures in SAPIEN / Isaac Sim / O3DE -->
       <visual name="${ee_prefix}right_finger_visual">
         <xacro:openarm-ee-kinematics-link config="${ee_kinematics_link}" name="right_finger" />
         <geometry>
-          <mesh filename="package://${description_pkg}/meshes/openarm/ee/${ee_type}/visual/finger.dae" scale="0.001 -0.001 0.001"/>
+          <mesh filename="package://${description_pkg}/meshes/openarm/ee/${ee_type}/visual/finger_inv.dae" scale="0.001 0.001 0.001"/>
         </geometry>
       </visual>
